File: Duo_RC1A/Duo_BottomBoard_RC1A.sch (KiCad schematic (older format))
At the start: 0 parts

Commit message: wip balanced outputs
Changed lines of the file:
@@
 $Descr A4 11693 8268
 encoding utf-8
-Sheet 1 9
+Sheet 1 10
 Title "MOD Duo BottomBoard"
 Date "December/2014"
@@
 F1 "Rear_Pannel.sch" 50
 $EndSheet
+$Sheet
+S 5350 4850 1500 1000
+U 548BFDB4
+F0 "Audio _HEADPHONES" 60
+F1 "Audio_HEADPHONES.sch" 60
+$EndSheet
 $EndSCHEMATC
