File: hw-design/bottom-board/connectors.sch (KiCad schematic (older format))
At the start: 28 parts, among them J1 JACK_TRS_6PINS, J2 JACK_TRS_6PINS, J3 JACK_TRS_6PINS, J4 JACK_TRS_6PINS, J5 JACK_TRS_6PINS, J6 RJ45_LEDS, P5 BARREL_JACK, P6 HMI_POWER, P7 SD_CARD, P8 HMI_DATA, P9 SERIAL_DEBUG

Commit message: bottom-board,sch: new annotation
Parts:
- gave numbers to parts that had none: 5
- renumbered C43 to C55, C44 to C56, C45 to C57, R55 to R64, R56 to R65, R57 to R66, R58 to R67, R59 to R68, R60 to R69, R61 to R70, R63 to R76, R64 to R77
Changed lines of the file:
@@
 $EndComp
 $Comp
-L C_Small C43
+L C_Small C55
 U 1 1 550C63C7
 P 2600 1550
-F 0 "C43" H 2700 1550 50  0000 L CNN
+F 0 "C55" H 2700 1550 50  0000 L CNN
 F 1 "100nF" H 2650 1450 50  0000 L CNN
 F 2 "Capacitors_SMD:C_0603" H 2600 1550 60  0001 C CNN
@@
 $EndComp
 $Comp
-L GNDD #PWR0150
+L GNDD #PWR0155
 U 1 1 550C66E7
 P 2300 1700
-F 0 "#PWR0150" H 2300 1450 50  0001 C CNN
+F 0 "#PWR0155" H 2300 1450 50  0001 C CNN
 F 1 "GNDD" H 2300 1550 50  0000 C CNN
 F 2 "" H 2300 1700 60  0000 C CNN
@@
 $EndComp
 $Comp
-L GNDD #PWR0151
+L GNDD #PWR0156
 U 1 1 550C69B3
 P 2600 1700
-F 0 "#PWR0151" H 2600 1450 50  0001 C CNN
+F 0 "#PWR0156" H 2600 1450 50  0001 C CNN
 F 1 "GNDD" H 2600 1550 50  0000 C CNN
 F 2 "" H 2600 1700 60  0000 C CNN
@@
 $EndComp
 $Comp
-L GNDD #PWR0152
+L GNDD #PWR0157
 U 1 1 550C9AAB
 P 7950 5500
-F 0 "#PWR0152" H 7950 5250 50  0001 C CNN
+F 0 "#PWR0157" H 7950 5250 50  0001 C CNN
 F 1 "GNDD" H 7950 5350 50  0000 C CNN
 F 2 "" H 7950 5500 60  0000 C CNN
@@
 $EndComp
 $Comp
-L C_Small C45
+L C_Small C57
 U 1 1 550C9E35
 P 7250 4950
-F 0 "C45" H 7300 4850 50  0000 L CNN
+F 0 "C57" H 7300 4850 50  0000 L CNN
 F 1 "100nF" V 7300 5000 50  0000 L CNN
 F 2 "Capacitors_SMD:C_0603" H 7250 4950 60  0001 C CNN
@@
 $EndComp
 $Comp
-L CP_Small C44
+L CP_Small C56
 U 1 1 550C9E8B
 P 6950 4950
-F 0 "C44" H 7000 4850 50  0000 L CNN
+F 0 "C56" H 7000 4850 50  0000 L CNN
 F 1 "100uF" V 7000 5000 50  0000 L CNN
 F 2 "Capacitors_SMD:c_elec_6.3x5.3" H 6950 4950 60  0001 C CNN
@@
 $EndComp
 $Comp
-L GNDD #PWR0153
+L GNDD #PWR0158
 U 1 1 550CA830
 P 7050 5200
-F 0 "#PWR0153" H 7050 4950 50  0001 C CNN
+F 0 "#PWR0158" H 7050 4950 50  0001 C CNN
 F 1 "GNDD" H 7050 5050 50  0000 C CNN
 F 2 "" H 7050 5200 60  0000 C CNN
@@
 $EndComp
 $Comp
-L GNDA #PWR0154
+L GNDA #PWR0159
 U 1 1 550CF91F
 P 4750 6150
-F 0 "#PWR0154" H 4750 5900 50  0001 C CNN
+F 0 "#PWR0159" H 4750 5900 50  0001 C CNN
 F 1 "GNDA" H 4750 6000 50  0000 C CNN
 F 2 "" H 4750 6150 60  0000 C CNN
@@
 $EndComp
 $Comp
-L GNDA #PWR0155
+L GNDA #PWR0160
 U 1 1 550D3F89
 P 4750 5300
-F 0 "#PWR0155" H 4750 5050 50  0001 C CNN
+F 0 "#PWR0160" H 4750 5050 50  0001 C CNN
 F 1 "GNDA" H 4750 5150 50  0000 C CNN
 F 2 "" H 4750 5300 60  0000 C CNN
@@
 $EndComp
 $Comp
-L GNDA #PWR0156
+L GNDA #PWR0161
 U 1 1 550D3FB0
 P 4750 4450
-F 0 "#PWR0156" H 4750 4200 50  0001 C CNN
+F 0 "#PWR0161" H 4750 4200 50  0001 C CNN
 F 1 "GNDA" H 4750 4300 50  0000 C CNN
 F 2 "" H 4750 4450 60  0000 C CNN
@@
 $EndComp
 $Comp
-L GNDA #PWR0157
+L GNDA #PWR0162
 U 1 1 550D6CF9
 P 2450 5750
-F 0 "#PWR0157" H 2450 5500 50  0001 C CNN
+F 0 "#PWR0162" H 2450 5500 50  0001 C CNN
 F 1 "GNDA" H 2450 5600 50  0000 C CNN
 F 2 "" H 2450 5750 60  0000 C CNN
@@
 $EndComp
 $Comp
-L GNDA #PWR0158
+L GNDA #PWR0163
 U 1 1 550D7285
 P 2450 4900
-F 0 "#PWR0158" H 2450 4650 50  0001 C CNN
+F 0 "#PWR0163" H 2450 4650 50  0001 C CNN
 F 1 "GNDA" H 2450 4750 50  0000 C CNN
 F 2 "" H 2450 4900 60  0000 C CNN
@@
 $EndComp
 $Comp
-L GNDD #PWR0159
+L GNDD #PWR0164
 U 1 1 550DDA88
 P 1650 2500
-F 0 "#PWR0159" H 1650 2250 50  0001 C CNN
+F 0 "#PWR0164" H 1650 2250 50  0001 C CNN
 F 1 "GNDD" H 1650 2350 50  0000 C CNN
 F 2 "" H 1650 2500 60  0000 C CNN
@@
 $EndComp
 $Comp
-L GNDD #PWR0160
+L GNDD #PWR0165
 U 1 1 550DEDBA
 P 9500 2850
-F 0 "#PWR0160" H 9500 2600 50  0001 C CNN
+F 0 "#PWR0165" H 9500 2600 50  0001 C CNN
 F 1 "GNDD" H 9500 2700 50  0000 C CNN
 F 2 "" H 9500 2850 60  0000 C CNN
@@
 $EndComp
 $Comp
-L GNDD #PWR0161
+L GNDD #PWR0166
 U 1 1 550AE498
 P 8900 2200
-F 0 "#PWR0161" H 8900 1950 50  0001 C CNN
+F 0 "#PWR0166" H 8900 1950 50  0001 C CNN
 F 1 "GNDD" H 8900 2050 50  0000 C CNN
 F 2 "" H 8900 2200 60  0000 C CNN
@@
 $EndComp
 $Comp
-L GNDD #PWR0162
+L GNDD #PWR0167
 U 1 1 550B207C
 P 9600 2150
-F 0 "#PWR0162" H 9600 1900 50  0001 C CNN
+F 0 "#PWR0167" H 9600 1900 50  0001 C CNN
 F 1 "GNDD" H 9600 2000 50  0000 C CNN
 F 2 "" H 9600 2150 60  0000 C CNN
@@
 $EndComp
 $Comp
-L +3.3V #PWR0163
+L +3.3V #PWR0168
 U 1 1 550B8DEA
 P 5650 1200
-F 0 "#PWR0163" H 5650 1050 50  0001 C CNN
+F 0 "#PWR0168" H 5650 1050 50  0001 C CNN
 F 1 "+3.3V" H 5650 1340 50  0000 C CNN
 F 2 "" H 5650 1200 60  0000 C CNN
@@
 $EndComp
 $Comp
-L R_Small R55
+L R_Small R64
 U 1 1 550B9034
 P 5200 1450
-F 0 "R55" V 5150 1550 50  0000 L CNN
+F 0 "R64" V 5150 1550 50  0000 L CNN
 F 1 "10k" V 5150 1350 50  0000 L CNN
 F 2 "Resistors_SMD:R_0603" H 5200 1450 60  0001 C CNN
@@
 $EndComp
 $Comp
-L R_Small R56
+L R_Small R65
 U 1 1 550B9CEA
 P 5350 1450
-F 0 "R56" V 5300 1550 50  0000 L CNN
+F 0 "R65" V 5300 1550 50  0000 L CNN
 F 1 "10k" V 5300 1350 50  0000 L CNN
 F 2 "Resistors_SMD:R_0603" H 5350 1450 60  0001 C CNN
@@
 $EndComp
 $Comp
-L R_Small R57
+L R_Small R66
 U 1 1 550B9D20
 P 5500 1450
-F 0 "R57" V 5450 1550 50  0000 L CNN
+F 0 "R66" V 5450 1550 50  0000 L CNN
 F 1 "10k" V 5450 1350 50  0000 L CNN
 F 2 "Resistors_SMD:R_0603" H 5500 1450 60  0001 C CNN
@@
 $EndComp
 $Comp
-L R_Small R58
+L R_Small R67
 U 1 1 550B9D5C
 P 5650 1450
-F 0 "R58" V 5600 1550 50  0000 L CNN
+F 0 "R67" V 5600 1550 50  0000 L CNN
 F 1 "10k" V 5600 1350 50  0000 L CNN
 F 2 "Resistors_SMD:R_0603" H 5650 1450 60  0001 C CNN
@@
 $EndComp
 $Comp
-L R_Small R59
+L R_Small R68
 U 1 1 550B9D96
 P 5800 1450
-F 0 "R59" V 5750 1550 50  0000 L CNN
+F 0 "R68" V 5750 1550 50  0000 L CNN
 F 1 "10k" V 5750 1350 50  0000 L CNN
 F 2 "Resistors_SMD:R_0603" H 5800 1450 60  0001 C CNN
@@
 $EndComp
 $Comp
-L R_Small R60
+L R_Small R69
 U 1 1 550B9DD2
 P 5950 1450
-F 0 "R60" V 5900 1550 50  0000 L CNN
+F 0 "R69" V 5900 1550 50  0000 L CNN
 F 1 "10k" V 5900 1350 50  0000 L CNN
 F 2 "Resistors_SMD:R_0603" H 5950 1450 60  0001 C CNN
@@
 $EndComp
 $Comp
-L R_Small R61
+L R_Small R70
 U 1 1 550BB308
 P 6100 1450
-F 0 "R61" V 6050 1550 50  0000 L CNN
+F 0 "R70" V 6050 1550 50  0000 L CNN
 F 1 "10k" V 6050 1350 50  0000 L CNN
 F 2 "Resistors_SMD:R_0603" H 6100 1450 60  0001 C CNN
@@
 $EndComp
 $Comp
-L GNDD #PWR0164
+L GNDD #PWR0169
 U 1 1 550BE3FF
 P 6250 2850
-F 0 "#PWR0164" H 6250 2600 50  0001 C CNN
+F 0 "#PWR0169" H 6250 2600 50  0001 C CNN
 F 1 "GNDD" H 6250 2700 50  0000 C CNN
 F 2 "" H 6250 2850 60  0000 C CNN
@@
 $EndComp
 $Comp
-L R_Small R63
+L R_Small R76
 U 1 1 551A2D92
 P 9250 4350
-F 0 "R63" H 9300 4400 50  0000 L CNN
+F 0 "R76" H 9300 4400 50  0000 L CNN
 F 1 "330R" H 9300 4300 50  0000 L CNN
 F 2 "Resistors_SMD:R_0603" H 9250 4350 60  0001 C CNN
@@
 $EndComp
 $Comp
-L R_Small R64
+L R_Small R77
 U 1 1 551A4873
 P 9250 5050
-F 0 "R64" H 9300 5100 50  0000 L CNN
+F 0 "R77" H 9300 5100 50  0000 L CNN
 F 1 "330R" H 9300 5000 50  0000 L CNN
 F 2 "Resistors_SMD:R_0603" H 9250 5050 60  0001 C CNN
@@
 NoConn ~ 2300 5200
 $Comp
-L GNDD #PWR0165
+L GNDD #PWR0170
 U 1 1 55FAAD4C
 P 9150 4500
-F 0 "#PWR0165" H 9150 4250 50  0001 C CNN
+F 0 "#PWR0170" H 9150 4250 50  0001 C CNN
 F 1 "GNDD" H 9150 4350 50  0000 C CNN
 F 2 "" H 9150 4500 60  0000 C CNN
@@
 	9150 4450 9150 4500
 $Comp
-L GNDD #PWR0166
+L GNDD #PWR0171
 U 1 1 55FAB4D2
 P 9150 5200
-F 0 "#PWR0166" H 9150 4950 50  0001 C CNN
+F 0 "#PWR0171" H 9150 4950 50  0001 C CNN
 F 1 "GNDD" H 9150 5050 50  0000 C CNN
 F 2 "" H 9150 5200 60  0000 C CNN
@@
 	9450 4350 9350 4350
 $Comp
-L +12V #PWR0167
+L +12V #PWR0172
 U 1 1 55FADC86
 P 7250 4550
-F 0 "#PWR0167" H 7250 4400 50  0001 C CNN
+F 0 "#PWR0172" H 7250 4400 50  0001 C CNN
 F 1 "+12V" H 7250 4690 50  0000 C CNN
 F 2 "" H 7250 4550 60  0000 C CNN
@@
 $EndComp
 $Comp
-L +12V #PWR0168
+L +12V #PWR0173
 U 1 1 55FAF2FE
 P 2000 2500
-F 0 "#PWR0168" H 2000 2350 50  0001 C CNN
+F 0 "#PWR0173" H 2000 2350 50  0001 C CNN
 F 1 "+12V" H 2000 2640 50  0000 C CNN
 F 2 "" H 2000 2500 60  0000 C CNN
@@
 Connection ~ 2450 4550
 $Comp
-L R_Small R?
+L R_Small R74
 U 1 1 566413AE
 P 9250 2550
-F 0 "R?" V 9200 2350 50  0000 L CNN
+F 0 "R74" V 9200 2350 50  0000 L CNN
 F 1 "100R" V 9200 2650 50  0000 L CNN
 F 2 "Resistors_SMD:R_0603" H 9250 2550 60  0001 C CNN
@@
 $EndComp
 $Comp
-L R_Small R?
+L R_Small R75
 U 1 1 56642329
 P 9250 2650
-F 0 "R?" V 9200 2450 50  0000 L CNN
+F 0 "R75" V 9200 2450 50  0000 L CNN
 F 1 "100R" V 9200 2750 50  0000 L CNN
 F 2 "Resistors_SMD:R_0603" H 9250 2650 60  0001 C CNN
@@
 	9000 2650 9150 2650
 $Comp
-L R_Small R?
+L R_Small R72
 U 1 1 566433EA
 P 8550 1500
-F 0 "R?" V 8500 1300 50  0000 L CNN
+F 0 "R72" V 8500 1300 50  0000 L CNN
 F 1 "100R" V 8500 1600 50  0000 L CNN
 F 2 "Resistors_SMD:R_0603" H 8550 1500 60  0001 C CNN
@@
 $EndComp
 $Comp
-L R_Small R?
+L R_Small R73
 U 1 1 566433F1
 P 8550 1600
-F 0 "R?" V 8500 1400 50  0000 L CNN
+F 0 "R73" V 8500 1400 50  0000 L CNN
 F 1 "100R" V 8500 1700 50  0000 L CNN
 F 2 "Resistors_SMD:R_0603" H 8550 1600 60  0001 C CNN
@@
 	8300 1600 8450 1600
 $Comp
-L R_Small R?
+L R_Small R71
 U 1 1 56645EF2
 P 7950 5350
-F 0 "R?" H 8000 5400 50  0000 L CNN
+F 0 "R71" H 8000 5400 50  0000 L CNN
 F 1 "100R" H 8000 5300 50  0000 L CNN
 F 2 "Resistors_SMD:R_0805" H 7950 5350 60  0001 C CNN
