File: hw-design/bottom-board/control-chain.sch (KiCad schematic (older format))
At the start: 20 parts, among them Q14 BSS84, Q15 BSS84, U12 ISL83491

Commit message: bottom,sch: fix parts after updating to kicad 5
Parts:
- removed J?: RJ45_LEDS, Connect:RJHSE538X, symbol RJ45_LEDS
- added J?: CC_CONN, symbol Connector:RJ45_LED_Shielded
- C4, C54, C6, C?: symbol C_Small -> Device:C_Small
- C?: symbol CP_Small -> Device:CP_Small
- Q14, Q15: symbol Q_PMOS_GSD -> Transistor_FET:BSS84
- R55, R56, R57, R58, R59, R60, R61, R62, R63, R? (x2): symbol R_Small -> Device:R_Small
- U12: symbol ISL83491 -> Interface_UART:ISL83491
Connections:
- wire segments 68 -> 84

Commit message: bottom,sch: fix ERC issues
Parts:
- gave numbers to parts that had none: 5
- renumbered C6 to C67, C4 to C68, C54 to C71, Q14 to Q5, Q15 to Q6, R55 to R38, R56 to R39, R57 to R40, R58 to R41, R59 to R44, R60 to R45, R61 to R46, R62 to R47, R63 to R48, U12 to U18
Connections:
- wire segments 84 -> 87
Changed lines of the file:
@@
 $EndDescr
 $Comp
-L Device:R_Small R63
+L Device:R_Small R48
 U 1 1 550F230C
 P 7550 2450
-F 0 "R63" H 7600 2500 50  0000 L CNN
+F 0 "R48" H 7600 2500 50  0000 L CNN
 F 1 "100R" H 7600 2400 50  0000 L CNN
 F 2 "Resistors_SMD:R_0805" H 7550 2450 60  0001 C CNN
@@
 $EndComp
 $Comp
-L Device:R_Small R59
+L Device:R_Small R44
 U 1 1 550F26CE
 P 7000 2350
-F 0 "R59" H 6800 2400 50  0000 L CNN
+F 0 "R44" H 6800 2400 50  0000 L CNN
 F 1 "56R" H 6800 2300 50  0000 L CNN
 F 2 "Resistors_SMD:R_0805" H 7000 2350 60  0001 C CNN
@@
 $EndComp
 $Comp
-L Device:R_Small R60
+L Device:R_Small R45
 U 1 1 550F2702
 P 7000 2550
-F 0 "R60" H 7050 2600 50  0000 L CNN
+F 0 "R45" H 7050 2600 50  0000 L CNN
 F 1 "56R" H 7050 2500 50  0000 L CNN
 F 2 "Resistors_SMD:R_0805" H 7000 2550 60  0001 C CNN
@@
 $EndComp
 $Comp
-L Device:C_Small C54
+L Device:C_Small C71
 U 1 1 550F8A1E
 P 6550 1900
-F 0 "C54" V 6600 1950 50  0000 L CNN
+F 0 "C71" V 6600 1950 50  0000 L CNN
 F 1 "100nF" V 6450 1800 50  0000 L CNN
 F 2 "Capacitors_SMD:C_0603" H 6550 1900 60  0001 C CNN
@@
 $EndComp
 $Comp
-L power:GNDD #PWR0144
+L power:GNDD #PWR0194
 U 1 1 550C7BE5
 P 6750 1950
-F 0 "#PWR0144" H 6750 1700 50  0001 C CNN
+F 0 "#PWR0194" H 6750 1700 50  0001 C CNN
 F 1 "GNDD" H 6750 1800 50  0000 C CNN
 F 2 "" H 6750 1950 60  0000 C CNN
@@
 $EndComp
 $Comp
-L power:GNDD #PWR0145
+L power:GNDD #PWR0191
 U 1 1 550C7C57
 P 6400 3600
-F 0 "#PWR0145" H 6400 3350 50  0001 C CNN
+F 0 "#PWR0191" H 6400 3350 50  0001 C CNN
 F 1 "GNDD" H 6400 3450 50  0000 C CNN
 F 2 "" H 6400 3600 60  0000 C CNN
@@
 $EndComp
 $Comp
-L Device:R_Small R56
+L Device:R_Small R39
 U 1 1 5508D60C
 P 5550 2450
-F 0 "R56" V 5450 2350 50  0000 L CNN
+F 0 "R39" V 5450 2350 50  0000 L CNN
 F 1 "100R" V 5650 2350 50  0000 L CNN
 F 2 "Resistors_SMD:R_0603" H 5550 2450 60  0001 C CNN
@@
 $EndComp
 $Comp
-L Device:R_Small R55
+L Device:R_Small R38
 U 1 1 5508D6F9
 P 5500 2950
-F 0 "R55" V 5400 2850 50  0000 L CNN
+F 0 "R38" V 5400 2850 50  0000 L CNN
 F 1 "100R" V 5600 2850 50  0000 L CNN
 F 2 "Resistors_SMD:R_0603" H 5500 2950 60  0001 C CNN
@@
 $EndComp
 $Comp
-L Interface_UART:ISL83491 U12
+L Interface_UART:ISL83491 U18
 U 1 1 5519DD90
 P 6300 2750
-F 0 "U12" H 6100 2100 50  0000 L CNN
+F 0 "U18" H 6100 2100 50  0000 L CNN
 F 1 "ISL83491" H 6300 3350 50  0000 L CNN
 F 2 "Housings_SOIC:SOIC-14_3.9x8.7mm_Pitch1.27mm" H 6300 2750 50  0001 C CIN
@@
 $EndComp
 $Comp
-L power:+3.3V #PWR0146
+L power:+3.3V #PWR0190
 U 1 1 551A1FF5
 P 6200 1800
-F 0 "#PWR0146" H 6200 1650 50  0001 C CNN
+F 0 "#PWR0190" H 6200 1650 50  0001 C CNN
 F 1 "+3.3V" H 6200 1940 50  0000 C CNN
 F 2 "" H 6200 1800 60  0000 C CNN
@@
 $EndComp
 $Comp
-L Device:R_Small R61
+L Device:R_Small R46
 U 1 1 551AA590
 P 7250 2850
-F 0 "R61" H 7050 2900 50  0000 L CNN
+F 0 "R46" H 7050 2900 50  0000 L CNN
 F 1 "56R" H 7050 2800 50  0000 L CNN
 F 2 "Resistors_SMD:R_0805" H 7250 2850 60  0001 C CNN
@@
 $EndComp
 $Comp
-L Device:R_Small R62
+L Device:R_Small R47
 U 1 1 551AAAAD
 P 7250 3050
-F 0 "R62" H 7300 3100 50  0000 L CNN
+F 0 "R47" H 7300 3100 50  0000 L CNN
 F 1 "56R" H 7300 3000 50  0000 L CNN
 F 2 "Resistors_SMD:R_0805" H 7250 3050 60  0001 C CNN
@@
 	5700 2800 5700 2950
 $Comp
-L power:GNDD #PWR0147
+L power:GNDD #PWR0182
 U 1 1 5522D8E7
 P 3750 3450
-F 0 "#PWR0147" H 3750 3200 50  0001 C CNN
+F 0 "#PWR0182" H 3750 3200 50  0001 C CNN
 F 1 "GNDD" H 3750 3300 50  0000 C CNN
 F 2 "" H 3750 3450 60  0000 C CNN
@@
 	4550 1900 5350 1900
 $Comp
-L power:GNDD #PWR0148
+L power:GNDD #PWR0184
 U 1 1 5522FFC1
 P 4250 2550
-F 0 "#PWR0148" H 4250 2300 50  0001 C CNN
+F 0 "#PWR0184" H 4250 2300 50  0001 C CNN
 F 1 "GNDD" H 4250 2400 50  0000 C CNN
 F 2 "" H 4250 2550 60  0000 C CNN
@@
 $EndComp
 $Comp
-L Transistor_FET:BSS84 Q15
+L Transistor_FET:BSS84 Q6
 U 1 1 55FA4B32
 P 4350 1900
-F 0 "Q15" H 4700 1950 50  0000 R CNN
+F 0 "Q6" H 4700 1950 50  0000 R CNN
 F 1 "BSS84" H 4750 1850 50  0000 R CNN
 F 2 "Housings_SOT-23_SOT-143_TSOT-6:SOT-23" H 4550 2000 29  0001 C CNN
@@
 $EndComp
 $Comp
-L Transistor_FET:BSS84 Q14
+L Transistor_FET:BSS84 Q5
 U 1 1 55FA4BE1
 P 3850 2800
-F 0 "Q14" H 4200 2850 50  0000 R CNN
+F 0 "Q5" H 4200 2850 50  0000 R CNN
 F 1 "BSS84" H 4250 2750 50  0000 R CNN
 F 2 "Housings_SOT-23_SOT-143_TSOT-6:SOT-23" H 4050 2900 29  0001 C CNN
@@
 $EndComp
 $Comp
-L power:+3.3V #PWR0149
+L power:+3.3V #PWR0183
 U 1 1 55FA5E06
 P 4250 1600
-F 0 "#PWR0149" H 4250 1450 50  0001 C CNN
+F 0 "#PWR0183" H 4250 1450 50  0001 C CNN
 F 1 "+3.3V" H 4250 1740 50  0000 C CNN
 F 2 "" H 4250 1600 60  0000 C CNN
@@
 Connection ~ 4250 2200
 $Comp
-L power:+3.3V #PWR0150
+L power:+3.3V #PWR0181
 U 1 1 55FA859A
 P 3750 2500
-F 0 "#PWR0150" H 3750 2350 50  0001 C CNN
+F 0 "#PWR0181" H 3750 2350 50  0001 C CNN
 F 1 "+3.3V" H 3750 2640 50  0000 C CNN
 F 2 "" H 3750 2500 60  0000 C CNN
@@
 Connection ~ 3750 3100
 $Comp
-L Device:R_Small R57
+L Device:R_Small R40
 U 1 1 55FB1923
 P 5700 2150
-F 0 "R57" H 5750 2200 50  0000 L CNN
+F 0 "R40" H 5750 2200 50  0000 L CNN
 F 1 "10k" H 5750 2100 50  0000 L CNN
 F 2 "Resistors_SMD:R_0603" H 5700 2150 60  0001 C CNN
@@
 $EndComp
 $Comp
-L Device:R_Small R58
+L Device:R_Small R41
 U 1 1 55FB198B
 P 5700 3350
-F 0 "R58" H 5750 3400 50  0000 L CNN
+F 0 "R41" H 5750 3400 50  0000 L CNN
 F 1 "10k" H 5750 3300 50  0000 L CNN
 F 2 "Resistors_SMD:R_0603" H 5700 3350 60  0001 C CNN
@@
 Connection ~ 5700 3150
 $Comp
-L power:GNDD #PWR0151
+L power:GNDD #PWR0189
 U 1 1 55FB1C75
 P 5700 3500
-F 0 "#PWR0151" H 5700 3250 50  0001 C CNN
+F 0 "#PWR0189" H 5700 3250 50  0001 C CNN
 F 1 "GNDD" H 5700 3350 50  0000 C CNN
 F 2 "" H 5700 3500 60  0000 C CNN
@@
 Connection ~ 5700 2650
 $Comp
-L power:+3.3V #PWR0152
+L power:+3.3V #PWR0188
 U 1 1 55FB2896
 P 5700 1950
-F 0 "#PWR0152" H 5700 1800 50  0001 C CNN
+F 0 "#PWR0188" H 5700 1800 50  0001 C CNN
 F 1 "+3.3V" H 5700 2090 50  0000 C CNN
 F 2 "" H 5700 1950 60  0000 C CNN
@@
 	5700 1950 5700 2050
 $Comp
-L Device:C_Small C4
+L Device:C_Small C68
 U 1 1 59A54006
 P 4250 2400
-F 0 "C4" V 4150 2400 50  0000 R CNN
+F 0 "C68" V 4150 2400 50  0000 R CNN
 F 1 "10uF" V 4350 2300 50  0000 L CNN
 F 2 "Capacitors_SMD:C_0805" H 4250 2400 60  0001 C CNN
@@
 $EndComp
 $Comp
-L Device:C_Small C6
+L Device:C_Small C67
 U 1 1 59A543AD
 P 3750 3300
-F 0 "C6" V 3650 3300 50  0000 R CNN
+F 0 "C67" V 3650 3300 50  0000 R CNN
 F 1 "10uF" V 3850 3200 50  0000 L CNN
 F 2 "Capacitors_SMD:C_0805" H 3750 3300 60  0001 C CNN
@@
 $EndComp
 $Comp
-L power:GNDD #PWR0283
+L power:GNDD #PWR0187
 U 1 1 5B60F824
 P 5650 5600
-F 0 "#PWR0283" H 5650 5350 50  0001 C CNN
+F 0 "#PWR0187" H 5650 5350 50  0001 C CNN
 F 1 "GNDD" H 5650 5450 50  0000 C CNN
 F 2 "" H 5650 5600 60  0000 C CNN
@@
 $EndComp
 $Comp
-L Device:CP_Small C?
+L Device:CP_Small C69
 U 1 1 5B60F833
 P 4650 5400
-F 0 "C?" H 4700 5300 50  0000 L CNN
+F 0 "C69" H 4700 5300 50  0000 L CNN
 F 1 "100uF" V 4700 5450 50  0000 L CNN
 F 2 "Capacitors_SMD:c_elec_5x5.3" H 4650 5400 60  0001 C CNN
@@
 $EndComp
 $Comp
-L power:GNDD #PWR0284
+L power:GNDD #PWR0185
 U 1 1 5B60F83A
 P 4750 5650
-F 0 "#PWR0284" H 4750 5400 50  0001 C CNN
+F 0 "#PWR0185" H 4750 5400 50  0001 C CNN
 F 1 "GNDD" H 4750 5500 50  0000 C CNN
 F 2 "" H 4750 5650 60  0000 C CNN
@@
 $EndComp
 $Comp
-L Device:R_Small R?
+L Device:R_Small R42
 U 1 1 5B60F849
 P 6750 4800
-F 0 "R?" H 6800 4850 50  0000 L CNN
+F 0 "R42" H 6800 4850 50  0000 L CNN
 F 1 "330R" H 6800 4750 50  0000 L CNN
 F 2 "Resistors_SMD:R_0603" H 6750 4800 60  0001 C CNN
@@
 $EndComp
 $Comp
-L Device:R_Small R?
+L Device:R_Small R43
 U 1 1 5B60F851
 P 6750 5400
-F 0 "R?" H 6800 5450 50  0000 L CNN
+F 0 "R43" H 6800 5450 50  0000 L CNN
 F 1 "330R" H 6800 5350 50  0000 L CNN
 F 2 "Resistors_SMD:R_0603" H 6750 5400 60  0001 C CNN
@@
 Connection ~ 4750 5600
 $Comp
-L power:GNDD #PWR0285
+L power:GNDD #PWR0192
 U 1 1 5B60F872
 P 6650 4950
-F 0 "#PWR0285" H 6650 4700 50  0001 C CNN
+F 0 "#PWR0192" H 6650 4700 50  0001 C CNN
 F 1 "GNDD" H 6650 4800 50  0000 C CNN
 F 2 "" H 6650 4950 60  0000 C CNN
@@
 	6650 4900 6650 4950
 $Comp
-L power:GNDD #PWR0286
+L power:GNDD #PWR0193
 U 1 1 5B60F87A
 P 6650 5600
-F 0 "#PWR0286" H 6650 5350 50  0001 C CNN
+F 0 "#PWR0193" H 6650 5350 50  0001 C CNN
 F 1 "GNDD" H 6650 5450 50  0000 C CNN
 F 2 "" H 6650 5600 60  0000 C CNN
@@
 	6950 4800 6850 4800
 $Comp
-L power:+12V #PWR0287
+L power:+12V #PWR0186
 U 1 1 5B60F884
 P 4950 5000
-F 0 "#PWR0287" H 4950 4850 50  0001 C CNN
+F 0 "#PWR0186" H 4950 4850 50  0001 C CNN
 F 1 "+12V" H 4950 5140 50  0000 C CNN
 F 2 "" H 4950 5000 60  0000 C CNN
@@
 Connection ~ 5650 5500
 $Comp
-L Device:C_Small C?
+L Device:C_Small C70
 U 1 1 5B60F82B
 P 4950 5400
-F 0 "C?" H 5000 5300 50  0000 L CNN
+F 0 "C70" H 5000 5300 50  0000 L CNN
 F 1 "100nF" V 5000 5450 50  0000 L CNN
 F 2 "Capacitors_SMD:C_0603" H 4950 5400 60  0001 C CNN
@@
 	5650 5500 5650 5600
 $Comp
-L Connector:RJ45_LED_Shielded J?
+L Connector:RJ45_LED_Shielded J21
 U 1 1 5B7F0E1E
 P 6150 5100
-F 0 "J?" H 6150 5674 50  0000 C CNN
+F 0 "J21" H 6150 5674 50  0000 C CNN
 F 1 "CC_CONN" H 6150 5765 50  0000 C CNN
 F 2 "" V 6150 5125 50  0001 C CNN
@@
 Wire Wire Line
 	5675 5100 5750 5100
+$Comp
+L power:GNDD #PWR0236
+U 1 1 5B6371E3
+P 5925 4450
+F 0 "#PWR0236" H 5925 4200 50  0001 C CNN
+F 1 "GNDD" H 5925 4300 50  0000 C CNN
+F 2 "" H 5925 4450 60  0000 C CNN
+F 3 "" H 5925 4450 60  0000 C CNN
+	1    5925 4450
+	1    0    0    -1
+$EndComp
+Wire Wire Line
+	5925 4450 5925 4375
+Wire Wire Line
+	5925 4375 6150 4375
+Wire Wire Line
+	6150 4375 6150 4600
 $EndSCHEMATC

Commit message: bottom,sch: MPN updated on control chain sheet
Parts:
- removed C67, C68: 10uF, Capacitors_SMD:C_0805, symbol Device:C_Small
- removed C69: 100uF, Capacitors_SMD:c_elec_5x5.3, symbol Device:CP_Small
- removed C70: 100nF, Capacitors_SMD:C_0603, symbol Device:C_Small
- removed Q5: BSS84, Housings_SOT-23_SOT-143_TSOT-6:SOT-23, symbol Transistor_FET:BSS84
- removed R38, R39: 100R, Resistors_SMD:R_0603, symbol Device:R_Small
- removed R43: 330R, Resistors_SMD:R_0603, symbol Device:R_Small
- removed R45, R46, R47: 56R, Resistors_SMD:R_0805, symbol Device:R_Small
- added C? (x2): 10uF, Capacitor_SMD:C_0603_1608Metric, symbol Device:C_Small
- added C?: 10uF 16V, Capacitor_SMD:C_0805_2012Metric, symbol Device:C_Small
- added C?: 100nF, Capacitors_SMD:C_0603, symbol Device:C_Small
- added Q?: BSS84, Housings_SOT-23_SOT-143_TSOT-6:SOT-23, symbol Transistor_FET:BSS84
- added R? (x2): 22R, Resistors_SMD:R_0603, symbol Device:R_Small
- added R?: 220R, Resistors_SMD:R_0603, symbol Device:R_Small
- added R? (x3): 56R, Resistors_SMD:R_0805, symbol Device:R_Small
- C71: MPN C1608X7R1E104K080AA -> (none); MPN1 (none) -> GCM188R71C104KA37D; MPN2 (none) -> C0603X104K8RACTU; MPN3 (none) -> CS0603KRX7R7BB104
- J21: value CC_CONN -> RJHSE-5381; footprint (none) -> Connector_RJ:RJ45_Amphenol_RJHSE538X; MPN (none) -> RJHSE-5381
- Q6: MPN BSS84 -> (none); MPN1 (none) -> BSS84-7-F; MPN2 (none) -> BSS84LT1G; MPN3 (none) -> DMP3099L
- R40, R41: MPN RMCF0603JT10K0 -> (none); MPN1 (none) -> RMCF0603JT10K0; MPN2 (none) -> RCA060310K0JNEA; MPN3 (none) -> ESR03EZPJ103
- R42: value 330R -> 220R; MPN RMCF0603JT330R -> (none); MPN1 (none) -> ESR03EZPJ221; MPN2 (none) -> ERJ-PB3D2200V; MPN3 (none) -> CRCW0603220RJNEAHP
- R44: MPN ERJ-P6WJ560V -> (none); MPN1 (none) -> RMCF0603JT56R0; MPN2 (none) -> ESR03EZPJ560; MPN3 (none) -> RC1608J560CS
- R48: value 100R -> 100R 0.25W; footprint Resistors_SMD:R_0805 -> Resistor_SMD:R_0603_1608Metric; MPN ERJ-P06J101V -> (none); MPN1 (none) -> ESR03EZPJ101; MPN2 (none) -> ERJ-PA3J101V; MPN3 (none) -> RCA0603100RFKEAHP
- U18: footprint Housings_SOIC:SOIC-14_3.9x8.7mm_Pitch1.27mm -> Package_SO:SOIC-14_3.9x8.7mm_P1.27mm
