File: hw-design/bottom-board/control-chain.sch (KiCad schematic (older format))
At the start: 20 parts, among them J21 RJHSE-5381, Q6 BSS84, U18 ISL83491

Commit message: bottom,sch: fix/update footprints field
Parts:
- C70: renamed from C?; footprint Capacitors_SMD:C_0603 -> Capacitor_SMD:C_0603_1608Metric
- C71: footprint Capacitors_SMD:C_0603 -> Capacitor_SMD:C_0603_1608Metric
- Q5: renamed from Q?; footprint Housings_SOT-23_SOT-143_TSOT-6:SOT-23 -> Package_TO_SOT_SMD:SOT-23
- Q6: footprint Housings_SOT-23_SOT-143_TSOT-6:SOT-23 -> Package_TO_SOT_SMD:SOT-23
- R37, R38, R42: renamed from R?; footprint Resistors_SMD:R_0603 -> Resistor_SMD:R_0603_1608Metric
- R39: renamed from R40; footprint Resistors_SMD:R_0603 -> Resistor_SMD:R_0603_1608Metric
- R40: renamed from R41; footprint Resistors_SMD:R_0603 -> Resistor_SMD:R_0603_1608Metric
- R41: renamed from R42; footprint Resistors_SMD:R_0603 -> Resistor_SMD:R_0603_1608Metric
- R43: renamed from R44; footprint Resistors_SMD:R_0805 -> Resistor_SMD:R_0603_1608Metric
- R44, R45, R46: renamed from R?; footprint Resistors_SMD:R_0805 -> Resistor_SMD:R_0603_1608Metric
- gave numbers to parts that had none: 3
- renumbered R48 to R47
Changed lines of the file:
@@
 $EndDescr
 $Comp
-L Device:R_Small R48
+L Device:R_Small R47
 U 1 1 550F230C
 P 7550 2450
-F 0 "R48" H 7600 2500 50  0000 L CNN
+F 0 "R47" H 7600 2500 50  0000 L CNN
 F 1 "100R 0.25W" H 7600 2400 50  0000 L CNN
 F 2 "Resistor_SMD:R_0603_1608Metric" H 7550 2450 60  0001 C CNN
@@
 $EndComp
 $Comp
-L Device:R_Small R44
+L Device:R_Small R43
 U 1 1 550F26CE
 P 7000 2350
-F 0 "R44" H 6800 2400 50  0000 L CNN
+F 0 "R43" H 6800 2400 50  0000 L CNN
 F 1 "56R" H 6800 2300 50  0000 L CNN
-F 2 "Resistors_SMD:R_0805" H 7000 2350 60  0001 C CNN
+F 2 "Resistor_SMD:R_0603_1608Metric" H 7000 2350 60  0001 C CNN
 F 3 "" H 7000 2350 60  0000 C CNN
 F 4 "RMCF0603JT56R0" H 1000 150 50  0001 C CNN "MPN1"
@@
 F 0 "C71" V 6600 1950 50  0000 L CNN
 F 1 "100nF" V 6450 1800 50  0000 L CNN
-F 2 "Capacitors_SMD:C_0603" H 6550 1900 60  0001 C CNN
+F 2 "Capacitor_SMD:C_0603_1608Metric" H 6550 1900 60  0001 C CNN
 F 3 "" H 6550 1900 60  0000 C CNN
 F 4 "" H 1700 150 50  0001 C CNN "MPN"
@@
 	5700 2800 5700 2950
 $Comp
-L power:GNDD #PWR0182
+L power:GNDD #PWR0181
 U 1 1 5522D8E7
 P 3750 3450
-F 0 "#PWR0182" H 3750 3200 50  0001 C CNN
+F 0 "#PWR0181" H 3750 3200 50  0001 C CNN
 F 1 "GNDD" H 3750 3300 50  0000 C CNN
 F 2 "" H 3750 3450 60  0000 C CNN
@@
 	4550 1900 5350 1900
 $Comp
-L power:GNDD #PWR0184
+L power:GNDD #PWR0183
 U 1 1 5522FFC1
 P 4250 2550
-F 0 "#PWR0184" H 4250 2300 50  0001 C CNN
+F 0 "#PWR0183" H 4250 2300 50  0001 C CNN
 F 1 "GNDD" H 4250 2400 50  0000 C CNN
 F 2 "" H 4250 2550 60  0000 C CNN
@@
 F 0 "Q6" H 4550 1825 50  0000 L CNN
 F 1 "BSS84" H 4550 1900 50  0000 L CNN
-F 2 "Housings_SOT-23_SOT-143_TSOT-6:SOT-23" H 4550 2000 29  0001 C CNN
+F 2 "Package_TO_SOT_SMD:SOT-23" H 4550 2000 29  0001 C CNN
 F 3 "" H 4350 1900 60  0000 C CNN
 F 4 "" H 4350 1900 60  0001 C CNN "MPN"
@@
 $EndComp
 $Comp
-L power:+3.3V #PWR0183
+L power:+3.3V #PWR0182
 U 1 1 55FA5E06
 P 4250 1600
-F 0 "#PWR0183" H 4250 1450 50  0001 C CNN
+F 0 "#PWR0182" H 4250 1450 50  0001 C CNN
 F 1 "+3.3V" H 4250 1740 50  0000 C CNN
 F 2 "" H 4250 1600 60  0000 C CNN
@@
 Connection ~ 4250 2200
 $Comp
-L power:+3.3V #PWR0181
+L power:+3.3V #PWR0180
 U 1 1 55FA859A
 P 3750 2500
-F 0 "#PWR0181" H 3750 2350 50  0001 C CNN
+F 0 "#PWR0180" H 3750 2350 50  0001 C CNN
 F 1 "+3.3V" H 3750 2640 50  0000 C CNN
 F 2 "" H 3750 2500 60  0000 C CNN
@@
 Connection ~ 3750 3100
 $Comp
-L Device:R_Small R40
+L Device:R_Small R39
 U 1 1 55FB1923
 P 5700 2150
-F 0 "R40" H 5750 2200 50  0000 L CNN
+F 0 "R39" H 5750 2200 50  0000 L CNN
 F 1 "10k" H 5750 2100 50  0000 L CNN
-F 2 "Resistors_SMD:R_0603" H 5700 2150 60  0001 C CNN
+F 2 "Resistor_SMD:R_0603_1608Metric" H 5700 2150 60  0001 C CNN
 F 3 "" H 5700 2150 60  0000 C CNN
 F 4 "" H 2450 850 50  0001 C CNN "MPN"
@@
 $EndComp
 $Comp
-L Device:R_Small R41
+L Device:R_Small R40
 U 1 1 55FB198B
 P 5700 3350
-F 0 "R41" H 5750 3400 50  0000 L CNN
+F 0 "R40" H 5750 3400 50  0000 L CNN
 F 1 "10k" H 5750 3300 50  0000 L CNN
-F 2 "Resistors_SMD:R_0603" H 5700 3350 60  0001 C CNN
+F 2 "Resistor_SMD:R_0603_1608Metric" H 5700 3350 60  0001 C CNN
 F 3 "" H 5700 3350 60  0000 C CNN
 F 4 "" H 2450 2050 50  0001 C CNN "MPN"
@@
 Connection ~ 5700 3150
 $Comp
-L power:GNDD #PWR0189
+L power:GNDD #PWR0188
 U 1 1 55FB1C75
 P 5700 3500
-F 0 "#PWR0189" H 5700 3250 50  0001 C CNN
+F 0 "#PWR0188" H 5700 3250 50  0001 C CNN
 F 1 "GNDD" H 5700 3350 50  0000 C CNN
 F 2 "" H 5700 3500 60  0000 C CNN
@@
 Connection ~ 5700 2650
 $Comp
-L power:+3.3V #PWR0188
+L power:+3.3V #PWR0187
 U 1 1 55FB2896
 P 5700 1950
-F 0 "#PWR0188" H 5700 1800 50  0001 C CNN
+F 0 "#PWR0187" H 5700 1800 50  0001 C CNN
 F 1 "+3.3V" H 5700 2090 50  0000 C CNN
 F 2 "" H 5700 1950 60  0000 C CNN
@@
 	5700 1950 5700 2050
 $Comp
-L power:GNDD #PWR0187
+L power:GNDD #PWR0186
 U 1 1 5B60F824
 P 5650 5600
-F 0 "#PWR0187" H 5650 5350 50  0001 C CNN
+F 0 "#PWR0186" H 5650 5350 50  0001 C CNN
 F 1 "GNDD" H 5650 5450 50  0000 C CNN
 F 2 "" H 5650 5600 60  0000 C CNN
@@
 $EndComp
 $Comp
-L power:GNDD #PWR0185
+L power:GNDD #PWR0184
 U 1 1 5B60F83A
 P 4750 5650
-F 0 "#PWR0185" H 4750 5400 50  0001 C CNN
+F 0 "#PWR0184" H 4750 5400 50  0001 C CNN
 F 1 "GNDD" H 4750 5500 50  0000 C CNN
 F 2 "" H 4750 5650 60  0000 C CNN
@@
 $EndComp
 $Comp
-L Device:R_Small R42
+L Device:R_Small R41
 U 1 1 5B60F849
 P 6750 4800
-F 0 "R42" H 6800 4850 50  0000 L CNN
+F 0 "R41" H 6800 4850 50  0000 L CNN
 F 1 "220R" H 6800 4750 50  0000 L CNN
-F 2 "Resistors_SMD:R_0603" H 6750 4800 60  0001 C CNN
+F 2 "Resistor_SMD:R_0603_1608Metric" H 6750 4800 60  0001 C CNN
 F 3 "" H 6750 4800 60  0000 C CNN
 F 4 "ESR03EZPJ221" H -3200 600 50  0001 C CNN "MPN1"
@@
 	6950 4800 6850 4800
 $Comp
-L power:+12V #PWR0186
+L power:+12V #PWR0185
 U 1 1 5B60F884
 P 4950 5000
-F 0 "#PWR0186" H 4950 4850 50  0001 C CNN
+F 0 "#PWR0185" H 4950 4850 50  0001 C CNN
 F 1 "+12V" H 4950 5140 50  0000 C CNN
 F 2 "" H 4950 5000 60  0000 C CNN
@@
 	5675 5100 5750 5100
 $Comp
-L power:GNDD #PWR0236
+L power:GNDD #PWR0189
 U 1 1 5B6371E3
 P 5925 4450
-F 0 "#PWR0236" H 5925 4200 50  0001 C CNN
+F 0 "#PWR0189" H 5925 4200 50  0001 C CNN
 F 1 "GNDD" H 5925 4300 50  0000 C CNN
 F 2 "" H 5925 4450 60  0000 C CNN
@@
 P 5500 2950
 AR Path="/54F72B97/5B8069C2" Ref="R?"  Part="1"
-AR Path="/54F72FB6/5B8069C2" Ref="R?"  Part="1"
-F 0 "R?" V 5425 2950 50  0000 C CNN
+AR Path="/54F72FB6/5B8069C2" Ref="R37"  Part="1"
+F 0 "R37" V 5425 2950 50  0000 C CNN
 F 1 "22R" V 5575 2950 50  0000 C CNN
-F 2 "Resistors_SMD:R_0603" H 5500 2950 60  0001 C CNN
+F 2 "Resistor_SMD:R_0603_1608Metric" H 5500 2950 60  0001 C CNN
 F 3 "" H 5500 2950 60  0000 C CNN
 F 4 "RMCF0603JT22R0" H 1200 600 50  0001 C CNN "MPN1"
@@
 $EndComp
 $Comp
-L Transistor_FET:BSS84 Q?
+L Transistor_FET:BSS84 Q5
 U 1 1 5B80AEE9
 P 3850 2800
-F 0 "Q?" H 4050 2725 50  0000 L CNN
+F 0 "Q5" H 4050 2725 50  0000 L CNN
 F 1 "BSS84" H 4050 2800 50  0000 L CNN
-F 2 "Housings_SOT-23_SOT-143_TSOT-6:SOT-23" H 4050 2900 29  0001 C CNN
+F 2 "Package_TO_SOT_SMD:SOT-23" H 4050 2900 29  0001 C CNN
 F 3 "" H 3850 2800 60  0000 C CNN
 F 4 "" H 3850 2800 60  0001 C CNN "MPN"
@@
 AR Path="/54F725AE/5B80C0B0" Ref="C?"  Part="1"
 AR Path="/54F72B97/5B80C0B0" Ref="C?"  Part="1"
-AR Path="/54F72FB6/5B80C0B0" Ref="C?"  Part="1"
-F 0 "C?" V 4125 2400 50  0000 C CNN
+AR Path="/54F72FB6/5B80C0B0" Ref="C68"  Part="1"
+F 0 "C68" V 4125 2400 50  0000 C CNN
 F 1 "10uF" V 4050 2400 50  0000 C CNN
 F 2 "Capacitor_SMD:C_0603_1608Metric" H 4250 2400 60  0001 C CNN
@@
 AR Path="/54F725AE/5B80EB2C" Ref="C?"  Part="1"
 AR Path="/54F72B97/5B80EB2C" Ref="C?"  Part="1"
-AR Path="/54F72FB6/5B80EB2C" Ref="C?"  Part="1"
-F 0 "C?" V 3625 3300 50  0000 C CNN
+AR Path="/54F72FB6/5B80EB2C" Ref="C67"  Part="1"
+F 0 "C67" V 3625 3300 50  0000 C CNN
 F 1 "10uF" V 3550 3300 50  0000 C CNN
 F 2 "Capacitor_SMD:C_0603_1608Metric" H 3750 3300 60  0001 C CNN
@@
 P 4600 5350
 AR Path="/54F7244B/5B818B27" Ref="C?"  Part="1"
-AR Path="/54F72FB6/5B818B27" Ref="C?"  Part="1"
-F 0 "C?" V 4425 5350 50  0000 C CNN
+AR Path="/54F72FB6/5B818B27" Ref="C69"  Part="1"
+F 0 "C69" V 4425 5350 50  0000 C CNN
 F 1 "10uF 16V" V 4500 5350 50  0000 C CNN
 F 2 "Capacitor_SMD:C_0805_2012Metric" H 4600 5350 60  0001 C CNN
@@
 $EndComp
 $Comp
-L Device:C_Small C?
+L Device:C_Small C70
 U 1 1 5B81D52D
 P 4950 5350
-F 0 "C?" V 5125 5350 50  0000 C CNN
+F 0 "C70" V 5125 5350 50  0000 C CNN
 F 1 "100nF" V 5050 5350 50  0000 C CNN
-F 2 "Capacitors_SMD:C_0603" H 4950 5350 60  0001 C CNN
+F 2 "Capacitor_SMD:C_0603_1608Metric" H 4950 5350 60  0001 C CNN
 F 3 "" H 4950 5350 60  0000 C CNN
 F 4 "" H 100 3600 50  0001 C CNN "MPN"
@@
 P 5550 2450
 AR Path="/54F72B97/5B82DE56" Ref="R?"  Part="1"
-AR Path="/54F72FB6/5B82DE56" Ref="R?"  Part="1"
-F 0 "R?" V 5475 2450 50  0000 C CNN
+AR Path="/54F72FB6/5B82DE56" Ref="R38"  Part="1"
+F 0 "R38" V 5475 2450 50  0000 C CNN
 F 1 "22R" V 5625 2450 50  0000 C CNN
-F 2 "Resistors_SMD:R_0603" H 5550 2450 60  0001 C CNN
+F 2 "Resistor_SMD:R_0603_1608Metric" H 5550 2450 60  0001 C CNN
 F 3 "" H 5550 2450 60  0000 C CNN
 F 4 "RMCF0603JT22R0" H 1250 100 50  0001 C CNN "MPN1"
@@
 $EndComp
 $Comp
-L Device:R_Small R?
+L Device:R_Small R42
 U 1 1 5B82F078
 P 6750 5400
-F 0 "R?" H 6800 5450 50  0000 L CNN
+F 0 "R42" H 6800 5450 50  0000 L CNN
 F 1 "220R" H 6800 5350 50  0000 L CNN
-F 2 "Resistors_SMD:R_0603" H 6750 5400 60  0001 C CNN
+F 2 "Resistor_SMD:R_0603_1608Metric" H 6750 5400 60  0001 C CNN
 F 3 "" H 6750 5400 60  0000 C CNN
 F 4 "ESR03EZPJ221" H -3200 1200 50  0001 C CNN "MPN1"
@@
 $EndComp
 $Comp
-L Device:R_Small R?
+L Device:R_Small R44
 U 1 1 5B835BF4
 P 7000 2550
-F 0 "R?" H 6800 2600 50  0000 L CNN
+F 0 "R44" H 6800 2600 50  0000 L CNN
 F 1 "56R" H 6800 2500 50  0000 L CNN
-F 2 "Resistors_SMD:R_0805" H 7000 2550 60  0001 C CNN
+F 2 "Resistor_SMD:R_0603_1608Metric" H 7000 2550 60  0001 C CNN
 F 3 "" H 7000 2550 60  0000 C CNN
 F 4 "RMCF0603JT56R0" H 1000 350 50  0001 C CNN "MPN1"
@@
 $EndComp
 $Comp
-L Device:R_Small R?
+L Device:R_Small R45
 U 1 1 5B837DE0
 P 7250 2850
-F 0 "R?" H 7050 2900 50  0000 L CNN
+F 0 "R45" H 7050 2900 50  0000 L CNN
 F 1 "56R" H 7050 2800 50  0000 L CNN
-F 2 "Resistors_SMD:R_0805" H 7250 2850 60  0001 C CNN
+F 2 "Resistor_SMD:R_0603_1608Metric" H 7250 2850 60  0001 C CNN
 F 3 "" H 7250 2850 60  0000 C CNN
 F 4 "RMCF0603JT56R0" H 1250 650 50  0001 C CNN "MPN1"
@@
 $EndComp
 $Comp
-L Device:R_Small R?
+L Device:R_Small R46
 U 1 1 5B837E52
 P 7250 3050
-F 0 "R?" H 7050 3100 50  0000 L CNN
+F 0 "R46" H 7050 3100 50  0000 L CNN
 F 1 "56R" H 7050 3000 50  0000 L CNN
-F 2 "Resistors_SMD:R_0805" H 7250 3050 60  0001 C CNN
+F 2 "Resistor_SMD:R_0603_1608Metric" H 7250 3050 60  0001 C CNN
 F 3 "" H 7250 3050 60  0000 C CNN
 F 4 "RMCF0603JT56R0" H 1250 850 50  0001 C CNN "MPN1"

Commit message: bottom,sch: rename MPN1 to MPN
Parts:
- C67, C68: MPN (none) -> CL10A106MQ8NNNC; MPN1 CL10A106MQ8NNNC -> (none)
- C69: MPN (none) -> CL21A106KOFNNNE; MPN1 CL21A106KOFNNNE -> (none)
- C70, C71: MPN (none) -> GCM188R71C104KA37D; MPN1 GCM188R71C104KA37D -> (none)
- Q5, Q6: MPN (none) -> BSS84-7-F; MPN1 BSS84-7-F -> (none)
- R37, R38: MPN (none) -> RMCF0603JT22R0; MPN1 RMCF0603JT22R0 -> (none)
- R39, R40: MPN (none) -> RMCF0603JT10K0; MPN1 RMCF0603JT10K0 -> (none)
- R41, R42: MPN (none) -> ESR03EZPJ221; MPN1 ESR03EZPJ221 -> (none)
- R43, R44, R45, R46: MPN (none) -> RMCF0603JT56R0; MPN1 RMCF0603JT56R0 -> (none)
- R47: MPN (none) -> ESR03EZPJ101; MPN1 ESR03EZPJ101 -> (none)
Changed lines of the file:
@@
 F 2 "Resistor_SMD:R_0603_1608Metric" H 7550 2450 60  0001 C CNN
 F 3 "" H 7550 2450 60  0000 C CNN
-F 4 "ESR03EZPJ101" H 1000 150 50  0001 C CNN "MPN1"
+F 4 "ESR03EZPJ101" H 1000 150 50  0001 C CNN "MPN"
 F 5 "ERJ-PA3J101V" H 7550 2450 50  0001 C CNN "MPN2"
 F 6 "RCA0603100RFKEAHP" H 7550 2450 50  0001 C CNN "MPN3"
@@
 F 2 "Resistor_SMD:R_0603_1608Metric" H 7000 2350 60  0001 C CNN
 F 3 "" H 7000 2350 60  0000 C CNN
-F 4 "RMCF0603JT56R0" H 1000 150 50  0001 C CNN "MPN1"
+F 4 "RMCF0603JT56R0" H 1000 150 50  0001 C CNN "MPN"
 F 5 "ESR03EZPJ560" H 7000 2350 50  0001 C CNN "MPN2"
 F 6 "RC1608J560CS" H 7000 2350 50  0001 C CNN "MPN3"
@@
 F 2 "Capacitor_SMD:C_0603_1608Metric" H 6550 1900 60  0001 C CNN
 F 3 "" H 6550 1900 60  0000 C CNN
-F 4 "" H 1700 150 50  0001 C CNN "MPN"
-F 5 "GCM188R71C104KA37D" H 0   0   50  0001 C CNN "MPN1"
-F 6 "C0603X104K8RACTU" H 0   0   50  0001 C CNN "MPN2"
-F 7 "CS0603KRX7R7BB104" H 0   0   50  0001 C CNN "MPN3"
+F 4 "GCM188R71C104KA37D" H 0   0   50  0001 C CNN "MPN"
+F 5 "C0603X104K8RACTU" H 0   0   50  0001 C CNN "MPN2"
+F 6 "CS0603KRX7R7BB104" H 0   0   50  0001 C CNN "MPN3"
 	1    6550 1900
 	0    -1   1    0
@@
 F 2 "Package_TO_SOT_SMD:SOT-23" H 4550 2000 29  0001 C CNN
 F 3 "" H 4350 1900 60  0000 C CNN
-F 4 "" H 4350 1900 60  0001 C CNN "MPN"
-F 5 "BSS84-7-F" H 0   0   50  0001 C CNN "MPN1"
-F 6 "BSS84LT1G" H 0   0   50  0001 C CNN "MPN2"
-F 7 "DMP3099L" H 0   0   50  0001 C CNN "MPN3"
+F 4 "BSS84-7-F" H 0   0   50  0001 C CNN "MPN"
+F 5 "BSS84LT1G" H 0   0   50  0001 C CNN "MPN2"
+F 6 "DMP3099L" H 0   0   50  0001 C CNN "MPN3"
 	1    4350 1900
 	-1   0    0    1
@@
 F 2 "Resistor_SMD:R_0603_1608Metric" H 5700 2150 60  0001 C CNN
 F 3 "" H 5700 2150 60  0000 C CNN
-F 4 "" H 2450 850 50  0001 C CNN "MPN"
-F 5 "RMCF0603JT10K0" H 0   0   50  0001 C CNN "MPN1"
-F 6 "RCA060310K0JNEA" H 0   0   50  0001 C CNN "MPN2"
-F 7 "ESR03EZPJ103" H 0   0   50  0001 C CNN "MPN3"
+F 4 "RMCF0603JT10K0" H 0   0   50  0001 C CNN "MPN"
+F 5 "RCA060310K0JNEA" H 0   0   50  0001 C CNN "MPN2"
+F 6 "ESR03EZPJ103" H 0   0   50  0001 C CNN "MPN3"
 	1    5700 2150
 	1    0    0    -1
@@
 F 2 "Resistor_SMD:R_0603_1608Metric" H 5700 3350 60  0001 C CNN
 F 3 "" H 5700 3350 60  0000 C CNN
-F 4 "" H 2450 2050 50  0001 C CNN "MPN"
-F 5 "RMCF0603JT10K0" H 0   0   50  0001 C CNN "MPN1"
-F 6 "RCA060310K0JNEA" H 0   0   50  0001 C CNN "MPN2"
-F 7 "ESR03EZPJ103" H 0   0   50  0001 C CNN "MPN3"
+F 4 "RMCF0603JT10K0" H 0   0   50  0001 C CNN "MPN"
+F 5 "RCA060310K0JNEA" H 0   0   50  0001 C CNN "MPN2"
+F 6 "ESR03EZPJ103" H 0   0   50  0001 C CNN "MPN3"
 	1    5700 3350
 	1    0    0    -1
@@
 F 2 "Resistor_SMD:R_0603_1608Metric" H 6750 4800 60  0001 C CNN
 F 3 "" H 6750 4800 60  0000 C CNN
-F 4 "ESR03EZPJ221" H -3200 600 50  0001 C CNN "MPN1"
+F 4 "ESR03EZPJ221" H -3200 600 50  0001 C CNN "MPN"
 F 5 "ERJ-PB3D2200V" H 6750 4800 50  0001 C CNN "MPN2"
 F 6 "CRCW0603220RJNEAHP" H 6750 4800 50  0001 C CNN "MPN3"
@@
 F 2 "Resistor_SMD:R_0603_1608Metric" H 5500 2950 60  0001 C CNN
 F 3 "" H 5500 2950 60  0000 C CNN
-F 4 "RMCF0603JT22R0" H 1200 600 50  0001 C CNN "MPN1"
+F 4 "RMCF0603JT22R0" H 1200 600 50  0001 C CNN "MPN"
 F 5 "RC1608J220CS" V 5500 2950 50  0001 C CNN "MPN2"
 F 6 "ESR03EZPJ220" V 5500 2950 50  0001 C CNN "MPN3"
@@
 F 2 "Package_TO_SOT_SMD:SOT-23" H 4050 2900 29  0001 C CNN
 F 3 "" H 3850 2800 60  0000 C CNN
-F 4 "" H 3850 2800 60  0001 C CNN "MPN"
-F 5 "BSS84-7-F" H -500 900 50  0001 C CNN "MPN1"
-F 6 "BSS84LT1G" H -500 900 50  0001 C CNN "MPN2"
-F 7 "DMP3099L" H -500 900 50  0001 C CNN "MPN3"
+F 4 "BSS84-7-F" H -500 900 50  0001 C CNN "MPN"
+F 5 "BSS84LT1G" H -500 900 50  0001 C CNN "MPN2"
+F 6 "DMP3099L" H -500 900 50  0001 C CNN "MPN3"
 	1    3850 2800
 	-1   0    0    1
@@
 F 2 "Capacitor_SMD:C_0603_1608Metric" H 4250 2400 60  0001 C CNN
 F 3 "" H 4250 2400 60  0000 C CNN
-F 4 "CL10A106MQ8NNNC" H -1050 -2950 50  0001 C CNN "MPN1"
+F 4 "CL10A106MQ8NNNC" H -1050 -2950 50  0001 C CNN "MPN"
 F 5 "GRM188R60J106KE47D" H 4250 2400 50  0001 C CNN "MPN2"
 F 6 "CC0603MRX5R5BB106" V 4250 2400 50  0001 C CNN "MPN3"
@@
 F 2 "Capacitor_SMD:C_0603_1608Metric" H 3750 3300 60  0001 C CNN
 F 3 "" H 3750 3300 60  0000 C CNN
-F 4 "CL10A106MQ8NNNC" H -1550 -2050 50  0001 C CNN "MPN1"
+F 4 "CL10A106MQ8NNNC" H -1550 -2050 50  0001 C CNN "MPN"
 F 5 "GRM188R60J106KE47D" H 3750 3300 50  0001 C CNN "MPN2"
 F 6 "CC0603MRX5R5BB106" V 3750 3300 50  0001 C CNN "MPN3"
@@
 F 2 "Capacitor_SMD:C_0805_2012Metric" H 4600 5350 60  0001 C CNN
 F 3 "" H 4600 5350 60  0000 C CNN
-F 4 "CL21A106KOFNNNE" H -700 0   50  0001 C CNN "MPN1"
+F 4 "CL21A106KOFNNNE" H -700 0   50  0001 C CNN "MPN"
 F 5 "C2012X5R1C106M085AC" H 4600 5350 50  0001 C CNN "MPN2"
 	1    4600 5350
@@
 F 2 "Capacitor_SMD:C_0603_1608Metric" H 4950 5350 60  0001 C CNN
 F 3 "" H 4950 5350 60  0000 C CNN
-F 4 "" H 100 3600 50  0001 C CNN "MPN"
-F 5 "GCM188R71C104KA37D" H -1600 3450 50  0001 C CNN "MPN1"
-F 6 "C0603X104K8RACTU" H -1600 3450 50  0001 C CNN "MPN2"
-F 7 "CS0603KRX7R7BB104" H -1600 3450 50  0001 C CNN "MPN3"
+F 4 "GCM188R71C104KA37D" H -1600 3450 50  0001 C CNN "MPN"
+F 5 "C0603X104K8RACTU" H -1600 3450 50  0001 C CNN "MPN2"
+F 6 "CS0603KRX7R7BB104" H -1600 3450 50  0001 C CNN "MPN3"
 	1    4950 5350
 	-1   0    0    -1
@@
 F 2 "Resistor_SMD:R_0603_1608Metric" H 5550 2450 60  0001 C CNN
 F 3 "" H 5550 2450 60  0000 C CNN
-F 4 "RMCF0603JT22R0" H 1250 100 50  0001 C CNN "MPN1"
+F 4 "RMCF0603JT22R0" H 1250 100 50  0001 C CNN "MPN"
 F 5 "RC1608J220CS" V 5550 2450 50  0001 C CNN "MPN2"
 F 6 "ESR03EZPJ220" V 5550 2450 50  0001 C CNN "MPN3"
@@
 F 2 "Resistor_SMD:R_0603_1608Metric" H 6750 5400 60  0001 C CNN
 F 3 "" H 6750 5400 60  0000 C CNN
-F 4 "ESR03EZPJ221" H -3200 1200 50  0001 C CNN "MPN1"
+F 4 "ESR03EZPJ221" H -3200 1200 50  0001 C CNN "MPN"
 F 5 "ERJ-PB3D2200V" H 6750 5400 50  0001 C CNN "MPN2"
 F 6 "CRCW0603220RJNEAHP" H 6750 5400 50  0001 C CNN "MPN3"
@@
 F 2 "Resistor_SMD:R_0603_1608Metric" H 7000 2550 60  0001 C CNN
 F 3 "" H 7000 2550 60  0000 C CNN
-F 4 "RMCF0603JT56R0" H 1000 350 50  0001 C CNN "MPN1"
+F 4 "RMCF0603JT56R0" H 1000 350 50  0001 C CNN "MPN"
 F 5 "ESR03EZPJ560" H 7000 2550 50  0001 C CNN "MPN2"
 F 6 "RC1608J560CS" H 7000 2550 50  0001 C CNN "MPN3"
@@
 F 2 "Resistor_SMD:R_0603_1608Metric" H 7250 2850 60  0001 C CNN
 F 3 "" H 7250 2850 60  0000 C CNN
-F 4 "RMCF0603JT56R0" H 1250 650 50  0001 C CNN "MPN1"
+F 4 "RMCF0603JT56R0" H 1250 650 50  0001 C CNN "MPN"
 F 5 "ESR03EZPJ560" H 7250 2850 50  0001 C CNN "MPN2"
 F 6 "RC1608J560CS" H 7250 2850 50  0001 C CNN "MPN3"
@@
 F 2 "Resistor_SMD:R_0603_1608Metric" H 7250 3050 60  0001 C CNN
 F 3 "" H 7250 3050 60  0000 C CNN
-F 4 "RMCF0603JT56R0" H 1250 850 50  0001 C CNN "MPN1"
+F 4 "RMCF0603JT56R0" H 1250 850 50  0001 C CNN "MPN"
 F 5 "ESR03EZPJ560" H 7250 3050 50  0001 C CNN "MPN2"
 F 6 "RC1608J560CS" H 7250 3050 50  0001 C CNN "MPN3"

Commit message: bottom,sch: add comment field to some parts
Parts:
- J21: Comment (none) -> CONTROL CHAIN
Changed lines of the file:
@@
 F 3 "" V 6150 5125 50  0001 C CNN
 F 4 "RJHSE-5381" H 6150 5100 50  0001 C CNN "MPN"
+F 5 "CONTROL CHAIN" H 0   0   50  0001 C CNN "Comment"
 	1    6150 5100
 	-1   0    0    1
