File: hw-design/bottom-board/usb.sch (KiCad schematic (older format))
At the start: 14 parts, among them P1 USB_B, P2 USB_A, U10 RT9701

Commit message: bottom,sch: fix parts after updating to kicad 5
Parts:
- removed C50, C52: 100nF, Capacitors_SMD:C_0603, symbol C_Small
- removed D13, D14: PRTR5V0U2X, Housings_SOT-23_SOT-143_TSOT-6:SOT-143, symbol PRTR5V0U2X
- removed L2: 600R 1.5A, Capacitors_SMD:C_0805, symbol L_Small
- removed P1: USB_B, Connect:USB_B, symbol USB_B-RESCUE-bottom-board
- removed P2: USB_A, Connect:USB_A_Vertical, symbol USB_A-RESCUE-bottom-board
- added C?: 10uF, Capacitors_SMD:C_0805, symbol Device:C_Small
- added D? (x2): PRTR5V0U2X, symbol Power_Protection:PRTR5V0U2X
- added J?: USB_A, symbol Connector:USB_A
- added J?: USB_B, symbol Connector:USB_B
- added L? (x2): 60R 2A, Capacitors_SMD:C_0805, symbol Device:L_Small
- C48, C49, C51: symbol C_Small -> Device:C_Small
- R42, R43, R46: symbol R_Small -> Device:R_Small
- U10: symbol RT9701 -> Power_Management:RT9701

Commit message: bottom,sch: fix ERC issues
Parts:
- removed L? (x2): 60R 2A, Capacitors_SMD:C_0805, symbol Device:L_Small
- gave numbers to parts that had none: 5
- renumbered C49 to C62, C48 to C63, C51 to C64, R42 to R28, R43 to R29, R46 to R30, U10 to U16
Connections:
- wire segments 64 -> 62
Changed lines of the file:
@@
 $EndDescr
 $Comp
-L Device:R_Small R42
+L Device:R_Small R28
 U 1 1 5509EE84
 P 3850 2850
-F 0 "R42" H 3900 2900 50  0000 L CNN
+F 0 "R28" H 3900 2900 50  0000 L CNN
 F 1 "5k6" H 3900 2800 50  0000 L CNN
 F 2 "Resistors_SMD:R_0603" H 3850 2850 60  0001 C CNN
@@
 $EndComp
 $Comp
-L Device:R_Small R43
+L Device:R_Small R29
 U 1 1 5509EF09
 P 3850 3150
-F 0 "R43" H 3900 3200 50  0000 L CNN
+F 0 "R29" H 3900 3200 50  0000 L CNN
 F 1 "10k" H 3900 3100 50  0000 L CNN
 F 2 "Resistors_SMD:R_0603" H 3850 3150 60  0001 C CNN
@@
 $EndComp
 $Comp
-L Device:C_Small C48
+L Device:C_Small C63
 U 1 1 5509EF6F
 P 4100 3150
-F 0 "C48" H 3900 3150 50  0000 L CNN
+F 0 "C63" H 3900 3150 50  0000 L CNN
 F 1 "100nF" H 3850 3050 50  0000 L CNN
 F 2 "Capacitors_SMD:C_0603" H 4100 3150 60  0001 C CNN
@@
 $EndComp
 $Comp
-L power:GNDD #PWR0126
+L power:GNDD #PWR0163
 U 1 1 5509F619
 P 3850 3350
-F 0 "#PWR0126" H 3850 3100 50  0001 C CNN
+F 0 "#PWR0163" H 3850 3100 50  0001 C CNN
 F 1 "GNDD" H 3850 3200 50  0000 C CNN
 F 2 "" H 3850 3350 60  0000 C CNN
@@
 $EndComp
 $Comp
-L Power_Management:RT9701 U10
+L Power_Management:RT9701 U16
 U 1 1 55080DFB
 P 7575 3200
-F 0 "U10" H 7775 3450 50  0000 C CNN
+F 0 "U16" H 7775 3450 50  0000 C CNN
 F 1 "RT9701" H 7775 3050 50  0000 C CNN
 F 2 "Housings_SOT-23_SOT-143_TSOT-6:SOT-23-5" H 7575 3200 60  0001 C CNN
@@
 $EndComp
 $Comp
-L Device:R_Small R46
+L Device:R_Small R30
 U 1 1 55083C10
 P 6925 3450
-F 0 "R46" H 6975 3500 50  0000 L CNN
+F 0 "R30" H 6975 3500 50  0000 L CNN
 F 1 "10k" H 6975 3400 50  0000 L CNN
 F 2 "Resistors_SMD:R_0603" H 6925 3450 60  0001 C CNN
@@
 $EndComp
 $Comp
-L power:GNDD #PWR0130
+L power:GNDD #PWR0166
 U 1 1 55084544
 P 7575 3650
-F 0 "#PWR0130" H 7575 3400 50  0001 C CNN
+F 0 "#PWR0166" H 7575 3400 50  0001 C CNN
 F 1 "GNDD" H 7575 3500 50  0000 C CNN
 F 2 "" H 7575 3650 60  0000 C CNN
@@
 $EndComp
 $Comp
-L power:GNDD #PWR0132
+L power:GNDD #PWR0165
 U 1 1 5508613A
 P 7475 2800
-F 0 "#PWR0132" H 7475 2550 50  0001 C CNN
+F 0 "#PWR0165" H 7475 2550 50  0001 C CNN
 F 1 "GNDD" H 7475 2650 50  0000 C CNN
 F 2 "" H 7475 2800 60  0000 C CNN
@@
 $EndComp
 $Comp
-L Device:C_Small C51
+L Device:C_Small C64
 U 1 1 55085190
 P 7225 2750
-F 0 "C51" H 7325 2750 50  0000 L CNN
+F 0 "C64" H 7325 2750 50  0000 L CNN
 F 1 "100nF" H 7275 2650 50  0000 L CNN
 F 2 "Capacitors_SMD:C_0603" H 7225 2750 60  0001 C CNN
@@
 $EndComp
 $Comp
-L Device:C_Small C49
+L Device:C_Small C62
 U 1 1 551A8035
 P 3600 3000
-F 0 "C49" H 3700 3050 50  0000 L CNN
+F 0 "C62" H 3700 3050 50  0000 L CNN
 F 1 "10uF" H 3700 2950 50  0000 L CNN
 F 2 "Capacitors_SMD:C_0805" H 3600 3000 60  0001 C CNN
@@
 	3850 2700 3600 2700
 $Comp
-L power:+5VD #PWR0277
+L power:+5VD #PWR0164
 U 1 1 5B50357D
 P 6975 2650
-F 0 "#PWR0277" H 6975 2500 50  0001 C CNN
+F 0 "#PWR0164" H 6975 2500 50  0001 C CNN
 F 1 "+5VD" H 6975 2790 50  0000 C CNN
 F 2 "" H 6975 2650 50  0001 C CNN
@@
 	3850 3000 3850 3050
 $Comp
-L Power_Protection:PRTR5V0U2X D?
+L Power_Protection:PRTR5V0U2X D9
 U 1 1 5B808699
 P 3150 3750
-F 0 "D?" H 2900 4175 50  0000 L CNN
+F 0 "D9" H 2900 4175 50  0000 L CNN
 F 1 "PRTR5V0U2X" H 2525 4100 50  0000 L CNN
 F 2 "" H 3210 3750 50  0001 C CNN
@@
 $EndComp
 $Comp
-L Connector:USB_A J?
+L Connector:USB_A J20
 U 1 1 5B809B95
 P 10050 3300
-F 0 "J?" H 10050 3725 50  0000 C CNN
+F 0 "J20" H 10050 3725 50  0000 C CNN
 F 1 "USB_A" H 10050 3650 50  0000 C CNN
 F 2 "" H 10200 3250 50  0001 C CNN
@@
 $EndComp
 $Comp
-L Connector:USB_B J?
+L Connector:USB_B J19
 U 1 1 5B809C8F
 P 2100 2900
-F 0 "J?" H 2100 3325 50  0000 C CNN
+F 0 "J19" H 2100 3325 50  0000 C CNN
 F 1 "USB_B" H 2100 3250 50  0000 C CNN
 F 2 "" H 2250 2850 50  0001 C CNN
@@
 Wire Wire Line
 	2500 3000 2400 3000
-$Comp
-L Device:L_Small L?
-U 1 1 5B81585F
-P 2000 3450
-F 0 "L?" H 2050 3500 50  0000 L CNN
-F 1 "60R 2A" H 2050 3400 50  0000 L CNN
-F 2 "Capacitors_SMD:C_0805" H 2000 3450 60  0001 C CNN
-F 3 "" H 2000 3450 60  0000 C CNN
-F 4 "BKP1608HS600-T" H -1850 500 50  0001 C CNN "MPN"
-	1    2000 3450
-	-1   0    0    -1
-$EndComp
-Wire Wire Line
-	2000 3300 2000 3350
-$Comp
-L power:GNDD #PWR?
-U 1 1 5B817FD8
-P 2000 3700
-F 0 "#PWR?" H 2000 3450 50  0001 C CNN
-F 1 "GNDD" H 2000 3550 50  0000 C CNN
-F 2 "" H 2000 3700 60  0000 C CNN
-F 3 "" H 2000 3700 60  0000 C CNN
-	1    2000 3700
-	1    0    0    -1
-$EndComp
-Wire Wire Line
-	2000 3550 2000 3625
-Wire Wire Line
-	2100 3300 2100 3625
-Wire Wire Line
-	2100 3625 2000 3625
-Connection ~ 2000 3625
-Wire Wire Line
-	2000 3625 2000 3700
 Text GLabel 3700 3825 3    50   BiDi ~ 0
 USB_DEV_DP
@@
 	3150 2700 2400 2700
 $Comp
-L power:GNDD #PWR?
+L power:GNDD #PWR0162
 U 1 1 5B84273E
 P 3150 4300
-F 0 "#PWR?" H 3150 4050 50  0001 C CNN
+F 0 "#PWR0162" H 3150 4050 50  0001 C CNN
 F 1 "GNDD" H 3150 4150 50  0000 C CNN
 F 2 "" H 3150 4300 60  0000 C CNN
@@
 	9650 3400 9750 3400
 $Comp
-L Device:L_Small L?
-U 1 1 5B875C4C
-P 10150 3850
-F 0 "L?" H 10200 3900 50  0000 L CNN
-F 1 "60R 2A" H 10200 3800 50  0000 L CNN
-F 2 "Capacitors_SMD:C_0805" H 10150 3850 60  0001 C CNN
-F 3 "" H 10150 3850 60  0000 C CNN
-F 4 "BKP1608HS600-T" H 6300 900 50  0001 C CNN "MPN"
-	1    10150 3850
-	1    0    0    -1
-$EndComp
-Wire Wire Line
-	10150 3700 10150 3750
-$Comp
-L power:GNDD #PWR?
+L power:GNDD #PWR0169
 U 1 1 5B875C53
-P 10150 4100
-F 0 "#PWR?" H 10150 3850 50  0001 C CNN
-F 1 "GNDD" H 10150 3950 50  0000 C CNN
-F 2 "" H 10150 4100 60  0000 C CNN
-F 3 "" H 10150 4100 60  0000 C CNN
-	1    10150 4100
-	-1   0    0    -1
-$EndComp
-Wire Wire Line
-	10150 3950 10150 4025
-Wire Wire Line
-	10050 3700 10050 4025
-Wire Wire Line
-	10050 4025 10150 4025
-Connection ~ 10150 4025
-Wire Wire Line
-	10150 4025 10150 4100
+P 10050 3850
+F 0 "#PWR0169" H 10050 3600 50  0001 C CNN
+F 1 "GNDD" H 10050 3700 50  0000 C CNN
+F 2 "" H 10050 3850 60  0000 C CNN
+F 3 "" H 10050 3850 60  0000 C CNN
+	1    10050 3850
+	1    0    0    -1
+$EndComp
+Wire Wire Line
+	10050 3700 10050 3775
 Wire Wire Line
 	8625 3250 8625 3100
@@
 	8075 3750 8125 3750
 $Comp
-L power:GNDD #PWR?
+L power:GNDD #PWR0167
 U 1 1 5B8A007B
 P 8625 4300
-F 0 "#PWR?" H 8625 4050 50  0001 C CNN
+F 0 "#PWR0167" H 8625 4050 50  0001 C CNN
 F 1 "GNDD" H 8625 4150 50  0000 C CNN
 F 2 "" H 8625 4300 60  0000 C CNN
@@
 	8625 4250 8625 4300
 $Comp
-L Power_Protection:PRTR5V0U2X D?
+L Power_Protection:PRTR5V0U2X D10
 U 1 1 5B87078C
 P 8625 3750
-F 0 "D?" H 8375 4175 50  0000 L CNN
+F 0 "D10" H 8375 4175 50  0000 L CNN
 F 1 "PRTR5V0U2X" H 8000 4100 50  0000 L CNN
 F 2 "" H 8685 3750 50  0001 C CNN
@@
 	8175 3100 8625 3100
 $Comp
-L Device:C_Small C?
+L Device:C_Small C65
 U 1 1 5B8AF2FD
 P 8625 2875
-F 0 "C?" H 8725 2925 50  0000 L CNN
+F 0 "C65" H 8725 2925 50  0000 L CNN
 F 1 "10uF" H 8725 2825 50  0000 L CNN
 F 2 "Capacitors_SMD:C_0805" H 8625 2875 60  0001 C CNN
@@
 	8625 2975 8625 3100
 $Comp
-L power:GNDD #PWR?
+L power:GNDD #PWR0168
 U 1 1 5B8B4553
 P 8900 2800
-F 0 "#PWR?" H 8900 2550 50  0001 C CNN
+F 0 "#PWR0168" H 8900 2550 50  0001 C CNN
 F 1 "GNDD" H 8900 2650 50  0000 C CNN
 F 2 "" H 8900 2800 60  0000 C CNN
@@
 Wire Wire Line
 	8625 2725 8900 2725
+Wire Wire Line
+	10150 3700 10150 3775
+Wire Wire Line
+	10150 3775 10050 3775
+Connection ~ 10050 3775
+Wire Wire Line
+	10050 3775 10050 3850
+$Comp
+L power:GNDD #PWR0161
+U 1 1 5B686921
+P 2100 3450
+F 0 "#PWR0161" H 2100 3200 50  0001 C CNN
+F 1 "GNDD" H 2100 3300 50  0000 C CNN
+F 2 "" H 2100 3450 60  0000 C CNN
+F 3 "" H 2100 3450 60  0000 C CNN
+	1    2100 3450
+	-1   0    0    -1
+$EndComp
+Wire Wire Line
+	2100 3300 2100 3375
+Wire Wire Line
+	2000 3300 2000 3375
+Wire Wire Line
+	2000 3375 2100 3375
+Connection ~ 2100 3375
+Wire Wire Line
+	2100 3375 2100 3450
 $EndSCHEMATC

Commit message: bottom,sch: MPN updated on usb sheet
Parts:
- removed C62, C65: 10uF, Capacitors_SMD:C_0805, symbol Device:C_Small
- removed D10: PRTR5V0U2X, symbol Power_Protection:PRTR5V0U2X
- removed R28: 5k6, Resistors_SMD:R_0603, symbol Device:R_Small
- added C? (x2): 10uF, Capacitor_SMD:C_0603_1608Metric, symbol Device:C_Small
- added D?: PRTR5V0U2X, Package_TO_SOT_SMD:SOT-143, symbol Power_Protection:PRTR5V0U2X
- added R?: 5k6, Resistors_SMD:R_0603, symbol Device:R_Small
- C63, C64: MPN C1608X7R1E104K080AA -> (none); MPN1 (none) -> GCM188R71C104KA37D; MPN2 (none) -> C0603X104K8RACTU; MPN3 (none) -> CS0603KRX7R7BB104
- D9: footprint (none) -> Package_TO_SOT_SMD:SOT-143; MPN (none) -> PRTR5V0U2X,215
- J19: MPN (none) -> 61729-1011BLF
- J20: MPN (none) -> 73725-0110BLF
- R29, R30: MPN RMCF0603JT10K0 -> (none); MPN1 (none) -> RMCF0603JT10K0; MPN2 (none) -> RCA060310K0JNEA; MPN3 (none) -> ESR03EZPJ103
Changed lines of the file:
@@
 $EndDescr
-$Comp
-L Device:R_Small R28
-U 1 1 5509EE84
-P 3850 2850
-F 0 "R28" H 3900 2900 50  0000 L CNN
-F 1 "5k6" H 3900 2800 50  0000 L CNN
-F 2 "Resistors_SMD:R_0603" H 3850 2850 60  0001 C CNN
-F 3 "" H 3850 2850 60  0000 C CNN
-F 4 "RMCF0603JT5K60" H 1650 -550 50  0001 C CNN "MPN"
-	1    3850 2850
-	-1   0    0    -1
-$EndComp
 $Comp
 L Device:R_Small R29
@@
 F 2 "Resistors_SMD:R_0603" H 3850 3150 60  0001 C CNN
 F 3 "" H 3850 3150 60  0000 C CNN
-F 4 "RMCF0603JT10K0" H 1650 -550 50  0001 C CNN "MPN"
+F 4 "" H 1650 -550 50  0001 C CNN "MPN"
+F 5 "RMCF0603JT10K0" H 0   0   50  0001 C CNN "MPN1"
+F 6 "RCA060310K0JNEA" H 0   0   50  0001 C CNN "MPN2"
+F 7 "ESR03EZPJ103" H 0   0   50  0001 C CNN "MPN3"
 	1    3850 3150
 	-1   0    0    -1
@@
 U 1 1 5509EF6F
 P 4100 3150
-F 0 "C63" H 3900 3150 50  0000 L CNN
-F 1 "100nF" H 3850 3050 50  0000 L CNN
+F 0 "C63" H 4025 3150 50  0000 R CNN
+F 1 "100nF" H 4025 3075 50  0000 R CNN
 F 2 "Capacitors_SMD:C_0603" H 4100 3150 60  0001 C CNN
 F 3 "" H 4100 3150 60  0000 C CNN
-F 4 "C1608X7R1E104K080AA" H 2150 -550 50  0001 C CNN "MPN"
+F 4 "" H 2150 -550 50  0001 C CNN "MPN"
+F 5 "GCM188R71C104KA37D" H 0   0   50  0001 C CNN "MPN1"
+F 6 "C0603X104K8RACTU" H 0   0   50  0001 C CNN "MPN2"
+F 7 "CS0603KRX7R7BB104" H 0   0   50  0001 C CNN "MPN3"
 	1    4100 3150
 	-1   0    0    -1
@@
 F 2 "Resistors_SMD:R_0603" H 6925 3450 60  0001 C CNN
 F 3 "" H 6925 3450 60  0000 C CNN
-F 4 "RMCF0603JT10K0" H -25 -350 50  0001 C CNN "MPN"
+F 4 "" H -25 -350 50  0001 C CNN "MPN"
+F 5 "RMCF0603JT10K0" H 0   0   50  0001 C CNN "MPN1"
+F 6 "RCA060310K0JNEA" H 0   0   50  0001 C CNN "MPN2"
+F 7 "ESR03EZPJ103" H 0   0   50  0001 C CNN "MPN3"
 	1    6925 3450
 	1    0    0    -1
@@
 F 2 "Capacitors_SMD:C_0603" H 7225 2750 60  0001 C CNN
 F 3 "" H 7225 2750 60  0000 C CNN
-F 4 "C1608X7R1E104K080AA" H -25 -350 50  0001 C CNN "MPN"
+F 4 "" H -25 -350 50  0001 C CNN "MPN"
+F 5 "GCM188R71C104KA37D" H 0   0   50  0001 C CNN "MPN1"
+F 6 "C0603X104K8RACTU" H 0   0   50  0001 C CNN "MPN2"
+F 7 "CS0603KRX7R7BB104" H 0   0   50  0001 C CNN "MPN3"
 	1    7225 2750
 	0    -1   -1   0
-$EndComp
-$Comp
-L Device:C_Small C62
-U 1 1 551A8035
-P 3600 3000
-F 0 "C62" H 3700 3050 50  0000 L CNN
-F 1 "10uF" H 3700 2950 50  0000 L CNN
-F 2 "Capacitors_SMD:C_0805" H 3600 3000 60  0001 C CNN
-F 3 "" H 3600 3000 60  0000 C CNN
-F 4 "GRM219R61E106KA12D" H -1700 -2350 50  0001 C CNN "MPN"
-	1    3600 3000
-	-1   0    0    -1
 $EndComp
 Text GLabel 4300 3000 2    50   Output ~ 0
@@
 F 0 "D9" H 2900 4175 50  0000 L CNN
 F 1 "PRTR5V0U2X" H 2525 4100 50  0000 L CNN
-F 2 "" H 3210 3750 50  0001 C CNN
+F 2 "Package_TO_SOT_SMD:SOT-143" H 3210 3750 50  0001 C CNN
 F 3 "https://assets.nexperia.com/documents/data-sheet/PRTR5V0U2X.pdf" H 3210 3750 50  0001 C CNN
+F 4 "PRTR5V0U2X,215" H 3150 3750 50  0001 C CNN "MPN"
 	1    3150 3750
 	1    0    0    -1
@@
 F 2 "" H 10200 3250 50  0001 C CNN
 F 3 " ~" H 10200 3250 50  0001 C CNN
+F 4 "73725-0110BLF" H 10050 3300 50  0001 C CNN "MPN"
 	1    10050 3300
 	-1   0    0    -1
@@
 F 2 "" H 2250 2850 50  0001 C CNN
 F 3 " ~" H 2250 2850 50  0001 C CNN
+F 4 "61729-1011BLF" H 2100 2900 50  0001 C CNN "MPN"
 	1    2100 2900
 	1    0    0    -1
@@
 Wire Wire Line
 	8625 4250 8625 4300
-$Comp
-L Power_Protection:PRTR5V0U2X D10
-U 1 1 5B87078C
-P 8625 3750
-F 0 "D10" H 8375 4175 50  0000 L CNN
-F 1 "PRTR5V0U2X" H 8000 4100 50  0000 L CNN
-F 2 "" H 8685 3750 50  0001 C CNN
-F 3 "https://assets.nexperia.com/documents/data-sheet/PRTR5V0U2X.pdf" H 8685 3750 50  0001 C CNN
-	1    8625 3750
-	1    0    0    -1
-$EndComp
 Connection ~ 8625 3100
 Wire Wire Line
@@
 Wire Wire Line
 	8175 3100 8625 3100
-$Comp
-L Device:C_Small C65
-U 1 1 5B8AF2FD
-P 8625 2875
-F 0 "C65" H 8725 2925 50  0000 L CNN
-F 1 "10uF" H 8725 2825 50  0000 L CNN
-F 2 "Capacitors_SMD:C_0805" H 8625 2875 60  0001 C CNN
-F 3 "" H 8625 2875 60  0000 C CNN
-F 4 "GRM219R61E106KA12D" H 3325 -2475 50  0001 C CNN "MPN"
-	1    8625 2875
-	-1   0    0    -1
-$EndComp
 Wire Wire Line
 	8625 2975 8625 3100
@@
 Wire Wire Line
 	2100 3375 2100 3450
+$Comp
+L Device:R_Small R?
+U 1 1 5B845377
+P 3850 2850
+AR Path="/54F72FB4/5B845377" Ref="R?"  Part="1"
+AR Path="/54F72FB2/5B845377" Ref="R?"  Part="1"
+F 0 "R?" H 3900 2900 50  0000 L CNN
+F 1 "5k6" H 3900 2800 50  0000 L CNN
+F 2 "Resistors_SMD:R_0603" H 3850 2850 60  0001 C CNN
+F 3 "" H 3850 2850 60  0000 C CNN
+F 4 "RMCF0603JT5K60" H -550 -700 50  0001 C CNN "MPN1"
+F 5 "RC0603JR-075K6L" H 3850 2850 50  0001 C CNN "MPN2"
+F 6 "ESR03EZPJ562" H 3850 2850 50  0001 C CNN "MPN3"
+	1    3850 2850
+	-1   0    0    1
+$EndComp
+$Comp
+L Device:C_Small C?
+U 1 1 5B847993
+P 3600 3000
+AR Path="/54F7244B/5B847993" Ref="C?"  Part="1"
+AR Path="/54F725AE/5B847993" Ref="C?"  Part="1"
+AR Path="/54F72B97/5B847993" Ref="C?"  Part="1"
+AR Path="/54F72FB2/5B847993" Ref="C?"  Part="1"
+F 0 "C?" H 3675 3075 50  0000 L CNN
+F 1 "10uF" H 3675 3000 50  0000 L CNN
+F 2 "Capacitor_SMD:C_0603_1608Metric" H 3600 3000 60  0001 C CNN
+F 3 "" H 3600 3000 60  0000 C CNN
+F 4 "CL10A106MQ8NNNC" H -1700 -2350 50  0001 C CNN "MPN1"
+F 5 "GRM188R60J106KE47D" H 3600 3000 50  0001 C CNN "MPN2"
+F 6 "CC0603MRX5R5BB106" V 3600 3000 50  0001 C CNN "MPN3"
+	1    3600 3000
+	-1   0    0    -1
+$EndComp
+$Comp
+L Device:C_Small C?
+U 1 1 5B849472
+P 8625 2875
+AR Path="/54F7244B/5B849472" Ref="C?"  Part="1"
+AR Path="/54F725AE/5B849472" Ref="C?"  Part="1"
+AR Path="/54F72B97/5B849472" Ref="C?"  Part="1"
+AR Path="/54F72FB2/5B849472" Ref="C?"  Part="1"
+F 0 "C?" H 8700 2950 50  0000 L CNN
+F 1 "10uF" H 8700 2875 50  0000 L CNN
+F 2 "Capacitor_SMD:C_0603_1608Metric" H 8625 2875 60  0001 C CNN
+F 3 "" H 8625 2875 60  0000 C CNN
+F 4 "CL10A106MQ8NNNC" H 3325 -2475 50  0001 C CNN "MPN1"
+F 5 "GRM188R60J106KE47D" H 8625 2875 50  0001 C CNN "MPN2"
+F 6 "CC0603MRX5R5BB106" V 8625 2875 50  0001 C CNN "MPN3"
+	1    8625 2875
+	-1   0    0    -1
+$EndComp
+$Comp
+L Power_Protection:PRTR5V0U2X D?
+U 1 1 5B849CE3
+P 8625 3750
+F 0 "D?" H 8375 4175 50  0000 L CNN
+F 1 "PRTR5V0U2X" H 8000 4100 50  0000 L CNN
+F 2 "Package_TO_SOT_SMD:SOT-143" H 8685 3750 50  0001 C CNN
+F 3 "https://assets.nexperia.com/documents/data-sheet/PRTR5V0U2X.pdf" H 8685 3750 50  0001 C CNN
+F 4 "PRTR5V0U2X,215" H 8625 3750 50  0001 C CNN "MPN"
+	1    8625 3750
+	1    0    0    -1
+$EndComp
 $EndSCHEMATC

Commit message: bottom,sch: fix/update footprints field
Parts:
- C64: renamed from C63; footprint Capacitors_SMD:C_0603 -> Capacitor_SMD:C_0603_1608Metric
- C65: renamed from C64; footprint Capacitors_SMD:C_0603 -> Capacitor_SMD:C_0603_1608Metric
- R29: renamed from R?; footprint Resistors_SMD:R_0603 -> Resistor_SMD:R_0603_1608Metric
- R30: renamed from R29; footprint Resistors_SMD:R_0603 -> Resistor_SMD:R_0603_1608Metric
- R31: renamed from R30; footprint Resistors_SMD:R_0603 -> Resistor_SMD:R_0603_1608Metric
- U16: value RT9701 -> RT9742; footprint Housings_SOT-23_SOT-143_TSOT-6:SOT-23-5 -> Package_TO_SOT_SMD:TSOT-23-5; MPN RT9701GB -> RT9742MNGJ5
- gave numbers to parts that had none: 3
Changed lines of the file:
@@
 $EndDescr
 $Comp
-L Device:R_Small R29
+L Device:R_Small R30
 U 1 1 5509EF09
 P 3850 3150
-F 0 "R29" H 3900 3200 50  0000 L CNN
+F 0 "R30" H 3900 3200 50  0000 L CNN
 F 1 "10k" H 3900 3100 50  0000 L CNN
-F 2 "Resistors_SMD:R_0603" H 3850 3150 60  0001 C CNN
+F 2 "Resistor_SMD:R_0603_1608Metric" H 3850 3150 60  0001 C CNN
 F 3 "" H 3850 3150 60  0000 C CNN
 F 4 "" H 1650 -550 50  0001 C CNN "MPN"
@@
 $EndComp
 $Comp
-L Device:C_Small C63
+L Device:C_Small C64
 U 1 1 5509EF6F
 P 4100 3150
-F 0 "C63" H 4025 3150 50  0000 R CNN
+F 0 "C64" H 4025 3150 50  0000 R CNN
 F 1 "100nF" H 4025 3075 50  0000 R CNN
-F 2 "Capacitors_SMD:C_0603" H 4100 3150 60  0001 C CNN
+F 2 "Capacitor_SMD:C_0603_1608Metric" H 4100 3150 60  0001 C CNN
 F 3 "" H 4100 3150 60  0000 C CNN
 F 4 "" H 2150 -550 50  0001 C CNN "MPN"
@@
 $EndComp
 $Comp
-L power:GNDD #PWR0163
+L power:GNDD #PWR0166
 U 1 1 5509F619
 P 3850 3350
-F 0 "#PWR0163" H 3850 3100 50  0001 C CNN
+F 0 "#PWR0166" H 3850 3100 50  0001 C CNN
 F 1 "GNDD" H 3850 3200 50  0000 C CNN
 F 2 "" H 3850 3350 60  0000 C CNN
@@
 P 7575 3200
 F 0 "U16" H 7775 3450 50  0000 C CNN
-F 1 "RT9701" H 7775 3050 50  0000 C CNN
-F 2 "Housings_SOT-23_SOT-143_TSOT-6:SOT-23-5" H 7575 3200 60  0001 C CNN
+F 1 "RT9742" H 7775 3050 50  0000 C CNN
+F 2 "Package_TO_SOT_SMD:TSOT-23-5" H 7575 3200 60  0001 C CNN
 F 3 "" H 7575 3200 60  0000 C CNN
-F 4 "RT9701GB" H -25 -350 50  0001 C CNN "MPN"
+F 4 "RT9742MNGJ5" H -25 -350 50  0001 C CNN "MPN"
 	1    7575 3200
 	1    0    0    -1
 $EndComp
 $Comp
-L Device:R_Small R30
+L Device:R_Small R31
 U 1 1 55083C10
 P 6925 3450
-F 0 "R30" H 6975 3500 50  0000 L CNN
+F 0 "R31" H 6975 3500 50  0000 L CNN
 F 1 "10k" H 6975 3400 50  0000 L CNN
-F 2 "Resistors_SMD:R_0603" H 6925 3450 60  0001 C CNN
+F 2 "Resistor_SMD:R_0603_1608Metric" H 6925 3450 60  0001 C CNN
 F 3 "" H 6925 3450 60  0000 C CNN
 F 4 "" H -25 -350 50  0001 C CNN "MPN"
@@
 $EndComp
 $Comp
-L power:GNDD #PWR0166
+L power:GNDD #PWR0169
 U 1 1 55084544
 P 7575 3650
-F 0 "#PWR0166" H 7575 3400 50  0001 C CNN
+F 0 "#PWR0169" H 7575 3400 50  0001 C CNN
 F 1 "GNDD" H 7575 3500 50  0000 C CNN
 F 2 "" H 7575 3650 60  0000 C CNN
@@
 $EndComp
 $Comp
-L power:GNDD #PWR0165
+L power:GNDD #PWR0168
 U 1 1 5508613A
 P 7475 2800
-F 0 "#PWR0165" H 7475 2550 50  0001 C CNN
+F 0 "#PWR0168" H 7475 2550 50  0001 C CNN
 F 1 "GNDD" H 7475 2650 50  0000 C CNN
 F 2 "" H 7475 2800 60  0000 C CNN
@@
 $EndComp
 $Comp
-L Device:C_Small C64
+L Device:C_Small C65
 U 1 1 55085190
 P 7225 2750
-F 0 "C64" H 7325 2750 50  0000 L CNN
+F 0 "C65" H 7325 2750 50  0000 L CNN
 F 1 "100nF" H 7275 2650 50  0000 L CNN
-F 2 "Capacitors_SMD:C_0603" H 7225 2750 60  0001 C CNN
+F 2 "Capacitor_SMD:C_0603_1608Metric" H 7225 2750 60  0001 C CNN
 F 3 "" H 7225 2750 60  0000 C CNN
 F 4 "" H -25 -350 50  0001 C CNN "MPN"
@@
 	3850 2700 3600 2700
 $Comp
-L power:+5VD #PWR0164
+L power:+5VD #PWR0167
 U 1 1 5B50357D
 P 6975 2650
-F 0 "#PWR0164" H 6975 2500 50  0001 C CNN
+F 0 "#PWR0167" H 6975 2500 50  0001 C CNN
 F 1 "+5VD" H 6975 2790 50  0000 C CNN
 F 2 "" H 6975 2650 50  0001 C CNN
@@
 	3150 2700 2400 2700
 $Comp
-L power:GNDD #PWR0162
+L power:GNDD #PWR0165
 U 1 1 5B84273E
 P 3150 4300
-F 0 "#PWR0162" H 3150 4050 50  0001 C CNN
+F 0 "#PWR0165" H 3150 4050 50  0001 C CNN
 F 1 "GNDD" H 3150 4150 50  0000 C CNN
 F 2 "" H 3150 4300 60  0000 C CNN
@@
 	9650 3400 9750 3400
 $Comp
-L power:GNDD #PWR0169
+L power:GNDD #PWR0172
 U 1 1 5B875C53
 P 10050 3850
-F 0 "#PWR0169" H 10050 3600 50  0001 C CNN
+F 0 "#PWR0172" H 10050 3600 50  0001 C CNN
 F 1 "GNDD" H 10050 3700 50  0000 C CNN
 F 2 "" H 10050 3850 60  0000 C CNN
@@
 	8075 3750 8125 3750
 $Comp
-L power:GNDD #PWR0167
+L power:GNDD #PWR0170
 U 1 1 5B8A007B
 P 8625 4300
-F 0 "#PWR0167" H 8625 4050 50  0001 C CNN
+F 0 "#PWR0170" H 8625 4050 50  0001 C CNN
 F 1 "GNDD" H 8625 4150 50  0000 C CNN
 F 2 "" H 8625 4300 60  0000 C CNN
@@
 	8625 2975 8625 3100
 $Comp
-L power:GNDD #PWR0168
+L power:GNDD #PWR0171
 U 1 1 5B8B4553
 P 8900 2800
-F 0 "#PWR0168" H 8900 2550 50  0001 C CNN
+F 0 "#PWR0171" H 8900 2550 50  0001 C CNN
 F 1 "GNDD" H 8900 2650 50  0000 C CNN
 F 2 "" H 8900 2800 60  0000 C CNN
@@
 	10050 3775 10050 3850
 $Comp
-L power:GNDD #PWR0161
+L power:GNDD #PWR0164
 U 1 1 5B686921
 P 2100 3450
-F 0 "#PWR0161" H 2100 3200 50  0001 C CNN
+F 0 "#PWR0164" H 2100 3200 50  0001 C CNN
 F 1 "GNDD" H 2100 3300 50  0000 C CNN
 F 2 "" H 2100 3450 60  0000 C CNN
@@
 P 3850 2850
 AR Path="/54F72FB4/5B845377" Ref="R?"  Part="1"
-AR Path="/54F72FB2/5B845377" Ref="R?"  Part="1"
-F 0 "R?" H 3900 2900 50  0000 L CNN
+AR Path="/54F72FB2/5B845377" Ref="R29"  Part="1"
+F 0 "R29" H 3900 2900 50  0000 L CNN
 F 1 "5k6" H 3900 2800 50  0000 L CNN
-F 2 "Resistors_SMD:R_0603" H 3850 2850 60  0001 C CNN
+F 2 "Resistor_SMD:R_0603_1608Metric" H 3850 2850 60  0001 C CNN
 F 3 "" H 3850 2850 60  0000 C CNN
 F 4 "RMCF0603JT5K60" H -550 -700 50  0001 C CNN "MPN1"
@@
 AR Path="/54F725AE/5B847993" Ref="C?"  Part="1"
 AR Path="/54F72B97/5B847993" Ref="C?"  Part="1"
-AR Path="/54F72FB2/5B847993" Ref="C?"  Part="1"
-F 0 "C?" H 3675 3075 50  0000 L CNN
+AR Path="/54F72FB2/5B847993" Ref="C63"  Part="1"
+F 0 "C63" H 3675 3075 50  0000 L CNN
 F 1 "10uF" H 3675 3000 50  0000 L CNN
 F 2 "Capacitor_SMD:C_0603_1608Metric" H 3600 3000 60  0001 C CNN
@@
 AR Path="/54F725AE/5B849472" Ref="C?"  Part="1"
 AR Path="/54F72B97/5B849472" Ref="C?"  Part="1"
-AR Path="/54F72FB2/5B849472" Ref="C?"  Part="1"
-F 0 "C?" H 8700 2950 50  0000 L CNN
+AR Path="/54F72FB2/5B849472" Ref="C66"  Part="1"
+F 0 "C66" H 8700 2950 50  0000 L CNN
 F 1 "10uF" H 8700 2875 50  0000 L CNN
 F 2 "Capacitor_SMD:C_0603_1608Metric" H 8625 2875 60  0001 C CNN
@@
 $EndComp
 $Comp
-L Power_Protection:PRTR5V0U2X D?
+L Power_Protection:PRTR5V0U2X D10
 U 1 1 5B849CE3
 P 8625 3750
-F 0 "D?" H 8375 4175 50  0000 L CNN
+F 0 "D10" H 8375 4175 50  0000 L CNN
 F 1 "PRTR5V0U2X" H 8000 4100 50  0000 L CNN
 F 2 "Package_TO_SOT_SMD:SOT-143" H 8685 3750 50  0001 C CNN
