File: hw-design/bottom-board/usb.sch (KiCad schematic (older format))
At the start: 12 parts, among them J19 USB_B, J20 USB_A, U16 RT9742

Commit message: bottom,sch: update missing footprint fields
Parts:
- J19: footprint (none) -> Connector_USB:USB_B_OST_USB-B1HSxx_Horizontal
- J20: footprint (none) -> footprints:USB_A_Vertical
Changed lines of the file:
@@
 F 0 "J20" H 10050 3725 50  0000 C CNN
 F 1 "USB_A" H 10050 3650 50  0000 C CNN
-F 2 "" H 10200 3250 50  0001 C CNN
-F 3 " ~" H 10200 3250 50  0001 C CNN
+F 2 "footprints:USB_A_Vertical" H 10200 3250 50  0001 C CNN
+F 3 "" H 10200 3250 50  0001 C CNN
 F 4 "73725-0110BLF" H 10050 3300 50  0001 C CNN "MPN"
 	1    10050 3300
@@
 F 0 "J19" H 2100 3325 50  0000 C CNN
 F 1 "USB_B" H 2100 3250 50  0000 C CNN
-F 2 "" H 2250 2850 50  0001 C CNN
-F 3 " ~" H 2250 2850 50  0001 C CNN
+F 2 "Connector_USB:USB_B_OST_USB-B1HSxx_Horizontal" H 2250 2850 50  0001 C CNN
+F 3 "" H 2250 2850 50  0001 C CNN
 F 4 "61729-1011BLF" H 2100 2900 50  0001 C CNN "MPN"
 	1    2100 2900

Commit message: bottom,sch: rename MPN1 to MPN
Parts:
- C63, C66: MPN (none) -> CL10A106MQ8NNNC; MPN1 CL10A106MQ8NNNC -> (none)
- C64, C65: MPN (none) -> GCM188R71C104KA37D; MPN1 GCM188R71C104KA37D -> (none)
- R29: MPN (none) -> RMCF0603JT5K60; MPN1 RMCF0603JT5K60 -> (none)
- R30, R31: MPN (none) -> RMCF0603JT10K0; MPN1 RMCF0603JT10K0 -> (none)
Changed lines of the file:
@@
 F 2 "Resistor_SMD:R_0603_1608Metric" H 3850 3150 60  0001 C CNN
 F 3 "" H 3850 3150 60  0000 C CNN
-F 4 "" H 1650 -550 50  0001 C CNN "MPN"
-F 5 "RMCF0603JT10K0" H 0   0   50  0001 C CNN "MPN1"
-F 6 "RCA060310K0JNEA" H 0   0   50  0001 C CNN "MPN2"
-F 7 "ESR03EZPJ103" H 0   0   50  0001 C CNN "MPN3"
+F 4 "RMCF0603JT10K0" H 0   0   50  0001 C CNN "MPN"
+F 5 "RCA060310K0JNEA" H 0   0   50  0001 C CNN "MPN2"
+F 6 "ESR03EZPJ103" H 0   0   50  0001 C CNN "MPN3"
 	1    3850 3150
 	-1   0    0    -1
@@
 F 2 "Capacitor_SMD:C_0603_1608Metric" H 4100 3150 60  0001 C CNN
 F 3 "" H 4100 3150 60  0000 C CNN
-F 4 "" H 2150 -550 50  0001 C CNN "MPN"
-F 5 "GCM188R71C104KA37D" H 0   0   50  0001 C CNN "MPN1"
-F 6 "C0603X104K8RACTU" H 0   0   50  0001 C CNN "MPN2"
-F 7 "CS0603KRX7R7BB104" H 0   0   50  0001 C CNN "MPN3"
+F 4 "GCM188R71C104KA37D" H 0   0   50  0001 C CNN "MPN"
+F 5 "C0603X104K8RACTU" H 0   0   50  0001 C CNN "MPN2"
+F 6 "CS0603KRX7R7BB104" H 0   0   50  0001 C CNN "MPN3"
 	1    4100 3150
 	-1   0    0    -1
@@
 F 2 "Resistor_SMD:R_0603_1608Metric" H 6925 3450 60  0001 C CNN
 F 3 "" H 6925 3450 60  0000 C CNN
-F 4 "" H -25 -350 50  0001 C CNN "MPN"
-F 5 "RMCF0603JT10K0" H 0   0   50  0001 C CNN "MPN1"
-F 6 "RCA060310K0JNEA" H 0   0   50  0001 C CNN "MPN2"
-F 7 "ESR03EZPJ103" H 0   0   50  0001 C CNN "MPN3"
+F 4 "RMCF0603JT10K0" H 0   0   50  0001 C CNN "MPN"
+F 5 "RCA060310K0JNEA" H 0   0   50  0001 C CNN "MPN2"
+F 6 "ESR03EZPJ103" H 0   0   50  0001 C CNN "MPN3"
 	1    6925 3450
 	1    0    0    -1
@@
 F 2 "Capacitor_SMD:C_0603_1608Metric" H 7225 2750 60  0001 C CNN
 F 3 "" H 7225 2750 60  0000 C CNN
-F 4 "" H -25 -350 50  0001 C CNN "MPN"
-F 5 "GCM188R71C104KA37D" H 0   0   50  0001 C CNN "MPN1"
-F 6 "C0603X104K8RACTU" H 0   0   50  0001 C CNN "MPN2"
-F 7 "CS0603KRX7R7BB104" H 0   0   50  0001 C CNN "MPN3"
+F 4 "GCM188R71C104KA37D" H 0   0   50  0001 C CNN "MPN"
+F 5 "C0603X104K8RACTU" H 0   0   50  0001 C CNN "MPN2"
+F 6 "CS0603KRX7R7BB104" H 0   0   50  0001 C CNN "MPN3"
 	1    7225 2750
 	0    -1   -1   0
@@
 F 2 "Resistor_SMD:R_0603_1608Metric" H 3850 2850 60  0001 C CNN
 F 3 "" H 3850 2850 60  0000 C CNN
-F 4 "RMCF0603JT5K60" H -550 -700 50  0001 C CNN "MPN1"
+F 4 "RMCF0603JT5K60" H -550 -700 50  0001 C CNN "MPN"
 F 5 "RC0603JR-075K6L" H 3850 2850 50  0001 C CNN "MPN2"
 F 6 "ESR03EZPJ562" H 3850 2850 50  0001 C CNN "MPN3"
@@
 F 2 "Capacitor_SMD:C_0603_1608Metric" H 3600 3000 60  0001 C CNN
 F 3 "" H 3600 3000 60  0000 C CNN
-F 4 "CL10A106MQ8NNNC" H -1700 -2350 50  0001 C CNN "MPN1"
+F 4 "CL10A106MQ8NNNC" H -1700 -2350 50  0001 C CNN "MPN"
 F 5 "GRM188R60J106KE47D" H 3600 3000 50  0001 C CNN "MPN2"
 F 6 "CC0603MRX5R5BB106" V 3600 3000 50  0001 C CNN "MPN3"
@@
 F 2 "Capacitor_SMD:C_0603_1608Metric" H 8625 2875 60  0001 C CNN
 F 3 "" H 8625 2875 60  0000 C CNN
-F 4 "CL10A106MQ8NNNC" H 3325 -2475 50  0001 C CNN "MPN1"
+F 4 "CL10A106MQ8NNNC" H 3325 -2475 50  0001 C CNN "MPN"
 F 5 "GRM188R60J106KE47D" H 8625 2875 50  0001 C CNN "MPN2"
 F 6 "CC0603MRX5R5BB106" V 8625 2875 50  0001 C CNN "MPN3"

Commit message: bottom,sch: annotate schematic symbols again
Parts:
- renumbered J20 to J10, J19 to J9
Changed lines of the file:
@@
 $EndComp
 $Comp
-L Connector:USB_A J20
+L Connector:USB_A J10
 U 1 1 5B809B95
 P 10050 3300
-F 0 "J20" H 10050 3725 50  0000 C CNN
+F 0 "J10" H 10050 3725 50  0000 C CNN
 F 1 "USB_A" H 10050 3650 50  0000 C CNN
 F 2 "footprints:USB_A_Vertical" H 10200 3250 50  0001 C CNN
@@
 $EndComp
 $Comp
-L Connector:USB_B J19
+L Connector:USB_B J9
 U 1 1 5B809C8F
 P 2100 2900
-F 0 "J19" H 2100 3325 50  0000 C CNN
+F 0 "J9" H 2100 3325 50  0000 C CNN
 F 1 "USB_B" H 2100 3250 50  0000 C CNN
 F 2 "Connector_USB:USB_B_OST_USB-B1HSxx_Horizontal" H 2250 2850 50  0001 C CNN
