File: hw-design/bottom-board/midi.sch (KiCad schematic (older format))
At the start: 16 parts, among them P3 DIN_5, P4 DIN_5, Q12 2N7002, Q13 2N7002, U11 6N137S

Commit message: bottom,sch: fix parts after updating to kicad 5
Parts:
- removed D15, D16, D?: 1N4148, Diodes_SMD:SOD-323, symbol D_Small
- added D? (x3): 1N4148WS, Diode_SMD:D_SOD-323, symbol Diode:1N4148WS
- C53: symbol C_Small -> Device:C_Small
- P3, P4: symbol DIN_5 -> Connector:DIN-5_180degree
- Q12, Q13: symbol Q_NMOS_GSD -> Device:Q_NMOS_GSD
- R18, R47, R48, R49, R50, R51, R52: symbol R_Small -> Device:R_Small
- U11: symbol 6N136 -> Isolator:6N136S; MPN 6N137S -> 6N136S-TA1
Connections:
- wire segments 47 -> 45

Commit message: bottom,sch: fix ERC issues
Parts:
- gave numbers to parts that had none: 3
- renumbered C53 to C66, P3 to P4, P4 to P5, Q12 to Q3, Q13 to Q4, R47 to R31, R48 to R32, R18 to R33, R49 to R34, R50 to R35, R51 to R36, R52 to R37, U11 to U17
Changed lines of the file:
@@
 $EndDescr
 $Comp
-L Device:R_Small R47
+L Device:R_Small R31
 U 1 1 550EB368
 P 3000 3700
-F 0 "R47" H 3050 3750 50  0000 L CNN
+F 0 "R31" H 3050 3750 50  0000 L CNN
 F 1 "220R" H 3050 3650 50  0000 L CNN
 F 2 "Resistors_SMD:R_0805" H 3000 3700 60  0001 C CNN
@@
 $EndComp
 $Comp
-L Device:R_Small R49
+L Device:R_Small R34
 U 1 1 550EE5CB
 P 6700 3450
-F 0 "R49" H 6750 3500 50  0000 L CNN
+F 0 "R34" H 6750 3500 50  0000 L CNN
 F 1 "220R" H 6750 3400 50  0000 L CNN
 F 2 "Resistors_SMD:R_0805" H 6700 3450 60  0001 C CNN
@@
 $EndComp
 $Comp
-L Device:R_Small R50
+L Device:R_Small R35
 U 1 1 550EEE00
 P 7900 3650
-F 0 "R50" H 7950 3700 50  0000 L CNN
+F 0 "R35" H 7950 3700 50  0000 L CNN
 F 1 "220R" H 7950 3600 50  0000 L CNN
 F 2 "Resistors_SMD:R_0805" H 7900 3650 60  0001 C CNN
@@
 $EndComp
 $Comp
-L Device:R_Small R51
+L Device:R_Small R36
 U 1 1 550EEF86
 P 8150 3450
-F 0 "R51" H 8200 3500 50  0000 L CNN
+F 0 "R36" H 8200 3500 50  0000 L CNN
 F 1 "10k" H 8200 3400 50  0000 L CNN
 F 2 "Resistors_SMD:R_0603" H 8150 3450 60  0001 C CNN
@@
 $EndComp
 $Comp
-L Device:R_Small R52
+L Device:R_Small R37
 U 1 1 550EFE8C
 P 8700 3750
-F 0 "R52" H 8750 3800 50  0000 L CNN
+F 0 "R37" H 8750 3800 50  0000 L CNN
 F 1 "10k" H 8750 3700 50  0000 L CNN
 F 2 "Resistors_SMD:R_0603" H 8700 3750 60  0001 C CNN
@@
 $EndComp
 $Comp
-L power:GNDD #PWR0134
+L power:GNDD #PWR0172
 U 1 1 550D1DBB
 P 4250 4100
-F 0 "#PWR0134" H 4250 3850 50  0001 C CNN
+F 0 "#PWR0172" H 4250 3850 50  0001 C CNN
 F 1 "GNDD" H 4250 3950 50  0000 C CNN
 F 2 "" H 4250 4100 60  0000 C CNN
@@
 $EndComp
 $Comp
-L power:GNDD #PWR0135
+L power:GNDD #PWR0176
 U 1 1 550D24C3
 P 7150 3950
-F 0 "#PWR0135" H 7150 3700 50  0001 C CNN
+F 0 "#PWR0176" H 7150 3700 50  0001 C CNN
 F 1 "GNDD" H 7150 3800 50  0000 C CNN
 F 2 "" H 7150 3950 60  0000 C CNN
@@
 $EndComp
 $Comp
-L power:GNDD #PWR0136
+L power:GNDD #PWR0178
 U 1 1 550D24EA
 P 8150 4250
-F 0 "#PWR0136" H 8150 4000 50  0001 C CNN
+F 0 "#PWR0178" H 8150 4000 50  0001 C CNN
 F 1 "GNDD" H 8150 4100 50  0000 C CNN
 F 2 "" H 8150 4250 60  0000 C CNN
@@
 $EndComp
 $Comp
-L power:GNDD #PWR0137
+L power:GNDD #PWR0180
 U 1 1 550D2511
 P 8700 4550
-F 0 "#PWR0137" H 8700 4300 50  0001 C CNN
+F 0 "#PWR0180" H 8700 4300 50  0001 C CNN
 F 1 "GNDD" H 8700 4400 50  0000 C CNN
 F 2 "" H 8700 4550 60  0000 C CNN
@@
 $EndComp
 $Comp
-L Device:R_Small R48
+L Device:R_Small R32
 U 1 1 55092D4D
 P 4825 3650
-F 0 "R48" H 4875 3700 50  0000 L CNN
+F 0 "R32" H 4875 3700 50  0000 L CNN
 F 1 "5k6" H 4875 3600 50  0000 L CNN
 F 2 "Resistors_SMD:R_0603" H 4825 3650 60  0001 C CNN
@@
 $EndComp
 $Comp
-L Isolator:6N136S U11
+L Isolator:6N136S U?
 U 1 1 5518A50A
 P 3900 3800
-AR Path="/5518A50A" Ref="U11"  Part="1"
-AR Path="/54F72FB4/5518A50A" Ref="U11"  Part="1"
-F 0 "U11" H 3650 3500 50  0000 L CNN
+AR Path="/5518A50A" Ref="U?"  Part="1"
+AR Path="/54F72FB4/5518A50A" Ref="U17"  Part="1"
+F 0 "U17" H 3650 3500 50  0000 L CNN
 F 1 "6N137S" H 3900 3500 50  0000 L CNN
 F 2 "SMD_Packages:DIP-8_SMD" H 3700 3500 50  0001 L CIN
@@
 $EndComp
 $Comp
-L Device:C_Small C53
+L Device:C_Small C66
 U 1 1 5518B571
 P 4050 3300
-F 0 "C53" V 4100 3350 50  0000 L CNN
+F 0 "C66" V 4100 3350 50  0000 L CNN
 F 1 "100nF" V 3950 3150 50  0000 L CNN
 F 2 "Capacitors_SMD:C_0603" H 4050 3300 60  0001 C CNN
@@
 $EndComp
 $Comp
-L power:GNDD #PWR0143
+L power:GNDD #PWR0170
 U 1 1 5518B6A5
 P 3850 3350
-F 0 "#PWR0143" H 3850 3100 50  0001 C CNN
+F 0 "#PWR0170" H 3850 3100 50  0001 C CNN
 F 1 "GNDD" H 3850 3200 50  0000 C CNN
 F 2 "" H 3850 3350 60  0000 C CNN
@@
 $EndComp
 $Comp
-L Connector:DIN-5_180degree P3
+L Connector:DIN-5_180degree P4
 U 1 1 552F68D2
 P 2500 3600
-F 0 "P3" H 2625 3825 50  0000 C CNN
+F 0 "P4" H 2625 3825 50  0000 C CNN
 F 1 "DIN_5" H 2500 3350 50  0000 C CNN
 F 2 "Connect:SDS-50J" H 2500 3600 50  0001 C CNN
@@
 $EndComp
 $Comp
-L Connector:DIN-5_180degree P4
+L Connector:DIN-5_180degree P5
 U 1 1 552F86CD
 P 7150 3550
-F 0 "P4" H 7275 3775 50  0000 C CNN
+F 0 "P5" H 7275 3775 50  0000 C CNN
 F 1 "DIN_5" H 7150 3300 50  0000 C CNN
 F 2 "Connect:SDS-50J" H 7150 3550 50  0001 C CNN
@@
 $EndComp
 $Comp
-L Device:Q_NMOS_GSD Q12
+L Device:Q_NMOS_GSD Q3
 U 1 1 5550D667
 P 8250 3950
-F 0 "Q12" H 8600 4000 50  0000 R CNN
+F 0 "Q3" H 8600 4000 50  0000 R CNN
 F 1 "2N7002" H 8700 3900 50  0000 R CNN
 F 2 "Housings_SOT-23_SOT-143_TSOT-6:SOT-23" H 8450 4050 29  0001 C CNN
@@
 $EndComp
 $Comp
-L Device:Q_NMOS_GSD Q13
+L Device:Q_NMOS_GSD Q4
 U 1 1 5550D961
 P 8800 4250
-F 0 "Q13" H 9150 4300 50  0000 R CNN
+F 0 "Q4" H 9150 4300 50  0000 R CNN
 F 1 "2N7002" H 9250 4200 50  0000 R CNN
 F 2 "Housings_SOT-23_SOT-143_TSOT-6:SOT-23" H 9000 4350 29  0001 C CNN
@@
 NoConn ~ 2200 3600
 $Comp
-L Device:R_Small R18
+L Device:R_Small R33
 U 1 1 59A564F7
 P 4825 4150
-F 0 "R18" H 4875 4200 50  0000 L CNN
+F 0 "R33" H 4875 4200 50  0000 L CNN
 F 1 "10k" H 4875 4100 50  0000 L CNN
 F 2 "Resistors_SMD:R_0603" H 4825 4150 60  0001 C CNN
@@
 $EndComp
 $Comp
-L power:GNDD #PWR016
+L power:GNDD #PWR0174
 U 1 1 59A56573
 P 4825 4350
-F 0 "#PWR016" H 4825 4100 50  0001 C CNN
+F 0 "#PWR0174" H 4825 4100 50  0001 C CNN
 F 1 "GNDD" H 4825 4200 50  0000 C CNN
 F 2 "" H 4825 4350 60  0000 C CNN
@@
 	4825 4250 4825 4350
 $Comp
-L power:+5VD #PWR0278
+L power:+5VD #PWR0171
 U 1 1 5B503F50
 P 4250 3250
-F 0 "#PWR0278" H 4250 3100 50  0001 C CNN
+F 0 "#PWR0171" H 4250 3100 50  0001 C CNN
 F 1 "+5VD" H 4250 3390 50  0000 C CNN
 F 2 "" H 4250 3250 50  0001 C CNN
@@
 $EndComp
 $Comp
-L power:+5VD #PWR0279
+L power:+5VD #PWR0173
 U 1 1 5B503F8F
 P 4825 3450
-F 0 "#PWR0279" H 4825 3300 50  0001 C CNN
+F 0 "#PWR0173" H 4825 3300 50  0001 C CNN
 F 1 "+5VD" H 4825 3590 50  0000 C CNN
 F 2 "" H 4825 3450 50  0001 C CNN
@@
 $EndComp
 $Comp
-L power:+5VD #PWR0280
+L power:+5VD #PWR0175
 U 1 1 5B503FC7
 P 6700 3300
-F 0 "#PWR0280" H 6700 3150 50  0001 C CNN
+F 0 "#PWR0175" H 6700 3150 50  0001 C CNN
 F 1 "+5VD" H 6700 3440 50  0000 C CNN
 F 2 "" H 6700 3300 50  0001 C CNN
@@
 $EndComp
 $Comp
-L power:+5VD #PWR0281
+L power:+5VD #PWR0177
 U 1 1 5B503FFF
 P 8150 3300
-F 0 "#PWR0281" H 8150 3150 50  0001 C CNN
+F 0 "#PWR0177" H 8150 3150 50  0001 C CNN
 F 1 "+5VD" H 8150 3440 50  0000 C CNN
 F 2 "" H 8150 3300 50  0001 C CNN
@@
 $EndComp
 $Comp
-L power:+5VD #PWR0282
+L power:+5VD #PWR0179
 U 1 1 5B504181
 P 8700 3550
-F 0 "#PWR0282" H 8700 3400 50  0001 C CNN
+F 0 "#PWR0179" H 8700 3400 50  0001 C CNN
 F 1 "+5VD" H 8700 3690 50  0000 C CNN
 F 2 "" H 8700 3550 50  0001 C CNN
@@
 P 7550 3275
 AR Path="/54F72CD0/5B5D9D6F" Ref="D?"  Part="1"
-AR Path="/54F72FB4/5B5D9D6F" Ref="D?"  Part="1"
-F 0 "D?" H 7550 3100 50  0000 C CNN
+AR Path="/54F72FB4/5B5D9D6F" Ref="D13"  Part="1"
+F 0 "D13" H 7550 3100 50  0000 C CNN
 F 1 "1N4148WS" H 7550 3175 50  0000 C CNN
 F 2 "Diode_SMD:D_SOD-323" H 7550 3100 50  0001 C CNN
@@
 P 4500 3900
 AR Path="/54F72CD0/5B7DD60D" Ref="D?"  Part="1"
-AR Path="/54F72FB4/5B7DD60D" Ref="D?"  Part="1"
-F 0 "D?" H 4500 3725 50  0000 C CNN
+AR Path="/54F72FB4/5B7DD60D" Ref="D12"  Part="1"
+F 0 "D12" H 4500 3725 50  0000 C CNN
 F 1 "1N4148WS" H 4500 3800 50  0000 C CNN
 F 2 "Diode_SMD:D_SOD-323" H 4500 3725 50  0001 C CNN
@@
 P 3300 3950
 AR Path="/54F72CD0/5B7E2A8C" Ref="D?"  Part="1"
-AR Path="/54F72FB4/5B7E2A8C" Ref="D?"  Part="1"
-F 0 "D?" H 3300 3775 50  0000 C CNN
+AR Path="/54F72FB4/5B7E2A8C" Ref="D11"  Part="1"
+F 0 "D11" H 3300 3775 50  0000 C CNN
 F 1 "1N4148WS" H 3300 3850 50  0000 C CNN
 F 2 "Diode_SMD:D_SOD-323" H 3300 3775 50  0001 C CNN

Commit message: bottom,sch: MPN updated on midi sheet
Parts:
- removed R31, R34, R35: 220R, Resistors_SMD:R_0805, symbol Device:R_Small
- added R? (x3): 220R, Resistors_SMD:R_0603, symbol Device:R_Small
- C66: MPN C1608X7R1E104K080AA -> (none); MPN1 (none) -> GCM188R71C104KA37D; MPN2 (none) -> C0603X104K8RACTU; MPN3 (none) -> CS0603KRX7R7BB104
- D11, D12, D13: value 1N4148WS -> 1N4148; MPN 1N4148WX-TP -> (none); MPN1 (none) -> 1N4148WX-TP; MPN2 (none) -> 1N4148WS-7-F; MPN3 (none) -> 1N4148WS-G RVG
- Q3, Q4: MPN 2N7002P,215 -> (none); MPN1 (none) -> 2N7002P,215; MPN2 (none) -> 2N7002K-7; MPN3 (none) -> TSM2N7002KCX RFG
- R32: MPN RMCF0603JT5K60 -> (none); MPN1 (none) -> RMCF0603JT5K60; MPN2 (none) -> RC0603JR-075K6L; MPN3 (none) -> ESR03EZPJ562
- R33, R36, R37: MPN RMCF0603JT10K0 -> (none); MPN1 (none) -> RMCF0603JT10K0; MPN2 (none) -> RCA060310K0JNEA; MPN3 (none) -> ESR03EZPJ103
Other:
- note added: "Opto:\nIf = 16mA, Vf = 1.5V"
Changed lines of the file:
@@
 $EndDescr
-$Comp
-L Device:R_Small R31
-U 1 1 550EB368
-P 3000 3700
-F 0 "R31" H 3050 3750 50  0000 L CNN
-F 1 "220R" H 3050 3650 50  0000 L CNN
-F 2 "Resistors_SMD:R_0805" H 3000 3700 60  0001 C CNN
-F 3 "" H 3000 3700 60  0000 C CNN
-F 4 "ERJ-P06J221V" H 250 150 50  0001 C CNN "MPN"
-	1    3000 3700
-	0    1    1    0
-$EndComp
-$Comp
-L Device:R_Small R34
-U 1 1 550EE5CB
-P 6700 3450
-F 0 "R34" H 6750 3500 50  0000 L CNN
-F 1 "220R" H 6750 3400 50  0000 L CNN
-F 2 "Resistors_SMD:R_0805" H 6700 3450 60  0001 C CNN
-F 3 "" H 6700 3450 60  0000 C CNN
-F 4 "ERJ-P06J221V" H 400 100 50  0001 C CNN "MPN"
-	1    6700 3450
-	-1   0    0    1
-$EndComp
-$Comp
-L Device:R_Small R35
-U 1 1 550EEE00
-P 7900 3650
-F 0 "R35" H 7950 3700 50  0000 L CNN
-F 1 "220R" H 7950 3600 50  0000 L CNN
-F 2 "Resistors_SMD:R_0805" H 7900 3650 60  0001 C CNN
-F 3 "" H 7900 3650 60  0000 C CNN
-F 4 "ERJ-P06J221V" H 550 100 50  0001 C CNN "MPN"
-	1    7900 3650
-	0    -1   -1   0
-$EndComp
 $Comp
 L Device:R_Small R36
@@
 F 2 "Resistors_SMD:R_0603" H 8150 3450 60  0001 C CNN
 F 3 "" H 8150 3450 60  0000 C CNN
-F 4 "RMCF0603JT10K0" H 550 100 50  0001 C CNN "MPN"
+F 4 "" H 550 100 50  0001 C CNN "MPN"
+F 5 "RMCF0603JT10K0" H 0   0   50  0001 C CNN "MPN1"
+F 6 "RCA060310K0JNEA" H 0   0   50  0001 C CNN "MPN2"
+F 7 "ESR03EZPJ103" H 0   0   50  0001 C CNN "MPN3"
 	1    8150 3450
 	1    0    0    -1
@@
 F 2 "Resistors_SMD:R_0603" H 8700 3750 60  0001 C CNN
 F 3 "" H 8700 3750 60  0000 C CNN
-F 4 "RMCF0603JT10K0" H 350 100 50  0001 C CNN "MPN"
+F 4 "" H 350 100 50  0001 C CNN "MPN"
+F 5 "RMCF0603JT10K0" H 0   0   50  0001 C CNN "MPN1"
+F 6 "RCA060310K0JNEA" H 0   0   50  0001 C CNN "MPN2"
+F 7 "ESR03EZPJ103" H 0   0   50  0001 C CNN "MPN3"
 	1    8700 3750
 	1    0    0    -1
@@
 F 2 "Resistors_SMD:R_0603" H 4825 3650 60  0001 C CNN
 F 3 "" H 4825 3650 60  0000 C CNN
-F 4 "RMCF0603JT5K60" H 425 100 50  0001 C CNN "MPN"
+F 4 "RMCF0603JT5K60" H 425 100 50  0001 C CNN "MPN1"
+F 5 "RC0603JR-075K6L" H 4825 3650 50  0001 C CNN "MPN2"
+F 6 "ESR03EZPJ562" H 4825 3650 50  0001 C CNN "MPN3"
 	1    4825 3650
 	1    0    0    1
@@
 F 2 "Capacitors_SMD:C_0603" H 4050 3300 60  0001 C CNN
 F 3 "" H 4050 3300 60  0000 C CNN
-F 4 "C1608X7R1E104K080AA" H 250 150 50  0001 C CNN "MPN"
+F 4 "" H 250 150 50  0001 C CNN "MPN"
+F 5 "GCM188R71C104KA37D" H 0   0   50  0001 C CNN "MPN1"
+F 6 "C0603X104K8RACTU" H 0   0   50  0001 C CNN "MPN2"
+F 7 "CS0603KRX7R7BB104" H 0   0   50  0001 C CNN "MPN3"
 	1    4050 3300
 	0    1    1    0
@@
 U 1 1 5550D667
 P 8250 3950
-F 0 "Q3" H 8600 4000 50  0000 R CNN
-F 1 "2N7002" H 8700 3900 50  0000 R CNN
+F 0 "Q3" H 8475 3975 50  0000 L CNN
+F 1 "2N7002" H 8475 3900 50  0000 L CNN
 F 2 "Housings_SOT-23_SOT-143_TSOT-6:SOT-23" H 8450 4050 29  0001 C CNN
 F 3 "" H 8250 3950 60  0000 C CNN
-F 4 "2N7002P,215" H 8250 3950 60  0001 C CNN "MPN"
+F 4 "" H 8250 3950 60  0001 C CNN "MPN"
+F 5 "2N7002P,215" H 0   0   50  0001 C CNN "MPN1"
+F 6 "2N7002K-7" H 0   0   50  0001 C CNN "MPN2"
+F 7 "TSM2N7002KCX RFG" H 0   0   50  0001 C CNN "MPN3"
 	1    8250 3950
 	-1   0    0    -1
@@
 U 1 1 5550D961
 P 8800 4250
-F 0 "Q4" H 9150 4300 50  0000 R CNN
-F 1 "2N7002" H 9250 4200 50  0000 R CNN
+F 0 "Q4" H 9000 4275 50  0000 L CNN
+F 1 "2N7002" H 9000 4200 50  0000 L CNN
 F 2 "Housings_SOT-23_SOT-143_TSOT-6:SOT-23" H 9000 4350 29  0001 C CNN
 F 3 "" H 8800 4250 60  0000 C CNN
-F 4 "2N7002P,215" H 8800 4250 60  0001 C CNN "MPN"
+F 4 "" H 8800 4250 60  0001 C CNN "MPN"
+F 5 "2N7002P,215" H 0   0   50  0001 C CNN "MPN1"
+F 6 "2N7002K-7" H 0   0   50  0001 C CNN "MPN2"
+F 7 "TSM2N7002KCX RFG" H 0   0   50  0001 C CNN "MPN3"
 	1    8800 4250
 	-1   0    0    -1
@@
 F 2 "Resistors_SMD:R_0603" H 4825 4150 60  0001 C CNN
 F 3 "" H 4825 4150 60  0000 C CNN
-F 4 "RMCF0603JT10K0" H 425 600 50  0001 C CNN "MPN"
+F 4 "RMCF0603JT10K0" H 0   0   50  0001 C CNN "MPN1"
+F 5 "RCA060310K0JNEA" H 0   0   50  0001 C CNN "MPN2"
+F 6 "ESR03EZPJ103" H 0   0   50  0001 C CNN "MPN3"
 	1    4825 4150
 	1    0    0    1
@@
 AR Path="/54F72FB4/5B5D9D6F" Ref="D13"  Part="1"
 F 0 "D13" H 7550 3100 50  0000 C CNN
-F 1 "1N4148WS" H 7550 3175 50  0000 C CNN
+F 1 "1N4148" H 7550 3175 50  0000 C CNN
 F 2 "Diode_SMD:D_SOD-323" H 7550 3100 50  0001 C CNN
 F 3 "" H 7550 3275 50  0001 C CNN
-F 4 "1N4148WX-TP" H 200 375 50  0001 C CNN "MPN"
+F 4 "" H 200 375 50  0001 C CNN "MPN"
+F 5 "1N4148WX-TP" H 0   0   50  0001 C CNN "MPN1"
+F 6 "1N4148WS-7-F" H 0   0   50  0001 C CNN "MPN2"
+F 7 "1N4148WS-G RVG" H 0   0   50  0001 C CNN "MPN3"
 	1    7550 3275
 	0    -1   -1   0
@@
 AR Path="/54F72FB4/5B7DD60D" Ref="D12"  Part="1"
 F 0 "D12" H 4500 3725 50  0000 C CNN
-F 1 "1N4148WS" H 4500 3800 50  0000 C CNN
+F 1 "1N4148" H 4500 3800 50  0000 C CNN
 F 2 "Diode_SMD:D_SOD-323" H 4500 3725 50  0001 C CNN
 F 3 "" H 4500 3900 50  0001 C CNN
-F 4 "1N4148WX-TP" H -2850 1000 50  0001 C CNN "MPN"
+F 4 "" H -2850 1000 50  0001 C CNN "MPN"
+F 5 "1N4148WX-TP" H 0   0   50  0001 C CNN "MPN1"
+F 6 "1N4148WS-7-F" H 0   0   50  0001 C CNN "MPN2"
+F 7 "1N4148WS-G RVG" H 0   0   50  0001 C CNN "MPN3"
 	1    4500 3900
 	1    0    0    -1
@@
 AR Path="/54F72FB4/5B7E2A8C" Ref="D11"  Part="1"
 F 0 "D11" H 3300 3775 50  0000 C CNN
-F 1 "1N4148WS" H 3300 3850 50  0000 C CNN
+F 1 "1N4148" H 3300 3850 50  0000 C CNN
 F 2 "Diode_SMD:D_SOD-323" H 3300 3775 50  0001 C CNN
 F 3 "" H 3300 3950 50  0001 C CNN
-F 4 "1N4148WX-TP" H -4050 1050 50  0001 C CNN "MPN"
+F 4 "" H -4050 1050 50  0001 C CNN "MPN"
+F 5 "1N4148WX-TP" H 0   0   50  0001 C CNN "MPN1"
+F 6 "1N4148WS-7-F" H 0   0   50  0001 C CNN "MPN2"
+F 7 "1N4148WS-G RVG" H 0   0   50  0001 C CNN "MPN3"
 	1    3300 3950
 	0    1    1    0
@@
 Wire Wire Line
 	7550 3125 7550 2950
+Text Notes 3475 4600 0    60   ~ 0
+Opto:\nIf = 16mA, Vf = 1.5V
+$Comp
+L Device:R_Small R?
+U 1 1 5B8305A1
+P 3000 3700
+AR Path="/54F72FB6/5B8305A1" Ref="R?"  Part="1"
+AR Path="/54F72FB4/5B8305A1" Ref="R?"  Part="1"
+F 0 "R?" H 3050 3750 50  0000 L CNN
+F 1 "220R" H 3050 3650 50  0000 L CNN
+F 2 "Resistors_SMD:R_0603" H 3000 3700 60  0001 C CNN
+F 3 "" H 3000 3700 60  0000 C CNN
+F 4 "ESR03EZPJ221" H -6950 -500 50  0001 C CNN "MPN1"
+F 5 "ERJ-PB3D2200V" H 3000 3700 50  0001 C CNN "MPN2"
+F 6 "CRCW0603220RJNEAHP" H 3000 3700 50  0001 C CNN "MPN3"
+	1    3000 3700
+	0    -1   -1   0
+$EndComp
+$Comp
+L Device:R_Small R?
+U 1 1 5B830E90
+P 6700 3450
+AR Path="/54F72FB6/5B830E90" Ref="R?"  Part="1"
+AR Path="/54F72FB4/5B830E90" Ref="R?"  Part="1"
+F 0 "R?" H 6750 3500 50  0000 L CNN
+F 1 "220R" H 6750 3400 50  0000 L CNN
+F 2 "Resistors_SMD:R_0603" H 6700 3450 60  0001 C CNN
+F 3 "" H 6700 3450 60  0000 C CNN
+F 4 "ESR03EZPJ221" H -3250 -750 50  0001 C CNN "MPN1"
+F 5 "ERJ-PB3D2200V" H 6700 3450 50  0001 C CNN "MPN2"
+F 6 "CRCW0603220RJNEAHP" H 6700 3450 50  0001 C CNN "MPN3"
+	1    6700 3450
+	-1   0    0    -1
+$EndComp
+$Comp
+L Device:R_Small R?
+U 1 1 5B8317A5
+P 7900 3650
+AR Path="/54F72FB6/5B8317A5" Ref="R?"  Part="1"
+AR Path="/54F72FB4/5B8317A5" Ref="R?"  Part="1"
+F 0 "R?" H 7950 3700 50  0000 L CNN
+F 1 "220R" H 7950 3600 50  0000 L CNN
+F 2 "Resistors_SMD:R_0603" H 7900 3650 60  0001 C CNN
+F 3 "" H 7900 3650 60  0000 C CNN
+F 4 "ESR03EZPJ221" H -2050 -550 50  0001 C CNN "MPN1"
+F 5 "ERJ-PB3D2200V" H 7900 3650 50  0001 C CNN "MPN2"
+F 6 "CRCW0603220RJNEAHP" H 7900 3650 50  0001 C CNN "MPN3"
+	1    7900 3650
+	0    -1   -1   0
+$EndComp
 $EndSCHEMATC

Commit message: bottom,sch: replace midi opto
Parts:
- removed C66: 100nF, Capacitors_SMD:C_0603, symbol Device:C_Small
- removed R32: 5k6, Resistors_SMD:R_0603, symbol Device:R_Small
- removed R33: 10k, Resistors_SMD:R_0603, symbol Device:R_Small
- removed U17: 6N137S, SMD_Packages:DIP-8_SMD, symbol Isolator:6N136S
- added U?: LTV-356T, Package_SO:SO-4_4.4x3.6mm_P2.54mm, symbol Isolator:LTV-356T
- Q3, Q4: footprint Housings_SOT-23_SOT-143_TSOT-6:SOT-23 -> Package_TO_SOT_SMD:SOT-23
- R31, R34, R35: renamed from R?; footprint Resistors_SMD:R_0603 -> Resistor_SMD:R_0603_1608Metric
- R36, R37: footprint Resistors_SMD:R_0603 -> Resistor_SMD:R_0603_1608Metric
Connections:
- wire segments 45 -> 36
- no-connect marks 5 -> 4
Other:
- note added: "Opto:\nIf = 16mA, Vf = 1.4V"
- note removed: "Opto:\nIf = 16mA, Vf = 1.5V"

Commit message: bottom,sch: fix/update footprints field
Parts:
- gave numbers to parts that had none: 1
- renumbered R31 to R32, R34 to R33, R35 to R34, R36 to R35, R37 to R36
Changed lines of the file:
@@
 $EndDescr
 $Comp
-L Device:R_Small R36
+L Device:R_Small R35
 U 1 1 550EEF86
 P 8150 3450
-F 0 "R36" H 8200 3500 50  0000 L CNN
+F 0 "R35" H 8200 3500 50  0000 L CNN
 F 1 "10k" H 8200 3400 50  0000 L CNN
 F 2 "Resistor_SMD:R_0603_1608Metric" H 8150 3450 60  0001 C CNN
@@
 $EndComp
 $Comp
-L Device:R_Small R37
+L Device:R_Small R36
 U 1 1 550EFE8C
 P 8700 3750
-F 0 "R37" H 8750 3800 50  0000 L CNN
+F 0 "R36" H 8750 3800 50  0000 L CNN
 F 1 "10k" H 8750 3700 50  0000 L CNN
 F 2 "Resistor_SMD:R_0603_1608Metric" H 8700 3750 60  0001 C CNN
@@
 $EndComp
 $Comp
-L power:GNDD #PWR0172
+L power:GNDD #PWR0173
 U 1 1 550D1DBB
 P 4225 4000
-F 0 "#PWR0172" H 4225 3750 50  0001 C CNN
+F 0 "#PWR0173" H 4225 3750 50  0001 C CNN
 F 1 "GNDD" H 4225 3850 50  0000 C CNN
 F 2 "" H 4225 4000 60  0000 C CNN
@@
 $EndComp
 $Comp
-L power:GNDD #PWR0176
+L power:GNDD #PWR0175
 U 1 1 550D24C3
 P 7150 3950
-F 0 "#PWR0176" H 7150 3700 50  0001 C CNN
+F 0 "#PWR0175" H 7150 3700 50  0001 C CNN
 F 1 "GNDD" H 7150 3800 50  0000 C CNN
 F 2 "" H 7150 3950 60  0000 C CNN
@@
 $EndComp
 $Comp
-L power:GNDD #PWR0178
+L power:GNDD #PWR0177
 U 1 1 550D24EA
 P 8150 4250
-F 0 "#PWR0178" H 8150 4000 50  0001 C CNN
+F 0 "#PWR0177" H 8150 4000 50  0001 C CNN
 F 1 "GNDD" H 8150 4100 50  0000 C CNN
 F 2 "" H 8150 4250 60  0000 C CNN
@@
 $EndComp
 $Comp
-L power:GNDD #PWR0180
+L power:GNDD #PWR0179
 U 1 1 550D2511
 P 8700 4550
-F 0 "#PWR0180" H 8700 4300 50  0001 C CNN
+F 0 "#PWR0179" H 8700 4300 50  0001 C CNN
 F 1 "GNDD" H 8700 4400 50  0000 C CNN
 F 2 "" H 8700 4550 60  0000 C CNN
@@
 NoConn ~ 2225 3450
 $Comp
-L power:+5VD #PWR0175
+L power:+5VD #PWR0174
 U 1 1 5B503FC7
 P 6700 3300
-F 0 "#PWR0175" H 6700 3150 50  0001 C CNN
+F 0 "#PWR0174" H 6700 3150 50  0001 C CNN
 F 1 "+5VD" H 6700 3440 50  0000 C CNN
 F 2 "" H 6700 3300 50  0001 C CNN
@@
 $EndComp
 $Comp
-L power:+5VD #PWR0177
+L power:+5VD #PWR0176
 U 1 1 5B503FFF
 P 8150 3300
-F 0 "#PWR0177" H 8150 3150 50  0001 C CNN
+F 0 "#PWR0176" H 8150 3150 50  0001 C CNN
 F 1 "+5VD" H 8150 3440 50  0000 C CNN
 F 2 "" H 8150 3300 50  0001 C CNN
@@
 $EndComp
 $Comp
-L power:+5VD #PWR0179
+L power:+5VD #PWR0178
 U 1 1 5B504181
 P 8700 3550
-F 0 "#PWR0179" H 8700 3400 50  0001 C CNN
+F 0 "#PWR0178" H 8700 3400 50  0001 C CNN
 F 1 "+5VD" H 8700 3690 50  0000 C CNN
 F 2 "" H 8700 3550 50  0001 C CNN
@@
 P 3025 3550
 AR Path="/54F72FB6/5B8305A1" Ref="R?"  Part="1"
-AR Path="/54F72FB4/5B8305A1" Ref="R31"  Part="1"
-F 0 "R31" H 3075 3600 50  0000 L CNN
+AR Path="/54F72FB4/5B8305A1" Ref="R32"  Part="1"
+F 0 "R32" H 3075 3600 50  0000 L CNN
 F 1 "220R" H 3075 3500 50  0000 L CNN
 F 2 "Resistor_SMD:R_0603_1608Metric" H 3025 3550 60  0001 C CNN
@@
 P 6700 3450
 AR Path="/54F72FB6/5B830E90" Ref="R?"  Part="1"
-AR Path="/54F72FB4/5B830E90" Ref="R34"  Part="1"
-F 0 "R34" H 6750 3500 50  0000 L CNN
+AR Path="/54F72FB4/5B830E90" Ref="R33"  Part="1"
+F 0 "R33" H 6750 3500 50  0000 L CNN
 F 1 "220R" H 6750 3400 50  0000 L CNN
 F 2 "Resistor_SMD:R_0603_1608Metric" H 6700 3450 60  0001 C CNN
@@
 P 7900 3650
 AR Path="/54F72FB6/5B8317A5" Ref="R?"  Part="1"
-AR Path="/54F72FB4/5B8317A5" Ref="R35"  Part="1"
-F 0 "R35" H 7950 3700 50  0000 L CNN
+AR Path="/54F72FB4/5B8317A5" Ref="R34"  Part="1"
+F 0 "R34" H 7950 3700 50  0000 L CNN
 F 1 "220R" H 7950 3600 50  0000 L CNN
 F 2 "Resistor_SMD:R_0603_1608Metric" H 7900 3650 60  0001 C CNN
@@
 $EndComp
 $Comp
-L Isolator:LTV-356T U?
+L Isolator:LTV-356T U17
 U 1 1 5B64C88A
 P 3875 3800
-F 0 "U?" H 3875 4125 50  0000 C CNN
+F 0 "U17" H 3875 4125 50  0000 C CNN
 F 1 "LTV-356T" H 3875 4034 50  0000 C CNN
 F 2 "Package_SO:SO-4_4.4x3.6mm_P2.54mm" H 3675 3600 50  0001 L CIN
