File: hw-design/bottom-board/midi.sch (KiCad schematic (older format))
At the start: 13 parts, among them P4 DIN_5, P5 DIN_5, Q3 2N7002, Q4 2N7002, U17 LTV-356T

Commit message: bottom,sch: rename MPN1 to MPN
Parts:
- D11, D12, D13: MPN (none) -> 1N4148WX-TP; MPN1 1N4148WX-TP -> (none)
- Q3, Q4: MPN (none) -> 2N7002P,215; MPN1 2N7002P,215 -> (none)
- R32, R33, R34: MPN (none) -> ESR03EZPJ221; MPN1 ESR03EZPJ221 -> (none)
- R35, R36: MPN (none) -> RMCF0603JT10K0; MPN1 RMCF0603JT10K0 -> (none)
Changed lines of the file:
@@
 F 2 "Resistor_SMD:R_0603_1608Metric" H 8150 3450 60  0001 C CNN
 F 3 "" H 8150 3450 60  0000 C CNN
-F 4 "" H 550 100 50  0001 C CNN "MPN"
-F 5 "RMCF0603JT10K0" H 0   0   50  0001 C CNN "MPN1"
-F 6 "RCA060310K0JNEA" H 0   0   50  0001 C CNN "MPN2"
-F 7 "ESR03EZPJ103" H 0   0   50  0001 C CNN "MPN3"
+F 4 "RMCF0603JT10K0" H 0   0   50  0001 C CNN "MPN"
+F 5 "RCA060310K0JNEA" H 0   0   50  0001 C CNN "MPN2"
+F 6 "ESR03EZPJ103" H 0   0   50  0001 C CNN "MPN3"
 	1    8150 3450
 	1    0    0    -1
@@
 F 2 "Resistor_SMD:R_0603_1608Metric" H 8700 3750 60  0001 C CNN
 F 3 "" H 8700 3750 60  0000 C CNN
-F 4 "" H 350 100 50  0001 C CNN "MPN"
-F 5 "RMCF0603JT10K0" H 0   0   50  0001 C CNN "MPN1"
-F 6 "RCA060310K0JNEA" H 0   0   50  0001 C CNN "MPN2"
-F 7 "ESR03EZPJ103" H 0   0   50  0001 C CNN "MPN3"
+F 4 "RMCF0603JT10K0" H 0   0   50  0001 C CNN "MPN"
+F 5 "RCA060310K0JNEA" H 0   0   50  0001 C CNN "MPN2"
+F 6 "ESR03EZPJ103" H 0   0   50  0001 C CNN "MPN3"
 	1    8700 3750
 	1    0    0    -1
@@
 F 2 "Package_TO_SOT_SMD:SOT-23" H 8450 4050 29  0001 C CNN
 F 3 "" H 8250 3950 60  0000 C CNN
-F 4 "" H 8250 3950 60  0001 C CNN "MPN"
-F 5 "2N7002P,215" H 0   0   50  0001 C CNN "MPN1"
-F 6 "2N7002K-7" H 0   0   50  0001 C CNN "MPN2"
-F 7 "TSM2N7002KCX RFG" H 0   0   50  0001 C CNN "MPN3"
+F 4 "2N7002P,215" H 0   0   50  0001 C CNN "MPN"
+F 5 "2N7002K-7" H 0   0   50  0001 C CNN "MPN2"
+F 6 "TSM2N7002KCX RFG" H 0   0   50  0001 C CNN "MPN3"
 	1    8250 3950
 	-1   0    0    -1
@@
 F 2 "Package_TO_SOT_SMD:SOT-23" H 9000 4350 29  0001 C CNN
 F 3 "" H 8800 4250 60  0000 C CNN
-F 4 "" H 8800 4250 60  0001 C CNN "MPN"
-F 5 "2N7002P,215" H 0   0   50  0001 C CNN "MPN1"
-F 6 "2N7002K-7" H 0   0   50  0001 C CNN "MPN2"
-F 7 "TSM2N7002KCX RFG" H 0   0   50  0001 C CNN "MPN3"
+F 4 "2N7002P,215" H 0   0   50  0001 C CNN "MPN"
+F 5 "2N7002K-7" H 0   0   50  0001 C CNN "MPN2"
+F 6 "TSM2N7002KCX RFG" H 0   0   50  0001 C CNN "MPN3"
 	1    8800 4250
 	-1   0    0    -1
@@
 F 2 "Diode_SMD:D_SOD-323" H 7550 3100 50  0001 C CNN
 F 3 "" H 7550 3275 50  0001 C CNN
-F 4 "" H 200 375 50  0001 C CNN "MPN"
-F 5 "1N4148WX-TP" H 0   0   50  0001 C CNN "MPN1"
-F 6 "1N4148WS-7-F" H 0   0   50  0001 C CNN "MPN2"
-F 7 "1N4148WS-G RVG" H 0   0   50  0001 C CNN "MPN3"
+F 4 "1N4148WX-TP" H 0   0   50  0001 C CNN "MPN"
+F 5 "1N4148WS-7-F" H 0   0   50  0001 C CNN "MPN2"
+F 6 "1N4148WS-G RVG" H 0   0   50  0001 C CNN "MPN3"
 	1    7550 3275
 	0    -1   -1   0
@@
 F 2 "Diode_SMD:D_SOD-323" H 4425 3525 50  0001 C CNN
 F 3 "" H 4425 3700 50  0001 C CNN
-F 4 "" H -2925 800 50  0001 C CNN "MPN"
-F 5 "1N4148WX-TP" H -75 -200 50  0001 C CNN "MPN1"
-F 6 "1N4148WS-7-F" H -75 -200 50  0001 C CNN "MPN2"
-F 7 "1N4148WS-G RVG" H -75 -200 50  0001 C CNN "MPN3"
+F 4 "1N4148WX-TP" H -75 -200 50  0001 C CNN "MPN"
+F 5 "1N4148WS-7-F" H -75 -200 50  0001 C CNN "MPN2"
+F 6 "1N4148WS-G RVG" H -75 -200 50  0001 C CNN "MPN3"
 	1    4425 3700
 	1    0    0    -1
@@
 F 2 "Diode_SMD:D_SOD-323" H 3325 3625 50  0001 C CNN
 F 3 "" H 3325 3800 50  0001 C CNN
-F 4 "" H -4025 900 50  0001 C CNN "MPN"
-F 5 "1N4148WX-TP" H 25  -150 50  0001 C CNN "MPN1"
-F 6 "1N4148WS-7-F" H 25  -150 50  0001 C CNN "MPN2"
-F 7 "1N4148WS-G RVG" H 25  -150 50  0001 C CNN "MPN3"
+F 4 "1N4148WX-TP" H 25  -150 50  0001 C CNN "MPN"
+F 5 "1N4148WS-7-F" H 25  -150 50  0001 C CNN "MPN2"
+F 6 "1N4148WS-G RVG" H 25  -150 50  0001 C CNN "MPN3"
 	1    3325 3800
 	0    1    1    0
@@
 F 2 "Resistor_SMD:R_0603_1608Metric" H 3025 3550 60  0001 C CNN
 F 3 "" H 3025 3550 60  0000 C CNN
-F 4 "ESR03EZPJ221" H -6925 -650 50  0001 C CNN "MPN1"
+F 4 "ESR03EZPJ221" H -6925 -650 50  0001 C CNN "MPN"
 F 5 "ERJ-PB3D2200V" H 3025 3550 50  0001 C CNN "MPN2"
 F 6 "CRCW0603220RJNEAHP" H 3025 3550 50  0001 C CNN "MPN3"
@@
 F 2 "Resistor_SMD:R_0603_1608Metric" H 6700 3450 60  0001 C CNN
 F 3 "" H 6700 3450 60  0000 C CNN
-F 4 "ESR03EZPJ221" H -3250 -750 50  0001 C CNN "MPN1"
+F 4 "ESR03EZPJ221" H -3250 -750 50  0001 C CNN "MPN"
 F 5 "ERJ-PB3D2200V" H 6700 3450 50  0001 C CNN "MPN2"
 F 6 "CRCW0603220RJNEAHP" H 6700 3450 50  0001 C CNN "MPN3"
@@
 F 2 "Resistor_SMD:R_0603_1608Metric" H 7900 3650 60  0001 C CNN
 F 3 "" H 7900 3650 60  0000 C CNN
-F 4 "ESR03EZPJ221" H -2050 -550 50  0001 C CNN "MPN1"
+F 4 "ESR03EZPJ221" H -2050 -550 50  0001 C CNN "MPN"
 F 5 "ERJ-PB3D2200V" H 7900 3650 50  0001 C CNN "MPN2"
 F 6 "CRCW0603220RJNEAHP" H 7900 3650 50  0001 C CNN "MPN3"

Commit message: bottom,sch: annotate schematic symbols again
Parts:
- J11: renamed from P4; footprint Connect:SDS-50J -> footprints:SDS-50J
- J12: renamed from P5; footprint Connect:SDS-50J -> footprints:SDS-50J
Changed lines of the file:
@@
 $EndComp
 $Comp
-L Connector:DIN-5_180degree P4
+L Connector:DIN-5_180degree J11
 U 1 1 552F68D2
 P 2525 3450
-F 0 "P4" H 2650 3675 50  0000 C CNN
+F 0 "J11" H 2650 3675 50  0000 C CNN
 F 1 "DIN_5" H 2525 3200 50  0000 C CNN
-F 2 "Connect:SDS-50J" H 2525 3450 50  0001 C CNN
+F 2 "footprints:SDS-50J" H 2525 3450 50  0001 C CNN
 F 3 "" H 2525 3450 50  0001 C CNN
 F 4 "SDS-50J" H 2525 3450 60  0001 C CNN "MPN"
@@
 $EndComp
 $Comp
-L Connector:DIN-5_180degree P5
+L Connector:DIN-5_180degree J12
 U 1 1 552F86CD
 P 7150 3550
-F 0 "P5" H 7275 3775 50  0000 C CNN
+F 0 "J12" H 7275 3775 50  0000 C CNN
 F 1 "DIN_5" H 7150 3300 50  0000 C CNN
-F 2 "Connect:SDS-50J" H 7150 3550 50  0001 C CNN
+F 2 "footprints:SDS-50J" H 7150 3550 50  0001 C CNN
 F 3 "" H 7150 3550 50  0001 C CNN
 F 4 "SDS-50J" H 7150 3550 60  0001 C CNN "MPN"

Commit message: bottom: replace coreboard connector
Parts:
- renumbered J11 to J13, J12 to J14
Changed lines of the file:
@@
 $EndComp
 $Comp
-L power:GNDD #PWR0173
+L power:GNDD #PWR0164
 U 1 1 550D1DBB
 P 4225 4000
-F 0 "#PWR0173" H 4225 3750 50  0001 C CNN
+F 0 "#PWR0164" H 4225 3750 50  0001 C CNN
 F 1 "GNDD" H 4225 3850 50  0000 C CNN
 F 2 "" H 4225 4000 60  0000 C CNN
@@
 $EndComp
 $Comp
-L power:GNDD #PWR0175
+L power:GNDD #PWR0166
 U 1 1 550D24C3
 P 7150 3950
-F 0 "#PWR0175" H 7150 3700 50  0001 C CNN
+F 0 "#PWR0166" H 7150 3700 50  0001 C CNN
 F 1 "GNDD" H 7150 3800 50  0000 C CNN
 F 2 "" H 7150 3950 60  0000 C CNN
@@
 $EndComp
 $Comp
-L power:GNDD #PWR0177
+L power:GNDD #PWR0168
 U 1 1 550D24EA
 P 8150 4250
-F 0 "#PWR0177" H 8150 4000 50  0001 C CNN
+F 0 "#PWR0168" H 8150 4000 50  0001 C CNN
 F 1 "GNDD" H 8150 4100 50  0000 C CNN
 F 2 "" H 8150 4250 60  0000 C CNN
@@
 $EndComp
 $Comp
-L power:GNDD #PWR0179
+L power:GNDD #PWR0170
 U 1 1 550D2511
 P 8700 4550
-F 0 "#PWR0179" H 8700 4300 50  0001 C CNN
+F 0 "#PWR0170" H 8700 4300 50  0001 C CNN
 F 1 "GNDD" H 8700 4400 50  0000 C CNN
 F 2 "" H 8700 4550 60  0000 C CNN
@@
 $EndComp
 $Comp
-L Connector:DIN-5_180degree J11
+L Connector:DIN-5_180degree J13
 U 1 1 552F68D2
 P 2525 3450
-F 0 "J11" H 2650 3675 50  0000 C CNN
+F 0 "J13" H 2650 3675 50  0000 C CNN
 F 1 "DIN_5" H 2525 3200 50  0000 C CNN
 F 2 "footprints:SDS-50J" H 2525 3450 50  0001 C CNN
@@
 $EndComp
 $Comp
-L Connector:DIN-5_180degree J12
+L Connector:DIN-5_180degree J14
 U 1 1 552F86CD
 P 7150 3550
-F 0 "J12" H 7275 3775 50  0000 C CNN
+F 0 "J14" H 7275 3775 50  0000 C CNN
 F 1 "DIN_5" H 7150 3300 50  0000 C CNN
 F 2 "footprints:SDS-50J" H 7150 3550 50  0001 C CNN
@@
 NoConn ~ 2225 3450
 $Comp
-L power:+5VD #PWR0174
+L power:+5VD #PWR0165
 U 1 1 5B503FC7
 P 6700 3300
-F 0 "#PWR0174" H 6700 3150 50  0001 C CNN
+F 0 "#PWR0165" H 6700 3150 50  0001 C CNN
 F 1 "+5VD" H 6700 3440 50  0000 C CNN
 F 2 "" H 6700 3300 50  0001 C CNN
@@
 $EndComp
 $Comp
-L power:+5VD #PWR0176
+L power:+5VD #PWR0167
 U 1 1 5B503FFF
 P 8150 3300
-F 0 "#PWR0176" H 8150 3150 50  0001 C CNN
+F 0 "#PWR0167" H 8150 3150 50  0001 C CNN
 F 1 "+5VD" H 8150 3440 50  0000 C CNN
 F 2 "" H 8150 3300 50  0001 C CNN
@@
 $EndComp
 $Comp
-L power:+5VD #PWR0178
+L power:+5VD #PWR0169
 U 1 1 5B504181
 P 8700 3550
-F 0 "#PWR0178" H 8700 3400 50  0001 C CNN
+F 0 "#PWR0169" H 8700 3400 50  0001 C CNN
 F 1 "+5VD" H 8700 3690 50  0000 C CNN
 F 2 "" H 8700 3550 50  0001 C CNN
