File: hw-design/bottom-board/control-voltage.sch (KiCad schematic (older format))
At the start: 35 parts, among them J22 CV_INPUT, J23 HEADPHONES, Q7 BSS84, U19 TS5A23166, U20 ADC122S021, U21 MIC2076A, U22 74LVC3G17, U23 LMV321, U24 MCP4922-EP

Commit message: bottom,sch: fix/update footprints field
Parts:
- C72: footprint Capacitors_SMD:C_0603 -> Capacitor_SMD:C_0603_1608Metric
- C75, C80, C82, C83: renamed from C?; footprint Capacitors_SMD:C_0603 -> Capacitor_SMD:C_0603_1608Metric
- C78: renamed from C80; footprint Capacitors_SMD:C_0603 -> Capacitor_SMD:C_0603_1608Metric
- C79: renamed from C81; footprint Capacitors_SMD:C_0603 -> Capacitor_SMD:C_0603_1608Metric
- Q7: footprint Housings_SOT-23_SOT-143_TSOT-6:SOT-23 -> Package_TO_SOT_SMD:SOT-23
- Q8: renamed from Q?; footprint Housings_SOT-23_SOT-143_TSOT-6:SOT-23 -> Package_TO_SOT_SMD:SOT-23
- R48: renamed from R49; footprint Resistors_SMD:R_0603 -> Resistor_SMD:R_0603_1608Metric
- R49: renamed from R50; footprint Resistors_SMD:R_0603 -> Resistor_SMD:R_0603_1608Metric
- R50: renamed from R51; footprint Resistors_SMD:R_0603 -> Resistor_SMD:R_0603_1608Metric
- R51: renamed from R52; footprint Resistors_SMD:R_0603 -> Resistor_SMD:R_0603_1608Metric
- R52: renamed from R53; footprint Resistors_SMD:R_0603 -> Resistor_SMD:R_0603_1608Metric
- R53: renamed from R54; footprint Resistors_SMD:R_0603 -> Resistor_SMD:R_0603_1608Metric
- R54: renamed from R55; footprint Resistors_SMD:R_0603 -> Resistor_SMD:R_0603_1608Metric
- RA35, RA36, RA37, RA38: renamed from RA?; MPN3 RJ-PB3D1002V -> ERJ-PB3D1002V
- U20: footprint Housings_SSOP:VSSOP-8_2.4x2.1mm_Pitch0.5mm -> Package_SO:VSSOP-8_2.4x2.1mm_P0.5mm
- U21: footprint Housings_SOIC:SOIC-8_3.9x4.9mm_Pitch1.27mm -> Package_SO:SOIC-8_3.9x4.9mm_P1.27mm
- gave numbers to parts that had none: 4

Commit message: bottom,sch: update missing footprint fields
Parts:
- Q7: symbol Device:Q_PMOS_GSD -> Transistor_FET:BSS84
- U22: MPN1 (none) -> SN74LVC3G17DCUR; MPN2 (none) -> 74LVC3G17DC
Changed lines of the file:
@@
 F 1 "BAT54S" H 2800 2000 50  0000 C CNN
 F 2 "Package_TO_SOT_SMD:SOT-23" H 2800 1900 60  0001 C CNN
-F 3 "" H 2800 1900 60  0000 C CNN
+F 3 "https://www.diodes.com/assets/Datasheets/ds11005.pdf" H 2800 1900 60  0001 C CNN
 F 4 "" H -4450 -250 50  0001 C CNN "MPN"
 F 5 "BAT54SFILM" H 0   0   50  0001 C CNN "MPN1"
@@
 F 1 "BAT54S" H 3450 2000 50  0000 C CNN
 F 2 "Package_TO_SOT_SMD:SOT-23" H 3450 1900 60  0001 C CNN
-F 3 "" H 3450 1900 60  0000 C CNN
+F 3 "https://www.diodes.com/assets/Datasheets/ds11005.pdf" H 3450 1900 60  0001 C CNN
 F 4 "" H -3800 -250 50  0001 C CNN "MPN"
 F 5 "BAT54SFILM" H 0   0   50  0001 C CNN "MPN1"
@@
 $EndComp
 $Comp
-L Device:Q_PMOS_GSD Q7
+L Transistor_FET:BSS84 Q7
 U 1 1 5B4CC381
 P 6650 2475
@@
 F 2 "Package_SO:VSSOP-8_2.3x2mm_P0.5mm" H 7900 2550 50  0001 C CNN
 F 3 "http://www.ti.com/lit/ds/symlink/sn74lvc3g17.pdf" H 7900 2550 50  0001 C CNN
+F 4 "SN74LVC3G17DCUR" H 7900 2550 50  0001 C CNN "MPN1"
+F 5 "74LVC3G17DC" H 7900 2550 50  0001 C CNN "MPN2"
 	2    7900 2550
 	1    0    0    -1
@@
 F 2 "Package_SO:VSSOP-8_2.3x2mm_P0.5mm" H 8300 2375 50  0001 C CNN
 F 3 "http://www.ti.com/lit/ds/symlink/sn74lvc3g17.pdf" H 8300 2375 50  0001 C CNN
+F 4 "SN74LVC3G17DCUR" H 8300 2375 50  0001 C CNN "MPN1"
+F 5 "74LVC3G17DC" H 8300 2375 50  0001 C CNN "MPN2"
 	3    8300 2375
 	1    0    0    -1

Commit message: bottom,sch: rename MPN1 to MPN
Parts:
- C72, C75, C78, C79, C80, C82, C83: MPN (none) -> GCM188R71C104KA37D; MPN1 GCM188R71C104KA37D -> (none)
- C73, C74: MPN (none) -> C0603C333K4RACTU; MPN1 C0603C333K4RACTU -> (none)
- C76, C81: MPN (none) -> CL10A106MQ8NNNC; MPN1 CL10A106MQ8NNNC -> (none)
- C77: MPN (none) -> CL10B105KP8NNNC; MPN1 CL10B105KP8NNNC -> (none)
- D14, D15: MPN (none) -> BAT54SFILM; MPN1 BAT54SFILM -> (none)
- Q7: MPN (none) -> BSS84-7-F; MPN1 BSS84-7-F -> (none)
- Q8: MPN (none) -> 2N7002P,215; MPN1 2N7002P,215 -> (none)
- R48, R49, R53, R54: MPN (none) -> RR0816P-101-D; MPN1 RR0816P-101-D -> (none)
- R50, R51, R52: MPN (none) -> RMCF0603JT10K0; MPN1 RMCF0603JT10K0 -> (none)
- RA35, RA36, RA37, RA38: MPN (none) -> RR0816P-103-D; MPN1 RR0816P-103-D -> (none)
- U22: MPN (none) -> SN74LVC3G17DCUR; MPN1 SN74LVC3G17DCUR -> (none)
- U23: MPN (none) -> LMV321LILT; MPN1 LMV321LILT -> (none)

Commit message: bottom,sch: add comment field to some parts
Parts:
- J22: value CV_INPUT -> NMJ6HCD2; Comment (none) -> CV_INPUT
- J23: value HEADPHONES -> NMJ6HCD2; Comment (none) -> HEADPHONES
Changed lines of the file:
@@
 U 1 1 5B3B64D1
 P 1700 6850
-F 0 "J22" H 1700 7175 50  0000 C CNN
-F 1 "CV_INPUT" H 1650 6450 50  0000 C CNN
+F 0 "J22" H 1700 7250 50  0000 C CNN
+F 1 "NMJ6HCD2" H 1700 7175 50  0000 C CNN
 F 2 "footprints:NMJ6HCD2" H 1950 6950 50  0001 C CNN
 F 3 "" H 1950 6950 50  0001 C CNN
 F 4 "NMJ6HCD2" H 1700 6850 50  0001 C CNN "MPN"
+F 5 "CV_INPUT" H 1700 6475 50  0000 C CNN "Comment"
 	1    1700 6850
 	1    0    0    -1
@@
 U 1 1 5B46F4CC
 P 8850 5900
-F 0 "J23" H 8850 6225 50  0000 C CNN
-F 1 "HEADPHONES" H 8800 5500 50  0000 C CNN
+F 0 "J23" H 8850 6300 50  0000 C CNN
+F 1 "NMJ6HCD2" H 8850 6225 50  0000 C CNN
 F 2 "footprints:NMJ6HCD2" H 9100 6000 50  0001 C CNN
 F 3 "" H 9100 6000 50  0001 C CNN
 F 4 "NMJ6HCD2" H 8850 5900 50  0001 C CNN "MPN"
+F 5 "HEADPHONES" H 8850 5525 50  0000 C CNN "Comment"
 	1    8850 5900
 	-1   0    0    -1

Commit message: bottom,sch: annotate schematic symbols again
Parts:
- renumbered J22 to J14, J23 to J15
Changed lines of the file:
@@
 $EndComp
 $Comp
-L Connector:AudioJack3_Switch J22
+L Connector:AudioJack3_Switch J14
 U 1 1 5B3B64D1
 P 1700 6850
-F 0 "J22" H 1700 7250 50  0000 C CNN
+F 0 "J14" H 1700 7250 50  0000 C CNN
 F 1 "NMJ6HCD2" H 1700 7175 50  0000 C CNN
 F 2 "footprints:NMJ6HCD2" H 1950 6950 50  0001 C CNN
@@
 DAC outputs have Hi-Z when shutdown is on
 $Comp
-L Connector:AudioJack3_Switch J23
+L Connector:AudioJack3_Switch J15
 U 1 1 5B46F4CC
 P 8850 5900
-F 0 "J23" H 8850 6300 50  0000 C CNN
+F 0 "J15" H 8850 6300 50  0000 C CNN
 F 1 "NMJ6HCD2" H 8850 6225 50  0000 C CNN
 F 2 "footprints:NMJ6HCD2" H 9100 6000 50  0001 C CNN

Commit message: bottom: replace coreboard connector
Parts:
- renumbered J14 to J16, J15 to J17

Commit message: bottom: fix footprints U20 and U6
Parts:
- U20: footprint Package_SO:VSSOP-8_2.4x2.1mm_P0.5mm -> Package_SO:VSSOP-8_3.0x3.0mm_P0.65mm
Changed lines of the file:
@@
 F 0 "U20" H 3600 3400 50  0000 L CNN
 F 1 "ADC122S021" H 4450 3400 50  0000 R CNN
-F 2 "Package_SO:VSSOP-8_2.4x2.1mm_P0.5mm" H 4000 3100 50  0001 C CIN
+F 2 "Package_SO:VSSOP-8_3.0x3.0mm_P0.65mm" H 4000 3100 50  0001 C CIN
 F 3 "http://www.ti.com/lit/ds/symlink/adc122s021.pdf" H 4000 3100 50  0001 C CNN
 F 4 "ADC122S021CIMM/NOPB" H 3900 3100 50  0001 C CNN "MPN"

Commit message: bottom,sch: many fixes and addition of test points
Parts:
- removed C79: 100nF, Capacitor_SMD:C_0603_1608Metric, symbol Device:C_Small
- removed Q8: 2N7002, Package_TO_SOT_SMD:SOT-23, symbol Device:Q_NMOS_GSD
- removed U23: LMV321, Package_TO_SOT_SMD:TSOT-23-5, symbol Amplifier_Operational:LMV321
- added C39: 100nF, Capacitor_SMD:C_0603_1608Metric, symbol Device:C_Small
- added R63: 10k, Resistor_SMD:R_0603_1608Metric, symbol Device:R_Small
- added RA47, RA48: 10k 1%, Resistor_SMD:R_0603_1608Metric, symbol Device:R_Small
- added RA? (x2): 499k 1%, Resistor_SMD:R_0603_1608Metric, symbol Device:R_Small
- added TP13, TP14, TP15, TP16, TP17, TP18: TestPoint, TestPoint:TestPoint_Pad_D1.0mm, symbol Connector:TestPoint
- added U4: TS5A3167, Package_TO_SOT_SMD:SOT-23-5, symbol local-components:TS5A3167
Connections:
- net labels removed: HP_VGND
- wire segments 163 -> 175
Other:
- note added: "DAC outputs have Hi-Z (500k)\nwhen shutdown is on"
- note removed: "DAC outputs have Hi-Z when shutdown is on"
- moved on the sheet: Q7, U24
