File: hw-design/bottom-board/audio-inputs.sch (KiCad schematic (older format))
At the start: 35 parts, among them J5 NMJ6HCD2, J6 NMJ6HCD2, U10 TS5A23166, U8 LM4562, U9 TS5A23166

Commit message: bottom: replace coreboard connector
Parts:
- renumbered J5 to J7, J6 to J8
Changed lines of the file:
@@
 $EndComp
 $Comp
-L power:GNDA #PWR099
+L power:GNDA #PWR090
 U 1 1 5B52CB36
 P 2400 2350
-F 0 "#PWR099" H 2400 2100 50  0001 C CNN
+F 0 "#PWR090" H 2400 2100 50  0001 C CNN
 F 1 "GNDA" H 2400 2200 50  0000 C CNN
 F 2 "" H 2400 2350 60  0000 C CNN
@@
 $EndComp
 $Comp
-L power:GNDA #PWR0102
+L power:GNDA #PWR093
 U 1 1 5B52CB4C
 P 2650 2350
-F 0 "#PWR0102" H 2650 2100 50  0001 C CNN
+F 0 "#PWR093" H 2650 2100 50  0001 C CNN
 F 1 "GNDA" H 2650 2200 50  0000 C CNN
 F 2 "" H 2650 2350 60  0000 C CNN
@@
 IN1_GC1
 $Comp
-L power:-5VA #PWR0106
+L power:-5VA #PWR097
 U 1 1 5B52CB69
 P 2900 1600
-F 0 "#PWR0106" H 2900 1700 50  0001 C CNN
+F 0 "#PWR097" H 2900 1700 50  0001 C CNN
 F 1 "-5VA" H 2900 1750 50  0000 C CNN
 F 2 "" H 2900 1600 50  0001 C CNN
@@
 $EndComp
 $Comp
-L power:+5VA #PWR0107
+L power:+5VA #PWR098
 U 1 1 5B52CB6F
 P 3600 1600
-F 0 "#PWR0107" H 3600 1450 50  0001 C CNN
+F 0 "#PWR098" H 3600 1450 50  0001 C CNN
 F 1 "+5VA" H 3600 1740 50  0000 C CNN
 F 2 "" H 3600 1600 50  0001 C CNN
@@
 $EndComp
 $Comp
-L power:+5VA #PWR0100
+L power:+5VA #PWR091
 U 1 1 5B52CB8D
 P 2400 3200
-F 0 "#PWR0100" H 2400 3050 50  0001 C CNN
+F 0 "#PWR091" H 2400 3050 50  0001 C CNN
 F 1 "+5VA" H 2400 3340 50  0000 C CNN
 F 2 "" H 2400 3200 50  0001 C CNN
@@
 IN1_GC2
 $Comp
-L power:GNDA #PWR0101
+L power:GNDA #PWR092
 U 1 1 5B52CB94
 P 2400 4300
-F 0 "#PWR0101" H 2400 4050 50  0001 C CNN
+F 0 "#PWR092" H 2400 4050 50  0001 C CNN
 F 1 "GNDA" H 2400 4150 50  0000 C CNN
 F 2 "" H 2400 4300 60  0000 C CNN
@@
 $EndComp
 $Comp
-L power:GNDA #PWR096
+L power:GNDA #PWR087
 U 1 1 5B52CB9A
 P 1900 4200
-F 0 "#PWR096" H 1900 3950 50  0001 C CNN
+F 0 "#PWR087" H 1900 3950 50  0001 C CNN
 F 1 "GNDA" H 1900 4050 50  0000 C CNN
 F 2 "" H 1900 4200 60  0000 C CNN
@@
 Op Amp Bypass capacitors
 $Comp
-L Connector:AudioJack3_Switch J5
+L Connector:AudioJack3_Switch J7
 U 1 1 5B52CBD7
 P 4600 6700
-F 0 "J5" H 4600 7150 50  0000 C CNN
+F 0 "J7" H 4600 7150 50  0000 C CNN
 F 1 "NMJ6HCD2" H 4600 7050 50  0000 C CNN
 F 2 "footprints:NMJ6HCD2" H 4600 6700 50  0001 C CNN
@@
 $EndComp
 $Comp
-L Connector:AudioJack3_Switch J6
+L Connector:AudioJack3_Switch J8
 U 1 1 5B52CBDF
 P 5550 6700
-F 0 "J6" H 5550 7150 50  0000 C CNN
+F 0 "J8" H 5550 7150 50  0000 C CNN
 F 1 "NMJ6HCD2" H 5550 7050 50  0000 C CNN
 F 2 "footprints:NMJ6HCD2" H 5550 6700 50  0001 C CNN
@@
 IN2
 $Comp
-L power:GNDA #PWR0108
+L power:GNDA #PWR099
 U 1 1 5B52CBE8
 P 4850 7150
-F 0 "#PWR0108" H 4850 6900 50  0001 C CNN
+F 0 "#PWR099" H 4850 6900 50  0001 C CNN
 F 1 "GNDA" H 4850 7000 50  0000 C CNN
 F 2 "" H 4850 7150 60  0000 C CNN
@@
 NoConn ~ 5750 7000
 $Comp
-L power:GNDA #PWR0109
+L power:GNDA #PWR0100
 U 1 1 5B52CBF2
 P 5800 7150
-F 0 "#PWR0109" H 5800 6900 50  0001 C CNN
+F 0 "#PWR0100" H 5800 6900 50  0001 C CNN
 F 1 "GNDA" H 5800 7000 50  0000 C CNN
 F 2 "" H 5800 7150 60  0000 C CNN
@@
 	5750 6900 5850 6900
 $Comp
-L power:GNDA #PWR0111
+L power:GNDA #PWR0102
 U 1 1 5B52CC91
 P 7450 2350
-F 0 "#PWR0111" H 7450 2100 50  0001 C CNN
+F 0 "#PWR0102" H 7450 2100 50  0001 C CNN
 F 1 "GNDA" H 7450 2200 50  0000 C CNN
 F 2 "" H 7450 2350 60  0000 C CNN
@@
 $EndComp
 $Comp
-L power:GNDA #PWR0114
+L power:GNDA #PWR0105
 U 1 1 5B52CCA7
 P 7700 2350
-F 0 "#PWR0114" H 7700 2100 50  0001 C CNN
+F 0 "#PWR0105" H 7700 2100 50  0001 C CNN
 F 1 "GNDA" H 7700 2200 50  0000 C CNN
 F 2 "" H 7700 2350 60  0000 C CNN
@@
 IN2_GC1
 $Comp
-L power:+5VA #PWR094
+L power:+5VA #PWR085
 U 1 1 5B52CCB8
 P 1450 6350
-F 0 "#PWR094" H 1450 6200 50  0001 C CNN
+F 0 "#PWR085" H 1450 6200 50  0001 C CNN
 F 1 "+5VA" H 1450 6490 50  0000 C CNN
 F 2 "" H 1450 6350 50  0001 C CNN
@@
 $EndComp
 $Comp
-L power:-5VA #PWR095
+L power:-5VA #PWR086
 U 1 1 5B52CCBE
 P 1450 7050
-F 0 "#PWR095" H 1450 7150 50  0001 C CNN
+F 0 "#PWR086" H 1450 7150 50  0001 C CNN
 F 1 "-5VA" H 1450 7200 50  0000 C CNN
 F 2 "" H 1450 7050 50  0001 C CNN
@@
 $EndComp
 $Comp
-L power:+5VA #PWR0112
+L power:+5VA #PWR0103
 U 1 1 5B52CCD0
 P 7450 3200
-F 0 "#PWR0112" H 7450 3050 50  0001 C CNN
+F 0 "#PWR0103" H 7450 3050 50  0001 C CNN
 F 1 "+5VA" H 7450 3340 50  0000 C CNN
 F 2 "" H 7450 3200 50  0001 C CNN
@@
 IN2_GC2
 $Comp
-L power:GNDA #PWR0113
+L power:GNDA #PWR0104
 U 1 1 5B52CCD7
 P 7450 4300
-F 0 "#PWR0113" H 7450 4050 50  0001 C CNN
+F 0 "#PWR0104" H 7450 4050 50  0001 C CNN
 F 1 "GNDA" H 7450 4150 50  0000 C CNN
 F 2 "" H 7450 4300 60  0000 C CNN
@@
 $EndComp
 $Comp
-L power:GNDA #PWR0110
+L power:GNDA #PWR0101
 U 1 1 5B52CCDD
 P 6950 4200
-F 0 "#PWR0110" H 6950 3950 50  0001 C CNN
+F 0 "#PWR0101" H 6950 3950 50  0001 C CNN
 F 1 "GNDA" H 6950 4050 50  0000 C CNN
 F 2 "" H 6950 4200 60  0000 C CNN
@@
 0.0\n6.0\n15.0\n20.4
 $Comp
-L power:GNDA #PWR0105
+L power:GNDA #PWR096
 U 1 1 5B5D1412
 P 2850 3350
-F 0 "#PWR0105" H 2850 3100 50  0001 C CNN
+F 0 "#PWR096" H 2850 3100 50  0001 C CNN
 F 1 "GNDA" H 2850 3200 50  0000 C CNN
 F 2 "" H 2850 3350 60  0000 C CNN
@@
 Connection ~ 2400 3300
 $Comp
-L power:GNDA #PWR0115
+L power:GNDA #PWR0106
 U 1 1 5B5D762E
 P 7900 3350
-F 0 "#PWR0115" H 7900 3100 50  0001 C CNN
+F 0 "#PWR0106" H 7900 3100 50  0001 C CNN
 F 1 "GNDA" H 7900 3200 50  0000 C CNN
 F 2 "" H 7900 3350 60  0000 C CNN
@@
 P 2250 6950
 AR Path="/54F72B97/5B626602" Ref="#PWR?"  Part="1"
-AR Path="/54F72C8D/5B626602" Ref="#PWR098"  Part="1"
-F 0 "#PWR098" H 2250 6700 50  0001 C CNN
+AR Path="/54F72C8D/5B626602" Ref="#PWR089"  Part="1"
+F 0 "#PWR089" H 2250 6700 50  0001 C CNN
 F 1 "GNDA" H 2250 6800 50  0000 C CNN
 F 2 "" H 2250 6950 60  0000 C CNN
@@
 P 2250 6500
 AR Path="/54F72B97/5B626608" Ref="#PWR?"  Part="1"
-AR Path="/54F72C8D/5B626608" Ref="#PWR097"  Part="1"
-F 0 "#PWR097" H 2250 6350 50  0001 C CNN
+AR Path="/54F72C8D/5B626608" Ref="#PWR088"  Part="1"
+F 0 "#PWR088" H 2250 6350 50  0001 C CNN
 F 1 "+5VA" H 2250 6640 50  0000 C CNN
 F 2 "" H 2250 6500 60  0000 C CNN
@@
 P 2800 6950
 AR Path="/54F72B97/5B62F3AA" Ref="#PWR?"  Part="1"
-AR Path="/54F72C8D/5B62F3AA" Ref="#PWR0104"  Part="1"
-F 0 "#PWR0104" H 2800 6700 50  0001 C CNN
+AR Path="/54F72C8D/5B62F3AA" Ref="#PWR095"  Part="1"
+F 0 "#PWR095" H 2800 6700 50  0001 C CNN
 F 1 "GNDA" H 2800 6800 50  0000 C CNN
 F 2 "" H 2800 6950 60  0000 C CNN
@@
 $EndComp
 $Comp
-L power:-5VA #PWR0103
+L power:-5VA #PWR094
 U 1 1 5B63434B
 P 2800 6500
-F 0 "#PWR0103" H 2800 6600 50  0001 C CNN
+F 0 "#PWR094" H 2800 6600 50  0001 C CNN
 F 1 "-5VA" H 2800 6650 50  0000 C CNN
 F 2 "" H 2800 6500 50  0001 C CNN
@@
 Connection ~ 3250 2000
 $Comp
-L power:-5VA #PWR0116
+L power:-5VA #PWR0107
 U 1 1 5B68B991
 P 7950 1600
-F 0 "#PWR0116" H 7950 1700 50  0001 C CNN
+F 0 "#PWR0107" H 7950 1700 50  0001 C CNN
 F 1 "-5VA" H 7950 1750 50  0000 C CNN
 F 2 "" H 7950 1600 50  0001 C CNN
@@
 $EndComp
 $Comp
-L power:+5VA #PWR0117
+L power:+5VA #PWR0108
 U 1 1 5B68B997
 P 8650 1600
-F 0 "#PWR0117" H 8650 1450 50  0001 C CNN
+F 0 "#PWR0108" H 8650 1450 50  0001 C CNN
 F 1 "+5VA" H 8650 1740 50  0000 C CNN
 F 2 "" H 8650 1600 50  0001 C CNN

Commit message: bottom,sch: many fixes and addition of test points
Parts:
- removed C38, C41: 10uF, Capacitor_SMD:C_0603_1608Metric, symbol Device:C_Small
- removed C39, C40, C42: 100nF, Capacitor_SMD:C_0603_1608Metric, symbol Device:C_Small
- removed U10, U9: TS5A23166, Package_SO:VSSOP-8_2.3x2mm_P0.5mm, symbol local-components:TS5A23166
- added C10, C9: 10uF 16V, Capacitor_SMD:C_0805_2012Metric, symbol Device:C_Small
- added D16, D17, D18, D19: 1N4148, Diode_SMD:D_SOD-323, symbol Diode:1N4148WS
- added Q10, Q11, Q14, Q15: J109, Housings_SOT-23_SOT-143_TSOT-6:SOT-23, symbol Device:Q_NJFET_DSG
- added Q12, Q13, Q16, Q9: 2N7002, Package_TO_SOT_SMD:SOT-23, symbol Device:Q_NMOS_GSD
- added R18, R57, R60, R61: 1M, Resistor_SMD:R_0603_1608Metric, symbol Device:R_Small
- added R5, R58, R59, R62: 100k, Resistor_SMD:R_0603_1608Metric, symbol Device:R_Small
- added RA39, RA40: 10k 1%, Resistor_SMD:R_0603_1608Metric, symbol Device:R_Small
- added RA41, RA42: 1M 1%, Resistor_SMD:R_0603_1608Metric, symbol Device:R_Small
- added TP6, TP7, TP8, TP9: TestPoint, TestPoint:TestPoint_Pad_D1.0mm, symbol Connector:TestPoint
Connections:
- net labels added: +12VA, INPUT_BIAS
- net labels removed: +5VA, -5VA
- wire segments 122 -> 153
Other:
- note added: "Op Amp Bypass\ncapacitors"
- note added: "The gain calculation isn't\nincluding the RDSon value"
- note removed: "Op Amp Bypass capacitors"
- moved on the sheet: C37, CA3, CA4, CA7, CA8, RA1, RA2, RA8, RA9, U8C

Commit message: bottom,sch: fix jfet footprints
Parts:
- Q10, Q11, Q14, Q15: footprint Housings_SOT-23_SOT-143_TSOT-6:SOT-23 -> Package_TO_SOT_SMD:SOT-23
Changed lines of the file:
@@
 F 0 "Q10" H 3141 3771 50  0000 L CNN
 F 1 "J109" H 3141 3680 50  0000 L CNN
-F 2 "Housings_SOT-23_SOT-143_TSOT-6:SOT-23" H 3150 3825 50  0001 C CNN
+F 2 "Package_TO_SOT_SMD:SOT-23" H 3150 3825 50  0001 C CNN
 F 3 "https://www.nxp.com/docs/en/data-sheet/PMBFJ108_109_110.pdf" H 2950 3725 50  0001 C CNN
 F 4 "PMBFJ109,215" H 2950 3725 50  0001 C CNN "MPN"
@@
 F 0 "Q11" H 4041 3771 50  0000 L CNN
 F 1 "J109" H 4041 3680 50  0000 L CNN
-F 2 "Housings_SOT-23_SOT-143_TSOT-6:SOT-23" H 4050 3825 50  0001 C CNN
+F 2 "Package_TO_SOT_SMD:SOT-23" H 4050 3825 50  0001 C CNN
 F 3 "https://www.nxp.com/docs/en/data-sheet/PMBFJ108_109_110.pdf" H 3850 3725 50  0001 C CNN
 F 4 "PMBFJ109,215" H 3850 3725 50  0001 C CNN "MPN"
@@
 F 0 "Q14" H 8191 3771 50  0000 L CNN
 F 1 "J109" H 8191 3680 50  0000 L CNN
-F 2 "Housings_SOT-23_SOT-143_TSOT-6:SOT-23" H 8200 3825 50  0001 C CNN
+F 2 "Package_TO_SOT_SMD:SOT-23" H 8200 3825 50  0001 C CNN
 F 3 "https://www.nxp.com/docs/en/data-sheet/PMBFJ108_109_110.pdf" H 8000 3725 50  0001 C CNN
 F 4 "PMBFJ109,215" H 8000 3725 50  0001 C CNN "MPN"
@@
 F 0 "Q15" H 9090 3771 50  0000 L CNN
 F 1 "J109" H 9090 3680 50  0000 L CNN
-F 2 "Housings_SOT-23_SOT-143_TSOT-6:SOT-23" H 9100 3825 50  0001 C CNN
+F 2 "Package_TO_SOT_SMD:SOT-23" H 9100 3825 50  0001 C CNN
 F 3 "https://www.nxp.com/docs/en/data-sheet/PMBFJ108_109_110.pdf" H 8900 3725 50  0001 C CNN
 F 4 "PMBFJ109,215" H 8900 3725 50  0001 C CNN "MPN"

Commit message: bottom,sch: add more test points
Parts:
- added TP20: TestPoint, TestPoint:TestPoint_Pad_D1.0mm, symbol Connector:TestPoint
Connections:
- wire segments 153 -> 154
Changed lines of the file:
@@
 Wire Wire Line
 	9975 4025 9900 4025
+$Comp
+L Connector:TestPoint TP?
+U 1 1 5BB4E9C8
+P 1175 6650
+AR Path="/54F7244B/5BB4E9C8" Ref="TP?"  Part="1"
+AR Path="/54F72C8D/5BB4E9C8" Ref="TP20"  Part="1"
+F 0 "TP20" H 1125 6775 50  0000 R CNN
+F 1 "TestPoint" H 1233 6679 50  0001 L CNN
+F 2 "TestPoint:TestPoint_Pad_D1.0mm" H 1375 6650 50  0001 C CNN
+F 3 "~" H 1375 6650 50  0001 C CNN
+	1    1175 6650
+	0    -1   1    0
+$EndComp
+Wire Wire Line
+	1175 6650 1250 6650
 $EndSCHEMATC

Commit message: bottom,sch: change gain control pull up to pull down
Parts:
- added R1, R2, R3, R4: 10k, Resistor_SMD:R_0603_1608Metric, symbol Device:R_Small
Connections:
- wire segments 154 -> 162
Changed lines of the file:
@@
 Wire Wire Line
 	1175 6650 1250 6650
+$Comp
+L Device:R_Small R?
+U 1 1 5BBEADC0
+P 1875 4200
+AR Path="/54F725AE/5BBEADC0" Ref="R?"  Part="1"
+AR Path="/54F72C8D/5BBEADC0" Ref="R1"  Part="1"
+F 0 "R1" H 1925 4250 50  0000 L CNN
+F 1 "10k" H 1925 4150 50  0000 L CNN
+F 2 "Resistor_SMD:R_0603_1608Metric" H 1875 4200 60  0001 C CNN
+F 3 "" H 1875 4200 60  0000 C CNN
+F 4 "RMCF0603JT10K0" H 125 -2450 50  0001 C CNN "MPN"
+F 5 "RCA060310K0JNEA" H 1875 4200 50  0001 C CNN "MPN2"
+F 6 "ESR03EZPJ103" H 1875 4200 50  0001 C CNN "MPN3"
+	1    1875 4200
+	1    0    0    -1
+$EndComp
+$Comp
+L Device:R_Small R?
+U 1 1 5BBEADCA
+P 4925 4200
+AR Path="/54F725AE/5BBEADCA" Ref="R?"  Part="1"
+AR Path="/54F72C8D/5BBEADCA" Ref="R2"  Part="1"
+F 0 "R2" H 4975 4250 50  0000 L CNN
+F 1 "10k" H 4975 4150 50  0000 L CNN
+F 2 "Resistor_SMD:R_0603_1608Metric" H 4925 4200 60  0001 C CNN
+F 3 "" H 4925 4200 60  0000 C CNN
+F 4 "RMCF0603JT10K0" H 3175 -2450 50  0001 C CNN "MPN"
+F 5 "RCA060310K0JNEA" H 4925 4200 50  0001 C CNN "MPN2"
+F 6 "ESR03EZPJ103" H 4925 4200 50  0001 C CNN "MPN3"
+	1    4925 4200
+	1    0    0    -1
+$EndComp
+$Comp
+L Device:R_Small R?
+U 1 1 5BBEADD4
+P 6925 4200
+AR Path="/54F725AE/5BBEADD4" Ref="R?"  Part="1"
+AR Path="/54F72C8D/5BBEADD4" Ref="R3"  Part="1"
+F 0 "R3" H 6975 4250 50  0000 L CNN
+F 1 "10k" H 6975 4150 50  0000 L CNN
+F 2 "Resistor_SMD:R_0603_1608Metric" H 6925 4200 60  0001 C CNN
+F 3 "" H 6925 4200 60  0000 C CNN
+F 4 "RMCF0603JT10K0" H 5175 -2450 50  0001 C CNN "MPN"
+F 5 "RCA060310K0JNEA" H 6925 4200 50  0001 C CNN "MPN2"
+F 6 "ESR03EZPJ103" H 6925 4200 50  0001 C CNN "MPN3"
+	1    6925 4200
+	1    0    0    -1
+$EndComp
+$Comp
+L Device:R_Small R?
+U 1 1 5BBEADDE
+P 9975 4200
+AR Path="/54F725AE/5BBEADDE" Ref="R?"  Part="1"
+AR Path="/54F72C8D/5BBEADDE" Ref="R4"  Part="1"
+F 0 "R4" H 10025 4250 50  0000 L CNN
+F 1 "10k" H 10025 4150 50  0000 L CNN
+F 2 "Resistor_SMD:R_0603_1608Metric" H 9975 4200 60  0001 C CNN
+F 3 "" H 9975 4200 60  0000 C CNN
+F 4 "RMCF0603JT10K0" H 8225 -2450 50  0001 C CNN "MPN"
+F 5 "RCA060310K0JNEA" H 9975 4200 50  0001 C CNN "MPN2"
+F 6 "ESR03EZPJ103" H 9975 4200 50  0001 C CNN "MPN3"
+	1    9975 4200
+	1    0    0    -1
+$EndComp
+Wire Wire Line
+	1875 4100 1875 4025
+Wire Wire Line
+	4925 4100 4925 4025
+$Comp
+L power:GNDA #PWR0178
+U 1 1 5BC120DD
+P 4925 4350
+F 0 "#PWR0178" H 4925 4100 50  0001 C CNN
+F 1 "GNDA" H 4925 4200 50  0000 C CNN
+F 2 "" H 4925 4350 60  0000 C CNN
+F 3 "" H 4925 4350 60  0000 C CNN
+	1    4925 4350
+	-1   0    0    -1
+$EndComp
+Wire Wire Line
+	4925 4300 4925 4350
+$Comp
+L power:GNDA #PWR0181
+U 1 1 5BC222DA
+P 1875 4350
+F 0 "#PWR0181" H 1875 4100 50  0001 C CNN
+F 1 "GNDA" H 1875 4200 50  0000 C CNN
+F 2 "" H 1875 4350 60  0000 C CNN
+F 3 "" H 1875 4350 60  0000 C CNN
+	1    1875 4350
+	1    0    0    -1
+$EndComp
+Wire Wire Line
+	1875 4300 1875 4350
+Wire Wire Line
+	9975 4100 9975 4025
+$Comp
+L power:GNDA #PWR0208
+U 1 1 5BC33DF2
+P 9975 4350
+F 0 "#PWR0208" H 9975 4100 50  0001 C CNN
+F 1 "GNDA" H 9975 4200 50  0000 C CNN
+F 2 "" H 9975 4350 60  0000 C CNN
+F 3 "" H 9975 4350 60  0000 C CNN
+	1    9975 4350
+	-1   0    0    -1
+$EndComp
+Wire Wire Line
+	9975 4300 9975 4350
+Wire Wire Line
+	6925 4100 6925 4025
+$Comp
+L power:GNDA #PWR0209
+U 1 1 5BC443FC
+P 6925 4350
+F 0 "#PWR0209" H 6925 4100 50  0001 C CNN
+F 1 "GNDA" H 6925 4200 50  0000 C CNN
+F 2 "" H 6925 4350 60  0000 C CNN
+F 3 "" H 6925 4350 60  0000 C CNN
+	1    6925 4350
+	1    0    0    -1
+$EndComp
+Wire Wire Line
+	6925 4300 6925 4350
 $EndSCHEMATC

Commit message: bottom,sch: update bom
Parts:
- RA2, RA41, RA42, RA9: MPN RT0603DRE071ML -> RT0603BRD071ML; MPN2 RNCF0603DTE1M00 -> CRCW060310M0DHEAP; MPN3 ERJ-S03D1004V -> CPF0603B1M0E1
Changed lines of the file:
@@
 F 2 "Resistor_SMD:R_0603_1608Metric" H 2050 2200 60  0001 C CNN
 F 3 "" H 2050 2200 60  0000 C CNN
-F 4 "RT0603DRE071ML" H 2050 2200 60  0001 C CNN "MPN"
-F 5 "RNCF0603DTE1M00" H 2050 2200 50  0001 C CNN "MPN2"
-F 6 "ERJ-S03D1004V" H 2050 2200 50  0001 C CNN "MPN3"
+F 4 "RT0603BRD071ML" H 2050 2200 60  0001 C CNN "MPN"
+F 5 "CRCW060310M0DHEAP" H 2050 2200 50  0001 C CNN "MPN2"
+F 6 "CPF0603B1M0E1" H 2050 2200 50  0001 C CNN "MPN3"
 	1    2050 2200
 	-1   0    0    1
@@
 F 2 "Resistor_SMD:R_0603_1608Metric" H 7100 2200 60  0001 C CNN
 F 3 "" H 7100 2200 60  0000 C CNN
-F 4 "RT0603DRE071ML" H 7100 2200 60  0001 C CNN "MPN"
-F 5 "RNCF0603DTE1M00" H 7100 2200 50  0001 C CNN "MPN2"
-F 6 "ERJ-S03D1004V" H 7100 2200 50  0001 C CNN "MPN3"
+F 4 "RT0603BRD071ML" H 7100 2200 60  0001 C CNN "MPN"
+F 5 "CRCW060310M0DHEAP" H 7100 2200 50  0001 C CNN "MPN2"
+F 6 "CPF0603B1M0E1" H 7100 2200 50  0001 C CNN "MPN3"
 	1    7100 2200
 	-1   0    0    1
@@
 F 2 "Resistor_SMD:R_0603_1608Metric" H 2825 2225 60  0001 C CNN
 F 3 "" H 2825 2225 60  0000 C CNN
-F 4 "RT0603DRE071ML" H 2825 2225 60  0001 C CNN "MPN"
-F 5 "RNCF0603DTE1M00" H 2825 2225 50  0001 C CNN "MPN2"
-F 6 "ERJ-S03D1004V" H 2825 2225 50  0001 C CNN "MPN3"
+F 4 "RT0603BRD071ML" H 2825 2225 60  0001 C CNN "MPN"
+F 5 "CRCW060310M0DHEAP" H 2825 2225 50  0001 C CNN "MPN2"
+F 6 "CPF0603B1M0E1" H 2825 2225 50  0001 C CNN "MPN3"
 	1    2825 2225
 	-1   0    0    1
@@
 F 2 "Resistor_SMD:R_0603_1608Metric" H 7875 2225 60  0001 C CNN
 F 3 "" H 7875 2225 60  0000 C CNN
-F 4 "RT0603DRE071ML" H 7875 2225 60  0001 C CNN "MPN"
-F 5 "RNCF0603DTE1M00" H 7875 2225 50  0001 C CNN "MPN2"
-F 6 "ERJ-S03D1004V" H 7875 2225 50  0001 C CNN "MPN3"
+F 4 "RT0603BRD071ML" H 7875 2225 60  0001 C CNN "MPN"
+F 5 "CRCW060310M0DHEAP" H 7875 2225 50  0001 C CNN "MPN2"
+F 6 "CPF0603B1M0E1" H 7875 2225 50  0001 C CNN "MPN3"
 	1    7875 2225
 	-1   0    0    1

Commit message: bottom,sch: fix default state of input gains (pull-up); change J109 -> J110
Parts:
- added R65, R66, R67, R68: 2k7, Resistor_SMD:R_0603_1608Metric, symbol Device:R_Small
- Q10, Q11, Q14, Q15: value J109 -> J110; MPN PMBFJ109,215 -> PMBFJ110,215
Connections:
- wire segments 162 -> 178
Other:
- note added: "1, 1\n1, 0\n0, 1\n0, 0"
- note added: "The gain calculation isn't\nincluding the RDSon value\n\nJ110: RDSon = 18R"
- note removed: "0, 0\n0, 1\n1, 0\n1, 1"
- note removed: "The gain calculation isn't\nincluding the RDSon value"
- moved on the sheet: R1, R2, R3, R4
