File: hw-design/bottom-board/audio-inputs.sch (KiCad schematic (older format))
At the start: 67 parts, among them J7 NMJ6HCD2, J8 NMJ6HCD2, Q10 J110, Q11 J110, Q12 2N7002, Q13 2N7002, Q14 J110, Q15 J110, Q16 2N7002, Q9 2N7002, U8 LM4562

Commit message: bottom,sch: update gain-in feedback resistor to keep values of last revision
Parts:
- RA10, RA3: value 2k49 1% -> 5k62 1%; MPN RR0816P-2491-D-39H -> ERA-3AEB5621V; MPN2 RT0603DRE072K49L -> RT0603BRD075K62L; MPN3 ERJ-PB3D2491V -> RG1608P-5621-B-T5
- RA11, RA4: value 10k 1% -> 21k 1%; MPN RR0816P-103-D -> RR0816P-2102-D-32C; MPN2 RT0603DRE0710KL -> RT0603DRD0721KL; MPN3 ERJ-PB3D1002V -> ERJ-PB3B2102V
- RA12, RA13, RA5, RA6: value 1k5 1% -> 4k99 1%; MPN RR0816P-152-D -> ERA-3AEB4991V; MPN2 RT0603DRE071K5L -> RT0603BRD074K99L; MPN3 ERJ-PB3D1501V -> RG1608P-4991-B-T5
Other:
- note added: "The gain calculation includes\nthe RDSon value\n\nJ110: RDSon = 18R"
- note removed: "The gain calculation isn't\nincluding the RDSon value\n\nJ110: RDSon = 18R"
Changed lines of the file:
@@
 P 3050 3300
 F 0 "RA3" H 3000 3325 50  0000 R CNN
-F 1 "2k49 1%" H 3000 3250 50  0000 R CNN
+F 1 "5k62 1%" H 3000 3250 50  0000 R CNN
 F 2 "Resistor_SMD:R_0603_1608Metric" H 3050 3300 60  0001 C CNN
 F 3 "" H 3050 3300 60  0000 C CNN
-F 4 "RR0816P-2491-D-39H" H -400 650 50  0001 C CNN "MPN"
-F 5 "RT0603DRE072K49L" H 3050 3300 50  0001 C CNN "MPN2"
-F 6 "ERJ-PB3D2491V" H 3050 3300 50  0001 C CNN "MPN3"
+F 4 "ERA-3AEB5621V" H -400 650 50  0001 C CNN "MPN"
+F 5 "RT0603BRD075K62L" H 3050 3300 50  0001 C CNN "MPN2"
+F 6 "RG1608P-5621-B-T5" H 3050 3300 50  0001 C CNN "MPN3"
 	1    3050 3300
 	-1   0    0    1
@@
 P 4150 3000
 F 0 "RA6" V 4075 3000 50  0000 C CNN
-F 1 "1k5 1%" V 4225 3000 50  0000 C CNN
+F 1 "4k99 1%" V 4225 3000 50  0000 C CNN
 F 2 "Resistor_SMD:R_0603_1608Metric" H 4150 3000 60  0001 C CNN
 F 3 "" H 4150 3000 60  0000 C CNN
-F 4 "RR0816P-152-D" H -550 600 50  0001 C CNN "MPN"
-F 5 "RT0603DRE071K5L" V 4150 3000 50  0001 C CNN "MPN2"
-F 6 "ERJ-PB3D1501V" V 4150 3000 50  0001 C CNN "MPN3"
+F 4 "ERA-3AEB4991V" H -550 600 50  0001 C CNN "MPN"
+F 5 "RT0603BRD074K99L" V 4150 3000 50  0001 C CNN "MPN2"
+F 6 "RG1608P-4991-B-T5" V 4150 3000 50  0001 C CNN "MPN3"
 	1    4150 3000
 	0    -1   -1   0
@@
 AR Path="/54F72C8D/5B6A7A98" Ref="RA4"  Part="1"
 F 0 "RA4" V 3325 3000 50  0000 C CNN
-F 1 "10k 1%" V 3475 3000 50  0000 C CNN
+F 1 "21k 1%" V 3475 3000 50  0000 C CNN
 F 2 "Resistor_SMD:R_0603_1608Metric" H 3400 3000 50  0001 C CNN
 F 3 "" H 3400 3000 50  0001 C CNN
-F 4 "RR0816P-103-D" V 3400 3000 60  0001 C CNN "MPN"
-F 5 "RT0603DRE0710KL" V 3400 3000 50  0001 C CNN "MPN2"
-F 6 "ERJ-PB3D1002V" V 3400 3000 50  0001 C CNN "MPN3"
+F 4 "RR0816P-2102-D-32C" V 3400 3000 60  0001 C CNN "MPN"
+F 5 "RT0603DRD0721KL" V 3400 3000 50  0001 C CNN "MPN2"
+F 6 "ERJ-PB3B2102V" V 3400 3000 50  0001 C CNN "MPN3"
 	1    3400 3000
-	0    -1   -1   0
-$EndComp
-$Comp
-L Device:R_Small RA?
-U 1 1 5B6AE289
-P 8450 3000
-AR Path="/54F7244B/5B6AE289" Ref="RA?"  Part="1"
-AR Path="/54F72C8D/5B6AE289" Ref="RA11"  Part="1"
-F 0 "RA11" V 8375 2925 50  0000 L CNN
-F 1 "10k 1%" V 8525 2825 50  0000 L CNN
-F 2 "Resistor_SMD:R_0603_1608Metric" H 8450 3000 50  0001 C CNN
-F 3 "" H 8450 3000 50  0001 C CNN
-F 4 "RR0816P-103-D" V 8450 3000 60  0001 C CNN "MPN"
-F 5 "RT0603DRE0710KL" V 8450 3000 50  0001 C CNN "MPN2"
-F 6 "ERJ-PB3D1002V" V 8450 3000 50  0001 C CNN "MPN3"
-	1    8450 3000
 	0    -1   -1   0
 $EndComp
@@
 P 3750 3300
 F 0 "RA5" H 3800 3275 50  0000 L CNN
-F 1 "1k5 1%" H 3800 3350 50  0000 L CNN
+F 1 "4k99 1%" H 3800 3350 50  0000 L CNN
 F 2 "Resistor_SMD:R_0603_1608Metric" H 3750 3300 60  0001 C CNN
 F 3 "" H 3750 3300 60  0000 C CNN
-F 4 "RR0816P-152-D" H -950 900 50  0001 C CNN "MPN"
-F 5 "RT0603DRE071K5L" V 3750 3300 50  0001 C CNN "MPN2"
-F 6 "ERJ-PB3D1501V" V 3750 3300 50  0001 C CNN "MPN3"
+F 4 "ERA-3AEB4991V" H -950 900 50  0001 C CNN "MPN"
+F 5 "RT0603BRD074K99L" V 3750 3300 50  0001 C CNN "MPN2"
+F 6 "RG1608P-4991-B-T5" V 3750 3300 50  0001 C CNN "MPN3"
 	1    3750 3300
 	1    0    0    -1
-$EndComp
-$Comp
-L Device:R_Small RA13
-U 1 1 5B6B9065
-P 9200 3000
-F 0 "RA13" V 9125 3000 50  0000 C CNN
-F 1 "1k5 1%" V 9275 3000 50  0000 C CNN
-F 2 "Resistor_SMD:R_0603_1608Metric" H 9200 3000 60  0001 C CNN
-F 3 "" H 9200 3000 60  0000 C CNN
-F 4 "RR0816P-152-D" H 4500 600 50  0001 C CNN "MPN"
-F 5 "RT0603DRE071K5L" V 9200 3000 50  0001 C CNN "MPN2"
-F 6 "ERJ-PB3D1501V" V 9200 3000 50  0001 C CNN "MPN3"
-	1    9200 3000
-	0    -1   -1   0
-$EndComp
-$Comp
-L Device:R_Small RA12
-U 1 1 5B6B9859
-P 8800 3300
-F 0 "RA12" H 8850 3275 50  0000 L CNN
-F 1 "1k5 1%" H 8850 3350 50  0000 L CNN
-F 2 "Resistor_SMD:R_0603_1608Metric" H 8800 3300 60  0001 C CNN
-F 3 "" H 8800 3300 60  0000 C CNN
-F 4 "RR0816P-152-D" H 4100 900 50  0001 C CNN "MPN"
-F 5 "RT0603DRE071K5L" V 8800 3300 50  0001 C CNN "MPN2"
-F 6 "ERJ-PB3D1501V" V 8800 3300 50  0001 C CNN "MPN3"
-	1    8800 3300
-	1    0    0    -1
-$EndComp
-$Comp
-L Device:R_Small RA10
-U 1 1 5B6BC180
-P 8100 3300
-F 0 "RA10" H 8050 3325 50  0000 R CNN
-F 1 "2k49 1%" H 8050 3250 50  0000 R CNN
-F 2 "Resistor_SMD:R_0603_1608Metric" H 8100 3300 60  0001 C CNN
-F 3 "" H 8100 3300 60  0000 C CNN
-F 4 "RR0816P-2491-D-39H" H 4650 650 50  0001 C CNN "MPN"
-F 5 "RT0603DRE072K49L" H 8100 3300 50  0001 C CNN "MPN2"
-F 6 "ERJ-PB3D2491V" H 8100 3300 50  0001 C CNN "MPN3"
-	1    8100 3300
-	-1   0    0    1
 $EndComp
 $Comp
@@
 	9600 3350 9600 3425
 Text Notes 9475 5500 0    60   ~ 0
-The gain calculation isn't\nincluding the RDSon value\n\nJ110: RDSon = 18R
+The gain calculation includes\nthe RDSon value\n\nJ110: RDSon = 18R
 $Comp
 L Device:C_Small C?
@@
 Wire Wire Line
 	10125 4025 9975 4025
+$Comp
+L Device:R_Small RA?
+U 1 1 5C3BF4A5
+P 8450 3000
+AR Path="/54F7244B/5C3BF4A5" Ref="RA?"  Part="1"
+AR Path="/54F72C8D/5C3BF4A5" Ref="RA11"  Part="1"
+F 0 "RA11" V 8375 3000 50  0000 C CNN
+F 1 "21k 1%" V 8525 3000 50  0000 C CNN
+F 2 "Resistor_SMD:R_0603_1608Metric" H 8450 3000 50  0001 C CNN
+F 3 "" H 8450 3000 50  0001 C CNN
+F 4 "RR0816P-2102-D-32C" V 8450 3000 60  0001 C CNN "MPN"
+F 5 "RT0603DRD0721KL" V 8450 3000 50  0001 C CNN "MPN2"
+F 6 "ERJ-PB3B2102V" V 8450 3000 50  0001 C CNN "MPN3"
+	1    8450 3000
+	0    -1   -1   0
+$EndComp
+$Comp
+L Device:R_Small RA13
+U 1 1 5C3BF57D
+P 9200 3000
+F 0 "RA13" V 9125 3000 50  0000 C CNN
+F 1 "4k99 1%" V 9275 3000 50  0000 C CNN
+F 2 "Resistor_SMD:R_0603_1608Metric" H 9200 3000 60  0001 C CNN
+F 3 "" H 9200 3000 60  0000 C CNN
+F 4 "ERA-3AEB4991V" H 4500 600 50  0001 C CNN "MPN"
+F 5 "RT0603BRD074K99L" V 9200 3000 50  0001 C CNN "MPN2"
+F 6 "RG1608P-4991-B-T5" V 9200 3000 50  0001 C CNN "MPN3"
+	1    9200 3000
+	0    -1   -1   0
+$EndComp
+$Comp
+L Device:R_Small RA10
+U 1 1 5C3C120E
+P 8100 3300
+F 0 "RA10" H 8050 3325 50  0000 R CNN
+F 1 "5k62 1%" H 8050 3250 50  0000 R CNN
+F 2 "Resistor_SMD:R_0603_1608Metric" H 8100 3300 60  0001 C CNN
+F 3 "" H 8100 3300 60  0000 C CNN
+F 4 "ERA-3AEB5621V" H 4650 650 50  0001 C CNN "MPN"
+F 5 "RT0603BRD075K62L" H 8100 3300 50  0001 C CNN "MPN2"
+F 6 "RG1608P-5621-B-T5" H 8100 3300 50  0001 C CNN "MPN3"
+	1    8100 3300
+	-1   0    0    1
+$EndComp
+$Comp
+L Device:R_Small RA12
+U 1 1 5C3C12F4
+P 8800 3300
+F 0 "RA12" H 8850 3275 50  0000 L CNN
+F 1 "4k99 1%" H 8850 3350 50  0000 L CNN
+F 2 "Resistor_SMD:R_0603_1608Metric" H 8800 3300 60  0001 C CNN
+F 3 "" H 8800 3300 60  0000 C CNN
+F 4 "ERA-3AEB4991V" H 4100 900 50  0001 C CNN "MPN"
+F 5 "RT0603BRD074K99L" V 8800 3300 50  0001 C CNN "MPN2"
+F 6 "RG1608P-4991-B-T5" V 8800 3300 50  0001 C CNN "MPN3"
+	1    8800 3300
+	1    0    0    -1
+$EndComp
 $EndSCHEMATC
