File: hw-design/bottom-board/audio-headphones.sch (KiCad schematic (older format))
At the start: 24 parts, among them U9 LM4811

Commit message: bottom,sch: fix ERC issues
Parts:
- gave numbers to parts that had none: 12
- renumbered C46 to C59, C47 to C60, R40 to R25, R41 to R26, RA39 to RA33, RA40 to RA34, U9 to U14

Commit message: bottom,sch: MPN updated on audio headphones sheet
Parts:
- removed C55, C57, C61: 100nF, Capacitors_SMD:C_0402, symbol Device:C_Small
- removed C56, C58, C59, CA23: 10uF, Capacitors_SMD:c_elec_5x5.3, symbol Device:CP_Small
- removed C60: 100nF, Capacitors_SMD:C_0603, symbol Device:C_Small
- removed CA21, CA22: 10uF, Capacitors_SMD:CP_Elec_4x5.7, symbol Device:CP_Small
- removed CA24, CA25: 100uF, symbol Device:CP_Small
- removed R25, R26: 22R, Resistors_SMD:R_0603, symbol Device:R_Small
- removed R27: 10k, Resistors_SMD:R_0603, symbol Device:R_Small
- removed RA31, RA32: 100R 0.1%, Resistors_SMD:R_0805, symbol Device:R_Small
- removed RA33, RA34: 75k, Resistors_SMD:R_0603, symbol Device:R_Small
- removed U13: LM4562, Housings_SOIC:SOIC-8_3.9x4.9mm_Pitch1.27mm, symbol Amplifier_Operational:LM4562
- added C? (x4): 100nF, Capacitors_SMD:C_0402, symbol Device:C_Small
- added C? (x4): 10uF, Capacitor_SMD:C_0603_1608Metric, symbol Device:C_Small
- added CA? (x2): 100uF, Capacitors_SMD:CP_Elec_6.3x7.7, symbol Device:CP_Small
- added CA? (x2): 10uF, Capacitors_SMD:CP_Elec_4x5.7, symbol Device:CP_Small
- added R? (x2): 22R, Resistors_SMD:R_0603, symbol Device:R_Small
- added R?: 10k, Resistors_SMD:R_0603, symbol Device:R_Small
- added RA? (x2): 100R 1%, Resistors_SMD:R_0603, symbol Device:R_Small
- added RA? (x2): 75k 1%, Resistors_SMD:R_0603, symbol Device:R_Small
- added U? (x3): OPA1678, Housings_SOIC:SOIC-8_3.9x4.9mm_Pitch1.27mm, symbol Amplifier_Operational:LM4562
- U15: footprint (none) -> Package_SO:VSSOP-8_2.3x2mm_P0.5mm; MPN (none) -> TS5A23167DCUR
Connections:
- wire segments 91 -> 90

Commit message: bottom,sch: fix/update footprints field
Parts:
- C55, C57, C61, C62: renamed from C?; footprint Capacitors_SMD:C_0402 -> Capacitor_SMD:C_0603_1608Metric
- R26, R27, R28: renamed from R?; footprint Resistors_SMD:R_0603 -> Resistor_SMD:R_0603_1608Metric
- RA31, RA32, RA33, RA34: renamed from RA?; footprint Resistors_SMD:R_0603 -> Resistor_SMD:R_0603_1608Metric
- U13: renamed from U?; footprint Housings_SOIC:SOIC-8_3.9x4.9mm_Pitch1.27mm -> Package_SO:SOIC-8_3.9x4.9mm_P1.27mm
- U14: footprint Housings_SSOP:MSOP-10_3x3mm_Pitch0.5mm -> Package_SO:MSOP-10_3x3mm_P0.5mm
- gave numbers to parts that had none: 8

Commit message: bottom,sch: rename MPN1 to MPN
Parts:
- C55, C57, C61, C62: MPN (none) -> GCM188R71C104KA37D; MPN1 GCM188R71C104KA37D -> (none)
- C56, C58, C59, C60: MPN (none) -> CL10A106MQ8NNNC; MPN1 CL10A106MQ8NNNC -> (none)
- CA19, CA20: MPN (none) -> EEE-HB1C100R; MPN1 EEE-HB1C100R -> (none)
- CA21, CA22: MPN (none) -> UWX1C101MCL1GB; MPN1 UWX1C101MCL1GB -> (none)
- R26, R27: MPN (none) -> RMCF0603JT22R0; MPN1 RMCF0603JT22R0 -> (none)
- R28: MPN (none) -> RMCF0603JT10K0; MPN1 RMCF0603JT10K0 -> (none)
- RA31, RA32: MPN (none) -> RR0816P-101-D; MPN1 RR0816P-101-D -> (none)
- RA33, RA34: MPN (none) -> RR0816P-753-D; MPN1 RR0816P-753-D -> (none)
Changed lines of the file:
@@
 F 2 "Resistor_SMD:R_0603_1608Metric" H 3150 2450 60  0001 C CNN
 F 3 "" H 3150 2450 60  0000 C CNN
-F 4 "RR0816P-101-D" H -1500 950 50  0001 C CNN "MPN1"
+F 4 "RR0816P-101-D" H -1500 950 50  0001 C CNN "MPN"
 F 5 "RT0603DRE07100RL" H 3150 2450 50  0001 C CNN "MPN2"
 F 6 "ERA-3AED101V" H 3150 2450 50  0001 C CNN "MPN3"
@@
 F 2 "Resistor_SMD:R_0603_1608Metric" H 3150 3900 60  0001 C CNN
 F 3 "" H 3150 3900 60  0000 C CNN
-F 4 "RR0816P-101-D" H -1500 2400 50  0001 C CNN "MPN1"
+F 4 "RR0816P-101-D" H -1500 2400 50  0001 C CNN "MPN"
 F 5 "RT0603DRE07100RL" H 3150 3900 50  0001 C CNN "MPN2"
 F 6 "ERA-3AED101V" H 3150 3900 50  0001 C CNN "MPN3"
@@
 F 2 "Resistor_SMD:R_0603_1608Metric" H 5250 3150 60  0001 C CNN
 F 3 "" H 5250 3150 60  0000 C CNN
-F 4 "RMCF0603JT22R0" H 950 800 50  0001 C CNN "MPN1"
+F 4 "RMCF0603JT22R0" H 950 800 50  0001 C CNN "MPN"
 F 5 "ESR03EZPJ220" V 5250 3150 50  0001 C CNN "MPN3"
 F 6 "RC1608J220CS" V 5250 3150 50  0001 C CNN "MPN2"
@@
 F 2 "Resistor_SMD:R_0603_1608Metric" H 5250 3050 60  0001 C CNN
 F 3 "" H 5250 3050 60  0000 C CNN
-F 4 "RMCF0603JT22R0" H 950 700 50  0001 C CNN "MPN1"
+F 4 "RMCF0603JT22R0" H 950 700 50  0001 C CNN "MPN"
 F 5 "ESR03EZPJ220" V 5250 3050 50  0001 C CNN "MPN3"
 F 6 "RC1608J220CS" V 5250 3050 50  0001 C CNN "MPN2"
@@
 F 2 "Capacitor_SMD:C_0603_1608Metric" H 2925 5475 60  0001 C CNN
 F 3 "" H 2925 5475 60  0000 C CNN
-F 4 "GCM188R71C104KA37D" H -2375 125 50  0001 C CNN "MPN1"
+F 4 "GCM188R71C104KA37D" H -2375 125 50  0001 C CNN "MPN"
 F 5 "C0603X104K8RACTU" V 2925 5475 50  0001 C CNN "MPN2"
 F 6 "CS0603KRX7R7BB104" V 2925 5475 50  0001 C CNN "MPN3"
@@
 F 2 "Capacitor_SMD:C_0603_1608Metric" H 3075 5475 60  0001 C CNN
 F 3 "" H 3075 5475 60  0000 C CNN
-F 4 "CL10A106MQ8NNNC" H -2225 125 50  0001 C CNN "MPN1"
+F 4 "CL10A106MQ8NNNC" H -2225 125 50  0001 C CNN "MPN"
 F 5 "GRM188R60J106KE47D" H 3075 5475 50  0001 C CNN "MPN2"
 F 6 "CC0603MRX5R5BB106" V 3075 5475 50  0001 C CNN "MPN3"
@@
 F 2 "Capacitor_SMD:C_0603_1608Metric" H 3375 5475 60  0001 C CNN
 F 3 "" H 3375 5475 60  0000 C CNN
-F 4 "GCM188R71C104KA37D" H -1925 125 50  0001 C CNN "MPN1"
+F 4 "GCM188R71C104KA37D" H -1925 125 50  0001 C CNN "MPN"
 F 5 "C0603X104K8RACTU" V 3375 5475 50  0001 C CNN "MPN2"
 F 6 "CS0603KRX7R7BB104" V 3375 5475 50  0001 C CNN "MPN3"
@@
 F 2 "Capacitor_SMD:C_0603_1608Metric" H 3525 5475 60  0001 C CNN
 F 3 "" H 3525 5475 60  0000 C CNN
-F 4 "CL10A106MQ8NNNC" H -1775 125 50  0001 C CNN "MPN1"
+F 4 "CL10A106MQ8NNNC" H -1775 125 50  0001 C CNN "MPN"
 F 5 "GRM188R60J106KE47D" H 3525 5475 50  0001 C CNN "MPN2"
 F 6 "CC0603MRX5R5BB106" V 3525 5475 50  0001 C CNN "MPN3"
@@
 F 2 "Capacitor_SMD:C_0603_1608Metric" H 6350 3800 60  0001 C CNN
 F 3 "" H 6350 3800 60  0000 C CNN
-F 4 "CL10A106MQ8NNNC" H 1050 -1550 50  0001 C CNN "MPN1"
+F 4 "CL10A106MQ8NNNC" H 1050 -1550 50  0001 C CNN "MPN"
 F 5 "GRM188R60J106KE47D" H 6350 3800 50  0001 C CNN "MPN2"
 F 6 "CC0603MRX5R5BB106" V 6350 3800 50  0001 C CNN "MPN3"
@@
 F 2 "Capacitor_SMD:C_0603_1608Metric" H 6375 2300 60  0001 C CNN
 F 3 "" H 6375 2300 60  0000 C CNN
-F 4 "GCM188R71C104KA37D" H 1075 -3050 50  0001 C CNN "MPN1"
+F 4 "GCM188R71C104KA37D" H 1075 -3050 50  0001 C CNN "MPN"
 F 5 "C0603X104K8RACTU" V 6375 2300 50  0001 C CNN "MPN2"
 F 6 "CS0603KRX7R7BB104" V 6375 2300 50  0001 C CNN "MPN3"
@@
 F 2 "Capacitor_SMD:C_0603_1608Metric" H 6375 2050 60  0001 C CNN
 F 3 "" H 6375 2050 60  0000 C CNN
-F 4 "CL10A106MQ8NNNC" H 1075 -3300 50  0001 C CNN "MPN1"
+F 4 "CL10A106MQ8NNNC" H 1075 -3300 50  0001 C CNN "MPN"
 F 5 "GRM188R60J106KE47D" H 6375 2050 50  0001 C CNN "MPN2"
 F 6 "CC0603MRX5R5BB106" V 6375 2050 50  0001 C CNN "MPN3"
@@
 F 2 "Capacitor_SMD:C_0603_1608Metric" H 9150 2600 60  0001 C CNN
 F 3 "" H 9150 2600 60  0000 C CNN
-F 4 "GCM188R71C104KA37D" H 3850 -2750 50  0001 C CNN "MPN1"
+F 4 "GCM188R71C104KA37D" H 3850 -2750 50  0001 C CNN "MPN"
 F 5 "C0603X104K8RACTU" V 9150 2600 50  0001 C CNN "MPN2"
 F 6 "CS0603KRX7R7BB104" V 9150 2600 50  0001 C CNN "MPN3"
@@
 F 2 "Capacitors_SMD:CP_Elec_6.3x7.7" H 7550 2750 60  0001 C CNN
 F 3 "" H 7550 2750 60  0000 C CNN
-F 4 "UWX1C101MCL1GB" H 2200 1100 50  0001 C CNN "MPN1"
+F 4 "UWX1C101MCL1GB" H 2200 1100 50  0001 C CNN "MPN"
 F 5 "EEE-HA1C101WP" V 7550 2750 50  0001 C CNN "MPN2"
 F 6 "EEV107M016A9GAA" V 7550 2750 50  0001 C CNN "MPN3"
@@
 F 2 "Capacitors_SMD:CP_Elec_6.3x7.7" H 7550 3550 60  0001 C CNN
 F 3 "" H 7550 3550 60  0000 C CNN
-F 4 "UWX1C101MCL1GB" H 2200 1900 50  0001 C CNN "MPN1"
+F 4 "UWX1C101MCL1GB" H 2200 1900 50  0001 C CNN "MPN"
 F 5 "EEE-HA1C101WP" V 7550 3550 50  0001 C CNN "MPN2"
 F 6 "EEV107M016A9GAA" V 7550 3550 50  0001 C CNN "MPN3"
@@
 F 2 "Capacitors_SMD:CP_Elec_4x5.7" H 2700 2000 60  0001 C CNN
 F 3 "" H 2700 2000 60  0000 C CNN
-F 4 "EEE-HB1C100R" H -2400 500 50  0001 C CNN "MPN1"
+F 4 "EEE-HB1C100R" H -2400 500 50  0001 C CNN "MPN"
 F 5 "UWT1C100MCL1GB" H 2700 2000 50  0001 C CNN "MPN2"
 F 6 "EDH106M016A9BAA" H 2700 2000 50  0001 C CNN "MPN3"
@@
 F 2 "Capacitors_SMD:CP_Elec_4x5.7" H 2700 3450 60  0001 C CNN
 F 3 "" H 2700 3450 60  0000 C CNN
-F 4 "EEE-HB1C100R" H -2400 1950 50  0001 C CNN "MPN1"
+F 4 "EEE-HB1C100R" H -2400 1950 50  0001 C CNN "MPN"
 F 5 "UWT1C100MCL1GB" H 2700 3450 50  0001 C CNN "MPN2"
 F 6 "EDH106M016A9BAA" H 2700 3450 50  0001 C CNN "MPN3"
@@
 F 2 "Resistor_SMD:R_0603_1608Metric" H 8350 3500 60  0001 C CNN
 F 3 "" H 8350 3500 60  0000 C CNN
-F 4 "RMCF0603JT10K0" H 6600 -3150 50  0001 C CNN "MPN1"
+F 4 "RMCF0603JT10K0" H 6600 -3150 50  0001 C CNN "MPN"
 F 5 "RCA060310K0JNEA" H 8350 3500 50  0001 C CNN "MPN2"
 F 6 "ESR03EZPJ103" H 8350 3500 50  0001 C CNN "MPN3"
@@
 F 2 "Resistor_SMD:R_0603_1608Metric" H 7800 3000 60  0001 C CNN
 F 3 "" H 7800 3000 60  0000 C CNN
-F 4 "RR0816P-753-D" H 3750 600 50  0001 C CNN "MPN1"
+F 4 "RR0816P-753-D" H 3750 600 50  0001 C CNN "MPN"
 F 5 "RT0603DRE0775KL" H 7800 3000 50  0001 C CNN "MPN2"
 F 6 "ERJ-PB3D7502V" H 7800 3000 50  0001 C CNN "MPN3"
@@
 F 2 "Resistor_SMD:R_0603_1608Metric" H 7800 3800 60  0001 C CNN
 F 3 "" H 7800 3800 60  0000 C CNN
-F 4 "RR0816P-753-D" H 3750 1400 50  0001 C CNN "MPN1"
+F 4 "RR0816P-753-D" H 3750 1400 50  0001 C CNN "MPN"
 F 5 "RT0603DRE0775KL" H 7800 3800 50  0001 C CNN "MPN2"
 F 6 "ERJ-PB3D7502V" H 7800 3800 50  0001 C CNN "MPN3"

Commit message: bottom,sch: fix few footprints name
Parts:
- CA19, CA20: footprint Capacitors_SMD:CP_Elec_4x5.7 -> Capacitor_SMD:CP_Elec_4x5.7
- CA21, CA22: footprint Capacitors_SMD:CP_Elec_6.3x7.7 -> Capacitor_SMD:CP_Elec_6.3x7.7
Changed lines of the file:
@@
 F 0 "CA21" V 7725 2700 50  0000 L CNN
 F 1 "100uF" V 7650 2650 50  0000 L CNN
-F 2 "Capacitors_SMD:CP_Elec_6.3x7.7" H 7550 2750 60  0001 C CNN
+F 2 "Capacitor_SMD:CP_Elec_6.3x7.7" H 7550 2750 60  0001 C CNN
 F 3 "" H 7550 2750 60  0000 C CNN
 F 4 "UWX1C101MCL1GB" H 2200 1100 50  0001 C CNN "MPN"
@@
 F 0 "CA22" V 7725 3500 50  0000 L CNN
 F 1 "100uF" V 7650 3450 50  0000 L CNN
-F 2 "Capacitors_SMD:CP_Elec_6.3x7.7" H 7550 3550 60  0001 C CNN
+F 2 "Capacitor_SMD:CP_Elec_6.3x7.7" H 7550 3550 60  0001 C CNN
 F 3 "" H 7550 3550 60  0000 C CNN
 F 4 "UWX1C101MCL1GB" H 2200 1900 50  0001 C CNN "MPN"
@@
 F 0 "CA19" H 2775 2050 50  0000 L CNN
 F 1 "10uF" H 2775 1975 50  0000 L CNN
-F 2 "Capacitors_SMD:CP_Elec_4x5.7" H 2700 2000 60  0001 C CNN
+F 2 "Capacitor_SMD:CP_Elec_4x5.7" H 2700 2000 60  0001 C CNN
 F 3 "" H 2700 2000 60  0000 C CNN
 F 4 "EEE-HB1C100R" H -2400 500 50  0001 C CNN "MPN"
@@
 F 0 "CA20" H 2775 3500 50  0000 L CNN
 F 1 "10uF" H 2775 3425 50  0000 L CNN
-F 2 "Capacitors_SMD:CP_Elec_4x5.7" H 2700 3450 60  0001 C CNN
+F 2 "Capacitor_SMD:CP_Elec_4x5.7" H 2700 3450 60  0001 C CNN
 F 3 "" H 2700 3450 60  0000 C CNN
 F 4 "EEE-HB1C100R" H -2400 1950 50  0001 C CNN "MPN"

Commit message: bottom,sch: many fixes and addition of test points
Parts:
- removed C57: 100nF, Capacitor_SMD:C_0603_1608Metric, symbol Device:C_Small
- removed C58: 10uF, Capacitor_SMD:C_0603_1608Metric, symbol Device:C_Small
Connections:
- net labels removed: -5VA
- wire segments 90 -> 82
Other:
- note added: "Op Amp Bypass\ncapacitors"
- note removed: "Op Amp Bypass capacitors"
- moved on the sheet: C55, C56, C62, CA19, CA20, CA21, CA22, R28, RA33, RA34, U13C

Commit message: Changed the headphone buffer to FETS, also remover pull-up from Uboot button
Parts:
- removed C55: 100nF, Capacitor_SMD:C_0603_1608Metric, symbol Device:C_Small
- removed C56: 10uF, Capacitor_SMD:C_0603_1608Metric, symbol Device:C_Small
- removed RA31, RA32: 100R 1%, Resistor_SMD:R_0603_1608Metric, symbol Device:R_Small
- removed U13: OPA1678, Package_SO:SOIC-8_3.9x4.9mm_P1.27mm, symbol Amplifier_Operational:LM4562
- added CA25, CA26: 10uF, Capacitor_SMD:CP_Elec_4x5.7, symbol Device:CP_Small
- added Q17, Q8: J110, Package_TO_SOT_SMD:SOT-23, symbol Device:Q_NJFET_DSG
- added R69, R70: 1Meg, Resistor_SMD:R_0603_1608Metric, symbol Device:R_Small
- added R71, R72: 56k, Resistor_SMD:R_0603_1608Metric, symbol Device:R_Small
- U14: symbol local-components:LM4811 -> bottom-board-rescue:LM4811-local-components
- U15: symbol local-components:TS5A23167 -> bottom-board-rescue:TS5A23167-local-components
Connections:
- wire segments 82 -> 76
Other:
- note removed: "Op Amp Bypass\ncapacitors"
