File: hw-design/bottom-board/spdif.sch (KiCad schematic (older format))
At the start: 6 parts

Commit message: bottom,sch: fix ERC issues
Parts:
- gave numbers to parts that had none: 6
Changed lines of the file:
@@
 CODEC_SPDIF_OUT
 $Comp
-L Device:R_Small R?
+L Device:R_Small R57
 U 1 1 5B562CEC
 P 3650 2150
-F 0 "R?" H 3680 2170 50  0000 L CNN
+F 0 "R57" H 3680 2170 50  0000 L CNN
 F 1 "107" H 3680 2110 50  0000 L CNN
 F 2 "" H 3650 2150 50  0001 C CNN
@@
 $EndComp
 $Comp
-L Device:C_Small C?
+L Device:C_Small C84
 U 1 1 5B562D29
 P 3050 1950
-F 0 "C?" H 3060 2020 50  0000 L CNN
+F 0 "C84" H 3060 2020 50  0000 L CNN
 F 1 "0.01uF" H 3060 1870 50  0000 L CNN
 F 2 "" H 3050 1950 50  0001 C CNN
@@
 $EndComp
 $Comp
-L Device:R_Small R?
+L Device:R_Small R56
 U 1 1 5B562ED8
 P 3400 1950
-F 0 "R?" H 3430 1970 50  0000 L CNN
+F 0 "R56" H 3430 1970 50  0000 L CNN
 F 1 "243" H 3430 1910 50  0000 L CNN
 F 2 "" H 3400 1950 50  0001 C CNN
@@
 $EndComp
 $Comp
-L power:GNDD #PWR0326
+L power:GNDD #PWR0233
 U 1 1 5B56348E
 P 3650 2350
-F 0 "#PWR0326" H 3650 2100 50  0001 C CNN
+F 0 "#PWR0233" H 3650 2100 50  0001 C CNN
 F 1 "GNDD" H 3650 2225 50  0000 C CNN
 F 2 "" H 3650 2350 50  0001 C CNN
@@
 $EndComp
 $Comp
-L Transformer:TRANSF1 TR?
+L Transformer:TRANSF1 TR1
 U 1 1 5B56F2F0
 P 4400 2150
-F 0 "TR?" H 4400 2400 50  0000 C CNN
+F 0 "TR1" H 4400 2400 50  0000 C CNN
 F 1 "PE-65812" H 4400 1900 50  0000 C CNN
 F 2 "" H 4400 2150 50  0001 C CNN
@@
 	3150 1950 3300 1950
 $Comp
-L power:GNDD #PWR0327
+L power:GNDD #PWR0234
 U 1 1 5B56F49A
 P 4100 2450
-F 0 "#PWR0327" H 4100 2200 50  0001 C CNN
+F 0 "#PWR0234" H 4100 2200 50  0001 C CNN
 F 1 "GNDD" H 4100 2325 50  0000 C CNN
 F 2 "" H 4100 2450 50  0001 C CNN
@@
 Connection ~ 3650 1950
 $Comp
-L Device:C_Small C?
+L Device:C_Small C85
 U 1 1 5B56F530
 P 5300 2550
-F 0 "C?" H 5310 2620 50  0000 L CNN
+F 0 "C85" H 5310 2620 50  0000 L CNN
 F 1 "22pF" H 5310 2470 50  0000 L CNN
 F 2 "" H 5300 2550 50  0001 C CNN
@@
 	4600 2350 5300 2350
 $Comp
-L power:GNDD #PWR0328
+L power:GNDD #PWR0235
 U 1 1 5B56F62E
 P 5300 2725
-F 0 "#PWR0328" H 5300 2475 50  0001 C CNN
+F 0 "#PWR0235" H 5300 2475 50  0001 C CNN
 F 1 "GNDD" H 5300 2600 50  0000 C CNN
 F 2 "" H 5300 2725 50  0001 C CNN
@@
 	5300 2350 5300 2450
 $Comp
-L Connector:AudioJack2_Ground_Switch J?
+L Connector:AudioJack2_Ground_Switch J24
 U 1 1 5B5D552C
 P 5575 1950
-F 0 "J?" H 5342 1929 50  0000 R CNN
+F 0 "J24" H 5342 1929 50  0000 R CNN
 F 1 "SPDIF" H 5342 2020 50  0000 R CNN
 F 2 "" H 5575 1950 50  0001 C CNN

Commit message: bottom,sch: MPN updated on spdif sheet
Parts:
- C84: MPN1 (none) -> CL10B103KA8NNNC; MPN2 (none) -> C0603C103M3RACTU; MPN3 (none) -> CC0603KRX7R8BB103
- C85: MPN1 (none) -> C0603C220K4GACTU; MPN2 (none) -> VJ0603A220JXACW1BC; MPN3 (none) -> GRM1885C1H220FA01D
- J24: footprint (none) -> footprints:MJ-3536N; MPN (none) -> MJ-3536N
- R56: value 243 -> 243R; footprint (none) -> Resistor_SMD:R_0603_1608Metric; MPN1 (none) -> RC0603FR-07243RL; MPN2 (none) -> ERJ-3EKF2430V; MPN3 (none) -> RMCF0603FT243R
- R57: value 107 -> 107R; footprint (none) -> Resistor_SMD:R_0603_1608Metric; MPN1 (none) -> RC0603FR-07107RL; MPN2 (none) -> ERJ-3EKF1070V; MPN3 (none) -> RMCF0603FT107R
- TR1: footprint (none) -> footprints:PE-65812NL
Other:
- moved on the sheet: C84, R56, R57
Changed lines of the file:
@@
 Comment4 ""
 $EndDescr
-Text GLabel 2650 1950 0    50   Input ~ 0
+Text GLabel 2775 1950 0    50   Input ~ 0
 CODEC_SPDIF_OUT
 $Comp
 L Device:R_Small R57
 U 1 1 5B562CEC
-P 3650 2150
-F 0 "R57" H 3680 2170 50  0000 L CNN
-F 1 "107" H 3680 2110 50  0000 L CNN
-F 2 "" H 3650 2150 50  0001 C CNN
-F 3 "" H 3650 2150 50  0001 C CNN
-	1    3650 2150
+P 3775 2150
+F 0 "R57" H 3825 2200 50  0000 L CNN
+F 1 "107R" H 3825 2100 50  0000 L CNN
+F 2 "Resistor_SMD:R_0603_1608Metric" H 3775 2150 50  0001 C CNN
+F 3 "" H 3775 2150 50  0001 C CNN
+F 4 "RC0603FR-07107RL" H 3775 2150 50  0001 C CNN "MPN1"
+F 5 "ERJ-3EKF1070V" H 3775 2150 50  0001 C CNN "MPN2"
+F 6 "RMCF0603FT107R" H 3775 2150 50  0001 C CNN "MPN3"
+	1    3775 2150
 	1    0    0    -1
 $EndComp
@@
 L Device:C_Small C84
 U 1 1 5B562D29
-P 3050 1950
-F 0 "C84" H 3060 2020 50  0000 L CNN
-F 1 "0.01uF" H 3060 1870 50  0000 L CNN
-F 2 "" H 3050 1950 50  0001 C CNN
-F 3 "" H 3050 1950 50  0001 C CNN
-	1    3050 1950
+P 3100 1950
+F 0 "C84" V 2925 1950 50  0000 C CNN
+F 1 "0.01uF" V 3000 1950 50  0000 C CNN
+F 2 "" H 3100 1950 50  0001 C CNN
+F 3 "" H 3100 1950 50  0001 C CNN
+F 4 "CL10B103KA8NNNC" H 3100 1950 50  0001 C CNN "MPN1"
+F 5 "C0603C103M3RACTU" V 3100 1950 50  0001 C CNN "MPN2"
+F 6 "CC0603KRX7R8BB103" V 3100 1950 50  0001 C CNN "MPN3"
+	1    3100 1950
 	0    1    1    0
 $EndComp
@@
 L Device:R_Small R56
 U 1 1 5B562ED8
-P 3400 1950
-F 0 "R56" H 3430 1970 50  0000 L CNN
-F 1 "243" H 3430 1910 50  0000 L CNN
-F 2 "" H 3400 1950 50  0001 C CNN
-F 3 "" H 3400 1950 50  0001 C CNN
-	1    3400 1950
+P 3450 1950
+F 0 "R56" H 3500 1900 50  0000 L CNN
+F 1 "243R" H 3500 2000 50  0000 L CNN
+F 2 "Resistor_SMD:R_0603_1608Metric" H 3450 1950 50  0001 C CNN
+F 3 "" H 3450 1950 50  0001 C CNN
+F 4 "RC0603FR-07243RL" H 3450 1950 50  0001 C CNN "MPN1"
+F 5 "ERJ-3EKF2430V" H 3450 1950 50  0001 C CNN "MPN2"
+F 6 "RMCF0603FT243R" H 3450 1950 50  0001 C CNN "MPN3"
+	1    3450 1950
 	0    1    1    0
 $EndComp
@@
 L power:GNDD #PWR0233
 U 1 1 5B56348E
-P 3650 2350
-F 0 "#PWR0233" H 3650 2100 50  0001 C CNN
-F 1 "GNDD" H 3650 2225 50  0000 C CNN
-F 2 "" H 3650 2350 50  0001 C CNN
-F 3 "" H 3650 2350 50  0001 C CNN
-	1    3650 2350
+P 3775 2350
+F 0 "#PWR0233" H 3775 2100 50  0001 C CNN
+F 1 "GNDD" H 3775 2225 50  0000 C CNN
+F 2 "" H 3775 2350 50  0001 C CNN
+F 3 "" H 3775 2350 50  0001 C CNN
+	1    3775 2350
 	1    0    0    -1
 $EndComp
@@
 F 0 "TR1" H 4400 2400 50  0000 C CNN
 F 1 "PE-65812" H 4400 1900 50  0000 C CNN
-F 2 "" H 4400 2150 50  0001 C CNN
-F 3 "" H 4400 2150 50  0001 C CNN
+F 2 "footprints:PE-65812NL" H 4400 2150 50  0001 C CNN
+F 3 "https://productfinder.pulseeng.com/doc_type/WEB301/doc_num/PE-65812NL/doc_part/PE-65812NL.pdf" H 4400 2150 50  0001 C CNN
 F 4 "PE-65812NL" H 4400 2150 60  0001 C CNN "MPN"
 	1    4400 2150
@@
 $EndComp
 Wire Wire Line
-	2650 1950 2950 1950
+	2775 1950 3000 1950
 Wire Wire Line
-	3150 1950 3300 1950
+	3200 1950 3350 1950
 $Comp
 L power:GNDD #PWR0234
@@
 	4100 2350 4200 2350
 Wire Wire Line
-	3650 2350 3650 2250
+	3775 2350 3775 2250
 Wire Wire Line
-	3500 1950 3650 1950
-Wire Wire Line
-	3650 2050 3650 1950
-Connection ~ 3650 1950
+	3775 2050 3775 1950
 $Comp
 L Device:C_Small C85
 U 1 1 5B56F530
 P 5300 2550
-F 0 "C85" H 5310 2620 50  0000 L CNN
-F 1 "22pF" H 5310 2470 50  0000 L CNN
+F 0 "C85" H 5200 2525 50  0000 R CNN
+F 1 "22pF" H 5200 2600 50  0000 R CNN
 F 2 "" H 5300 2550 50  0001 C CNN
 F 3 "" H 5300 2550 50  0001 C CNN
+F 4 "C0603C220K4GACTU" H 5300 2550 50  0001 C CNN "MPN1"
+F 5 "VJ0603A220JXACW1BC" H 5300 2550 50  0001 C CNN "MPN2"
+F 6 "GRM1885C1H220FA01D" H 5300 2550 50  0001 C CNN "MPN3"
 	1    5300 2550
 	-1   0    0    1
@@
 NoConn ~ 5375 1850
 Wire Wire Line
-	3650 1950 4200 1950
-Wire Wire Line
 	5300 2350 5300 2450
 $Comp
@@
 F 0 "J24" H 5342 1929 50  0000 R CNN
 F 1 "SPDIF" H 5342 2020 50  0000 R CNN
-F 2 "" H 5575 1950 50  0001 C CNN
-F 3 "~" H 5575 1950 50  0001 C CNN
+F 2 "footprints:MJ-3536N" H 5575 1950 50  0001 C CNN
+F 3 "https://www.cui.com/product/resource/digikeypdf/mj-3536n.pdf" H 5575 1950 50  0001 C CNN
+F 4 "MJ-3536N" H 5575 1950 50  0001 C CNN "MPN"
 	1    5575 1950
 	-1   0    0    1
@@
 Wire Wire Line
 	5375 1950 4600 1950
+Connection ~ 3775 1950
+Wire Wire Line
+	3775 1950 4200 1950
+Wire Wire Line
+	3550 1950 3775 1950
 $EndSCHEMATC

Commit message: bottom,sch: fix/update footprints field
Parts:
- C84, C85: footprint (none) -> Capacitor_SMD:C_0603_1608Metric
- renumbered R56 to R55, R57 to R56
Changed lines of the file:
@@
 CODEC_SPDIF_OUT
 $Comp
-L Device:R_Small R57
+L Device:R_Small R56
 U 1 1 5B562CEC
 P 3775 2150
-F 0 "R57" H 3825 2200 50  0000 L CNN
+F 0 "R56" H 3825 2200 50  0000 L CNN
 F 1 "107R" H 3825 2100 50  0000 L CNN
 F 2 "Resistor_SMD:R_0603_1608Metric" H 3775 2150 50  0001 C CNN
@@
 F 0 "C84" V 2925 1950 50  0000 C CNN
 F 1 "0.01uF" V 3000 1950 50  0000 C CNN
-F 2 "" H 3100 1950 50  0001 C CNN
+F 2 "Capacitor_SMD:C_0603_1608Metric" H 3100 1950 50  0001 C CNN
 F 3 "" H 3100 1950 50  0001 C CNN
 F 4 "CL10B103KA8NNNC" H 3100 1950 50  0001 C CNN "MPN1"
@@
 $EndComp
 $Comp
-L Device:R_Small R56
+L Device:R_Small R55
 U 1 1 5B562ED8
 P 3450 1950
-F 0 "R56" H 3500 1900 50  0000 L CNN
+F 0 "R55" H 3500 1900 50  0000 L CNN
 F 1 "243R" H 3500 2000 50  0000 L CNN
 F 2 "Resistor_SMD:R_0603_1608Metric" H 3450 1950 50  0001 C CNN
@@
 $EndComp
 $Comp
-L power:GNDD #PWR0233
+L power:GNDD #PWR0231
 U 1 1 5B56348E
 P 3775 2350
-F 0 "#PWR0233" H 3775 2100 50  0001 C CNN
+F 0 "#PWR0231" H 3775 2100 50  0001 C CNN
 F 1 "GNDD" H 3775 2225 50  0000 C CNN
 F 2 "" H 3775 2350 50  0001 C CNN
@@
 	3200 1950 3350 1950
 $Comp
-L power:GNDD #PWR0234
+L power:GNDD #PWR0232
 U 1 1 5B56F49A
 P 4100 2450
-F 0 "#PWR0234" H 4100 2200 50  0001 C CNN
+F 0 "#PWR0232" H 4100 2200 50  0001 C CNN
 F 1 "GNDD" H 4100 2325 50  0000 C CNN
 F 2 "" H 4100 2450 50  0001 C CNN
@@
 F 0 "C85" H 5200 2525 50  0000 R CNN
 F 1 "22pF" H 5200 2600 50  0000 R CNN
-F 2 "" H 5300 2550 50  0001 C CNN
+F 2 "Capacitor_SMD:C_0603_1608Metric" H 5300 2550 50  0001 C CNN
 F 3 "" H 5300 2550 50  0001 C CNN
 F 4 "C0603C220K4GACTU" H 5300 2550 50  0001 C CNN "MPN1"
@@
 	4600 2350 5300 2350
 $Comp
-L power:GNDD #PWR0235
+L power:GNDD #PWR0233
 U 1 1 5B56F62E
 P 5300 2725
-F 0 "#PWR0235" H 5300 2475 50  0001 C CNN
+F 0 "#PWR0233" H 5300 2475 50  0001 C CNN
 F 1 "GNDD" H 5300 2600 50  0000 C CNN
 F 2 "" H 5300 2725 50  0001 C CNN

Commit message: bottom,sch: rename MPN1 to MPN
Parts:
- C84: MPN (none) -> CL10B103KA8NNNC; MPN1 CL10B103KA8NNNC -> (none)
- C85: MPN (none) -> C0603C220K4GACTU; MPN1 C0603C220K4GACTU -> (none)
- R55: MPN (none) -> RC0603FR-07243RL; MPN1 RC0603FR-07243RL -> (none)
- R56: MPN (none) -> RC0603FR-07107RL; MPN1 RC0603FR-07107RL -> (none)
Changed lines of the file:
@@
 F 2 "Resistor_SMD:R_0603_1608Metric" H 3775 2150 50  0001 C CNN
 F 3 "" H 3775 2150 50  0001 C CNN
-F 4 "RC0603FR-07107RL" H 3775 2150 50  0001 C CNN "MPN1"
+F 4 "RC0603FR-07107RL" H 3775 2150 50  0001 C CNN "MPN"
 F 5 "ERJ-3EKF1070V" H 3775 2150 50  0001 C CNN "MPN2"
 F 6 "RMCF0603FT107R" H 3775 2150 50  0001 C CNN "MPN3"
@@
 F 2 "Capacitor_SMD:C_0603_1608Metric" H 3100 1950 50  0001 C CNN
 F 3 "" H 3100 1950 50  0001 C CNN
-F 4 "CL10B103KA8NNNC" H 3100 1950 50  0001 C CNN "MPN1"
+F 4 "CL10B103KA8NNNC" H 3100 1950 50  0001 C CNN "MPN"
 F 5 "C0603C103M3RACTU" V 3100 1950 50  0001 C CNN "MPN2"
 F 6 "CC0603KRX7R8BB103" V 3100 1950 50  0001 C CNN "MPN3"
@@
 F 2 "Resistor_SMD:R_0603_1608Metric" H 3450 1950 50  0001 C CNN
 F 3 "" H 3450 1950 50  0001 C CNN
-F 4 "RC0603FR-07243RL" H 3450 1950 50  0001 C CNN "MPN1"
+F 4 "RC0603FR-07243RL" H 3450 1950 50  0001 C CNN "MPN"
 F 5 "ERJ-3EKF2430V" H 3450 1950 50  0001 C CNN "MPN2"
 F 6 "RMCF0603FT243R" H 3450 1950 50  0001 C CNN "MPN3"
@@
 F 2 "Capacitor_SMD:C_0603_1608Metric" H 5300 2550 50  0001 C CNN
 F 3 "" H 5300 2550 50  0001 C CNN
-F 4 "C0603C220K4GACTU" H 5300 2550 50  0001 C CNN "MPN1"
+F 4 "C0603C220K4GACTU" H 5300 2550 50  0001 C CNN "MPN"
 F 5 "VJ0603A220JXACW1BC" H 5300 2550 50  0001 C CNN "MPN2"
 F 6 "GRM1885C1H220FA01D" H 5300 2550 50  0001 C CNN "MPN3"

Commit message: bottom,sch: add comment field to some parts
Parts:
- J24: value SPDIF -> MJ-3536N; Comment (none) -> SPDIF
Changed lines of the file:
@@
 P 5575 1950
 F 0 "J24" H 5342 1929 50  0000 R CNN
-F 1 "SPDIF" H 5342 2020 50  0000 R CNN
+F 1 "MJ-3536N" H 5342 2020 50  0000 R CNN
 F 2 "footprints:MJ-3536N" H 5575 1950 50  0001 C CNN
 F 3 "https://www.cui.com/product/resource/digikeypdf/mj-3536n.pdf" H 5575 1950 50  0001 C CNN
 F 4 "MJ-3536N" H 5575 1950 50  0001 C CNN "MPN"
+F 5 "SPDIF" H 0   0   50  0001 C CNN "Comment"
 	1    5575 1950
 	-1   0    0    1

Commit message: bottom,sch: annotate schematic symbols again
Parts:
- renumbered J24 to J16
Changed lines of the file:
@@
 	5300 2350 5300 2450
 $Comp
-L Connector:AudioJack2_Ground_Switch J24
+L Connector:AudioJack2_Ground_Switch J16
 U 1 1 5B5D552C
 P 5575 1950
-F 0 "J24" H 5342 1929 50  0000 R CNN
+F 0 "J16" H 5342 1929 50  0000 R CNN
 F 1 "MJ-3536N" H 5342 2020 50  0000 R CNN
 F 2 "footprints:MJ-3536N" H 5575 1950 50  0001 C CNN

Commit message: bottom: replace coreboard connector
Parts:
- renumbered J16 to J18
Changed lines of the file:
@@
 $EndComp
 $Comp
-L power:GNDD #PWR0231
+L power:GNDD #PWR0222
 U 1 1 5B56348E
 P 3775 2350
-F 0 "#PWR0231" H 3775 2100 50  0001 C CNN
+F 0 "#PWR0222" H 3775 2100 50  0001 C CNN
 F 1 "GNDD" H 3775 2225 50  0000 C CNN
 F 2 "" H 3775 2350 50  0001 C CNN
@@
 	3200 1950 3350 1950
 $Comp
-L power:GNDD #PWR0232
+L power:GNDD #PWR0223
 U 1 1 5B56F49A
 P 4100 2450
-F 0 "#PWR0232" H 4100 2200 50  0001 C CNN
+F 0 "#PWR0223" H 4100 2200 50  0001 C CNN
 F 1 "GNDD" H 4100 2325 50  0000 C CNN
 F 2 "" H 4100 2450 50  0001 C CNN
@@
 	4600 2350 5300 2350
 $Comp
-L power:GNDD #PWR0233
+L power:GNDD #PWR0224
 U 1 1 5B56F62E
 P 5300 2725
-F 0 "#PWR0233" H 5300 2475 50  0001 C CNN
+F 0 "#PWR0224" H 5300 2475 50  0001 C CNN
 F 1 "GNDD" H 5300 2600 50  0000 C CNN
 F 2 "" H 5300 2725 50  0001 C CNN
@@
 	5300 2350 5300 2450
 $Comp
-L Connector:AudioJack2_Ground_Switch J16
+L Connector:AudioJack2_Ground_Switch J18
 U 1 1 5B5D552C
 P 5575 1950
-F 0 "J16" H 5342 1929 50  0000 R CNN
+F 0 "J18" H 5342 1929 50  0000 R CNN
 F 1 "MJ-3536N" H 5342 2020 50  0000 R CNN
 F 2 "footprints:MJ-3536N" H 5575 1950 50  0001 C CNN

Commit message: Changed the headphone buffer to FETS, also remover pull-up from Uboot button
Parts:
- J18: symbol Connector:AudioJack2_Ground_Switch -> bottom-board-rescue:AudioJack2_Ground_Switch-Connector
Changed lines of the file:
@@
 	5300 2350 5300 2450
 $Comp
-L Connector:AudioJack2_Ground_Switch J18
+L bottom-board-rescue:AudioJack2_Ground_Switch-Connector J18
 U 1 1 5B5D552C
 P 5575 1950
+AR Path="/5B5D552C" Ref="J18"  Part="1"
+AR Path="/5B6E0697/5B5D552C" Ref="J18"  Part="1"
 F 0 "J18" H 5342 1929 50  0000 R CNN
 F 1 "MJ-3536N" H 5342 2020 50  0000 R CNN
@@
 	5300 2050 5300 2350
 Connection ~ 5300 2350
-Wire Wire Line
-	5375 1950 4600 1950
 Connection ~ 3775 1950
 Wire Wire Line
@@
 Wire Wire Line
 	3550 1950 3775 1950
+Wire Wire Line
+	4600 1950 5375 1950
 $EndSCHEMATC
