File: hw-design/top-board/actuators.sch (KiCad schematic (older format))
At the start: 46 parts, among them J1 Conn_01x03_Male, J2 Conn_01x03_Male, J3 Conn_01x03_Male, J4 Conn_01x03_Male, J5 Conn_01x03_Male, J6 Conn_01x03_Male, J7 Conn_01x03_Male, J8 Conn_01x03_Male, SW2 JB15HBPC-JB, SW3 JB15HBPC-JB, SW4 JB15HBPC-JB, SW5 JB15HBPC-JB, SW6 JB15HBPC-JB, SW7 JB15HBPC-JB, SW8 JB15HBPC-JB, U6 74HC4051

Commit message: mux routing
Parts:
- removed U6: 74HC4051, QFN50P250X350X100-17N:QFN50P250X350X100-17N, symbol 74HC4051
- added U6: MAX4781EUET, MAX4781EUET:21-0066J_16, symbol MAX4781EUET
- SW2, SW3, SW4, SW5, SW6, SW7, SW8: footprint buttonLED:BUTTON -> buttonLED:BUTTONFixed
Connections:
- net +3V3: now also R27.1, SW2.6 (GND), U6.16 (VCC)
- net GNDD: now also U6.6 (*ENABLE), U6.8 (GND)
- net POTS_C_B0: now also U6.11 (A)
- net POTS_C_B1: now also U6.10 (B)
- net POTS_C_B2: now also U6.9 (C)
- net POTS_INP: now also U6.3 (X)
- net POT_1: now also U6.1 (X4)
- net POT_2: now also U6.2 (X6)
- net POT_3: now also U6.4 (X7)
- net POT_4: now also U6.5 (X5)
- net POT_5: now also U6.13 (X0)
- net POT_6: now also U6.12 (X3)
- net POT_7: now also U6.14 (X1)
- net POT_8: now also U6.15 (X2)
- net SYS_B3: now also SW4.2
- no-connect marks 12 -> 14

Commit message: libraries conflit
Parts:
- C39, C40, C41, C42: symbol C -> C-RESCUE-top-board
- R10, R15, R16, R17, R18, R19, R20, R21, R22, R23, R24, R25, R26, R27, R28, R29, R30, R31, R32, R48, R49, R5, R7, R8: symbol R -> R-RESCUE-top-board
