File: hw-design/bottom-board/PCB Source/audio-headphones.kicad_sch (KiCad schematic)
At the start: 26 parts, among them Q17 J110, Q8 J110, U14 LM4811

Commit message: update fabrication data
Parts:
- R78, R81: MPN2 (none) -> RT0603BRD071ML
Changed lines of the file:
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@@
   (title_block
     (title "MOD DuoX - Bottom Board")
-    (date "2021-11-11")
-    (rev "Rev 1.05")
+    (date "2022-01-26")
+    (rev "Rev 2.0P2")
     (company "MOD Devices GmbH")
     (comment 1 "DuoX Audio processing board")
     (comment 2 "https://github.com/moddevices/mod-hw-duoX")
-    (comment 3 "Inp Power: 12V 700mA")
-    (comment 4 "USB outp Power: 500mA")
+    (comment 3 "Inp Power: 12V 1A")
   )
   (junction (at 72.39 83.82) (diameter 0) (color 0 0 0 0)
@@
       (effects (font (size 1.27 1.27)) hide)
     )
+    (property "MPN2" "RT0603BRD071ML" (id 5) (at 72.39 41.783 0)
+      (effects (font (size 1.524 1.524)) hide)
+    )
     (pin "1")
     (pin "2")
@@
       (effects (font (size 1.27 1.27)) hide)
     )
-    (pin "1")
+    (property "MPN2" "RT0603BRD071ML" (id 5) (at 72.39 79.629 0)
+      (effects (font (size 1.524 1.524)) hide)
+    )
+    (pin "1")
